Commit message: Stashing all my changes to github lol

File: robots/panda_arm_kkc.xacro (robot description, xacro)
@@ -280,6 +280,7 @@
             <box size = "0.05 0.05 0.05"/>
         </geometry>
-        <material name="green"/>
-      </visual>
+       <!-- <material name="Green"/> -->
+        <material>Gazebo/Orange</material>
+        </visual>
     </link>
     <gazebo reference="imu_link0">
@@ -287,5 +288,5 @@
     <sensor name="imu_sensor0" type="imu">
       <always_on>true</always_on>
-      <update_rate>10</update_rate>
+      <update_rate>100</update_rate>
       <visualize>true</visualize>
       <topic>imu_data0</topic>
@@ -293,4 +294,5 @@
         <topicName>imu_data0</topicName>
         <bodyName>imu_link0</bodyName>
+        <updateRateHZ>100.0</updateRateHZ>
         <gaussianNoise>0.0</gaussianNoise>
         <xyzOffset>0.06 0 0.05</xyzOffset>
@@ -314,5 +316,5 @@
       </inertial>
       <visual>
-        <origin xyz="0.06 0 -.15" rpy="0 0 0" />
+        <origin xyz="0 -0.12 .01" rpy="0 0 0" />
         <geometry>
             <box size = ".05 .05 .05"/>
@@ -325,5 +327,5 @@
     <sensor name="imu_sensor1" type="imu">
       <always_on>true</always_on>
-      <update_rate>10</update_rate>
+      <update_rate>100</update_rate>
       <visualize>true</visualize>
       <topic>imu_data1</topic>
@@ -331,6 +333,7 @@
         <topicName>imu_data1</topicName>
         <bodyName>imu_link1</bodyName>
+        <updateRateHZ>100.0</updateRateHZ>
         <gaussianNoise>0.0</gaussianNoise>
-        <xyzOffset>0.06 0 -.15</xyzOffset>
+        <xyzOffset>0 -0.12 .01</xyzOffset>
         <rpyOffset>0 0 0</rpyOffset>
         <frameName>imu_link1</frameName>
@@ -352,7 +355,7 @@
       </inertial>
       <visual>
-        <origin xyz="0.06 -.15 0" rpy="0 0 0" />
-        <geometry>
-            <box size = ".05 .05 .05"/>
+        <origin xyz="3 3 3" rpy="0 0 0" />
+        <geometry>
+            <box size = ".1 .1 .1"/>
         </geometry>
         <material name="orange"/>
@@ -363,5 +366,5 @@
     <sensor name="imu_sensor2" type="imu">
       <always_on>true</always_on>
-      <update_rate>10</update_rate>
+      <update_rate>100</update_rate>
       <visualize>true</visualize>
       <topic>imu_data2</topic>
@@ -369,6 +372,7 @@
         <topicName>imu_data2</topicName>
         <bodyName>imu_link2</bodyName>
+        <updateRateHZ>100.0</updateRateHZ>
         <gaussianNoise>0.0</gaussianNoise>
-        <xyzOffset>0.06 -.15 0</xyzOffset>
+        <xyzOffset>0 -0.12 .01</xyzOffset>
         <rpyOffset>0 0 0</rpyOffset>
         <frameName>imu_link2</frameName>
@@ -390,9 +394,10 @@
       </inertial>
       <visual>
-        <origin xyz="-0.06 0 -0.06" rpy="0 0 0" />
+        <origin xyz="0 -0.12 .01" rpy="0 0 0" />
         <geometry>
             <box size = ".05 .05 .05"/>
         </geometry>
-        <material name="orange"/>
+<!--        <material name="orange"/>-->
+        <material>Gazebo/Green</material>
         </visual>
     </link>
@@ -401,5 +406,5 @@
     <sensor name="imu_sensor3" type="imu">
       <always_on>true</always_on>
-      <update_rate>10</update_rate>
+      <update_rate>100</update_rate>
       <visualize>true</visualize>
       <topic>imu_data3</topic>
@@ -407,6 +412,7 @@
         <topicName>imu_data3</topicName>
         <bodyName>imu_link3</bodyName>
+        <updateRateHZ>100.0</updateRateHZ>
         <gaussianNoise>0.0</gaussianNoise>
-        <xyzOffset>-0.06 0 -0.06</xyzOffset>
+        <xyzOffset>0 -0.12 .01</xyzOffset>
         <rpyOffset>0 0 0</rpyOffset>
         <frameName>imu_link3</frameName>
@@ -428,5 +434,5 @@
       </inertial>
       <visual>
-        <origin xyz="-0.14 0.09 0" rpy="0 0 0" />
+        <origin xyz="0 -0.12 .01" rpy="0 0 0" />
         <geometry>
             <box size = ".05 .05 .05"/>
@@ -439,5 +445,5 @@
     <sensor name="imu_sensor4" type="imu">
       <always_on>true</always_on>
-      <update_rate>10</update_rate>
+      <update_rate>100</update_rate>
       <visualize>true</visualize>
       <topic>imu_data4</topic>
@@ -445,6 +451,7 @@
         <topicName>imu_data4</topicName>
         <bodyName>imu_link4</bodyName>
+        <updateRateHZ>100.0</updateRateHZ>
         <gaussianNoise>0.0</gaussianNoise>
-        <xyzOffset>-0.14 0.09 0</xyzOffset>
+        <xyzOffset>0 -0.12 .01</xyzOffset>
         <rpyOffset>0 0 0</rpyOffset>
         <frameName>imu_link4</frameName>
@@ -458,24 +465,24 @@
       <child link="imu_link5"/>
       <axis xyz="0 0 0"/>
-    </joint>
-    <link name="imu_link5">
-      <inertial>
-        <origin xyz="0 0 0" rpy="0 0 0"/>
-        <mass value="0.0"/>
-        <inertia ixx="0.0" ixy="0.0" ixz="0.0" iyy="0.0" iyz="0.0" izz="0.0"/>
-      </inertial>
-      <visual>
-        <origin xyz="0 0.10 -0.11" rpy="0 0 0" />
+  </joint>
+  <link name="imu_link5">
+      <inertial>
+        <origin xyz="0 0 0" rpy="0 0 0"/>
+        <mass value="0.0"/>
+        <inertia ixx="0.0" ixy="0.0" ixz="0.0" iyy="0.0" iyz="0.0" izz="0.0"/>
+      </inertial>
+      <visual>
+        <origin xyz="-0.2 0 0" rpy="0 0 0" />
         <geometry>
             <box size = ".05 .05 .05"/>
         </geometry>
-        <material name="orange"/>
-        </visual>
-    </link>
-    <gazebo reference="imu_link5">
-    <gravity>true</gravity>
+      </visual>
+  </link>
+  <gazebo reference="imu_link5">
+    <gravity>true</gravity>
+    <material name="Y">Gazebo/YellowGlow</material>
     <sensor name="imu_sensor5" type="imu">
       <always_on>true</always_on>
-      <update_rate>10</update_rate>
+      <update_rate>100</update_rate>
       <visualize>true</visualize>
       <topic>imu_data5</topic>
@@ -483,6 +490,7 @@
         <topicName>imu_data5</topicName>
         <bodyName>imu_link5</bodyName>
+        <updateRateHZ>100.0</updateRateHZ>
         <gaussianNoise>0.0</gaussianNoise>
-        <xyzOffset>0 0.10 -0.11</xyzOffset>
+        <xyzOffset>0 -0.12 .01</xyzOffset>
         <rpyOffset>0 0 0</rpyOffset>
         <frameName>imu_link5</frameName>
@@ -491,4 +499,79 @@
     </sensor>
   </gazebo>
+<!--    IMU 5 X Axis link-->
+  <joint name = "imu_link_joint5_x_axis" type ="fixed">
+      <origin rpy="0 0 0" xyz="0 0 0"/>
+      <parent link="${arm_id}_link5"/>
+      <child link="imu_link5_x_axis"/>
+      <axis xyz="0 0 0"/>
+  </joint>
+  <link name="imu_link5_x_axis">
+      <inertial>
+        <origin xyz="0 0 0" rpy="0 0 0"/>
+        <mass value="0.0"/>
+        <inertia ixx="0.0" ixy="0.0" ixz="0.0" iyy="0.0" iyz="0.0" izz="0.0"/>
+      </inertial>
+      <visual>
+        <origin xyz="0 0 0" rpy="0 0 1.57" />
+          <geometry>
+            <cylinder length="0.2" radius="0.001"/>
+          </geometry>
+        </visual>
+  </link>
+  <gazebo reference="imu_link5_x_axis">
+    <gravity>true</gravity>
+    <material>Gazebo/RedBright</material>
+  </gazebo>
+<!--    End-->
+<!--    IMU 5 Y Axis link-->
+    <joint name = "imu_link_joint5_y_axis" type ="fixed">
+      <origin rpy="0 0 0" xyz="0 0 0"/>
+      <parent link="${arm_id}_link5"/>
+      <child link="imu_link5_y_axis"/>
+      <axis xyz="0 0 0"/>
+  </joint>
+  <link name="imu_link5_y_axis">
+      <inertial>
+        <origin xyz="0 0 0" rpy="0 0 0"/>
+        <mass value="0.0"/>
+        <inertia ixx="0.0" ixy="0.0" ixz="0.0" iyy="0.0" iyz="0.0" izz="0.0"/>
+      </inertial>
+      <visual>
+        <origin xyz="-0.2 0 0" rpy="0 1.57 0" />
+          <geometry>
+            <cylinder length="0.2" radius="0.001"/>
+          </geometry>
+        </visual>
+  </link>
+  <gazebo reference="imu_link5_y_axis">
+    <gravity>true</gravity>
+    <material>Gazebo/Green</material>
+  </gazebo>
+<!--    End-->
+<!--    IMU 5 Z Axis link-->
+  <joint name = "imu_link_joint5_z_axis" type ="fixed">
+      <origin rpy="0 0 0" xyz="0 0 0"/>
+      <parent link="${arm_id}_link5"/>
+      <child link="imu_link5_z_axis"/>
+      <axis xyz="0 0 0"/>
+  </joint>
+  <link name="imu_link5_z_axis">
+      <inertial>
+        <origin xyz="0 0 0" rpy="0 0 0"/>
+        <mass value="0.0"/>
+        <inertia ixx="0.0" ixy="0.0" ixz="0.0" iyy="0.0" iyz="0.0" izz="0.0"/>
+      </inertial>
+      <visual>
+        <origin xyz="-0.2 0 0" rpy="1.57 0 0" />
+          <geometry>
+            <cylinder length="0.2" radius="0.001"/>
+          </geometry>
+        </visual>
+  </link>
+  <gazebo reference="imu_link5_z_axis">
+    <gravity>true</gravity>
+    <material>Gazebo/Blue</material>
+  </gazebo>
+<!--    End-->
   <joint name = "imu_link_joint6" type ="fixed">
       <origin rpy="0 0 0" xyz="0 0 0"/>
@@ -504,5 +587,5 @@
       </inertial>
       <visual>
-        <origin xyz="0.13 0.02 0" rpy="0 0 0" />
+        <origin xyz="0 -0.12 .01" rpy="0 0 0" />
         <geometry>
             <box size = ".05 .05 .05"/>
@@ -515,5 +598,5 @@
     <sensor name="imu_sensor6" type="imu">
       <always_on>true</always_on>
-      <update_rate>10</update_rate>
+      <update_rate>100</update_rate>
       <visualize>true</visualize>
       <topic>imu_data1</topic>
@@ -521,6 +604,7 @@
         <topicName>imu_data6</topicName>
         <bodyName>imu_link6</bodyName>
+        <updateRateHZ>100.0</updateRateHZ>
         <gaussianNoise>0.0</gaussianNoise>
-        <xyzOffset>0.13 0.02 0</xyzOffset>
+        <xyzOffset>0 -0.12 .01</xyzOffset>
         <rpyOffset>0 0 0</rpyOffset>
         <frameName>imu_link6</frameName>
