Commit message: Added dependencies to cmake.

File: robots/panda_arm.xacro (robot description, xacro)
@@ -262,5 +262,5 @@
       <axis xyz="0 0 0"/>
     </joint>
-    <joint name = "imu_link_joint0" type ="fixed">
+    <!--<joint name = "imu_link_joint0" type ="fixed">
       <origin rpy="0 0 0" xyz="0 0 0"/>
       <parent link="${arm_id}_link0"/>
@@ -277,5 +277,5 @@
         <origin xyz="0.06 0 0.05" rpy="0 0 0" />
         <geometry>
-            <box size = "0.05 0.05 0.05"/>
+            <box size = "0.25 0.25 0.25"/>
         </geometry>
         <material name="green"/>
@@ -300,4 +300,5 @@
     </sensor>
   </gazebo>
+-->
 <joint name = "imu_link_joint1" type ="fixed">
       <origin rpy="0 0 0" xyz="0 0 0"/>
@@ -351,7 +352,7 @@
       </inertial>
       <visual>
-        <origin xyz="0 -0.12 .01" rpy="0 0 0" />
-        <geometry>
-            <box size = ".05 .05 .05"/>
+        <origin xyz="3 3 3" rpy="0 0 0" />
+        <geometry>
+            <box size = ".1 .1 .1"/>
         </geometry>
         <material name="orange"/>

Commit message: modified-urdf

File: robots/panda_arm.xacro (robot description, xacro)
@@ -262,5 +262,6 @@
       <axis xyz="0 0 0"/>
     </joint>
-    <!--<joint name = "imu_link_joint0" type ="fixed">
+<!-- aaaaaaaaaaaaaaaaaaaaaaaaaaaaaaaaaaaaaaaaaaaaaaaaaaaaaaaaaaaaaaaaaaaaaaaaaaaaaaaaaaaaaaaaaaaaaaaaaaaaaaaaaaaaa -->
+    <joint name = "imu_link_joint0" type ="fixed">
       <origin rpy="0 0 0" xyz="0 0 0"/>
       <parent link="${arm_id}_link0"/>
@@ -277,5 +278,5 @@
         <origin xyz="0.06 0 0.05" rpy="0 0 0" />
         <geometry>
-            <box size = "0.25 0.25 0.25"/>
+            <box size = "0.05 0.05 0.05"/>
         </geometry>
         <material name="green"/>
@@ -300,5 +301,4 @@
     </sensor>
   </gazebo>
--->
 <joint name = "imu_link_joint1" type ="fixed">
       <origin rpy="0 0 0" xyz="0 0 0"/>

Commit message: Adjustments to IMU positions in Xacro

File: robots/panda_arm.xacro (robot description, xacro)
@@ -314,5 +314,5 @@
       </inertial>
       <visual>
-        <origin xyz="0 -0.12 .01" rpy="0 0 0" />
+        <origin xyz="0.06 0 -.15" rpy="0 0 0" />
         <geometry>
             <box size = ".05 .05 .05"/>
@@ -332,5 +332,5 @@
         <bodyName>imu_link1</bodyName>
         <gaussianNoise>0.0</gaussianNoise>
-        <xyzOffset>0 -0.12 .01</xyzOffset>
+        <xyzOffset>0.06 0 -.15</xyzOffset>
         <rpyOffset>0 0 0</rpyOffset>
         <frameName>imu_link1</frameName>
@@ -352,7 +352,7 @@
       </inertial>
       <visual>
-        <origin xyz="3 3 3" rpy="0 0 0" />
-        <geometry>
-            <box size = ".1 .1 .1"/>
+        <origin xyz="0.06 -.15 0" rpy="0 0 0" />
+        <geometry>
+            <box size = ".05 .05 .05"/>
         </geometry>
         <material name="orange"/>
@@ -370,5 +370,5 @@
         <bodyName>imu_link2</bodyName>
         <gaussianNoise>0.0</gaussianNoise>
-        <xyzOffset>0 -0.12 .01</xyzOffset>
+        <xyzOffset>0.06 -.15 0</xyzOffset>
         <rpyOffset>0 0 0</rpyOffset>
         <frameName>imu_link2</frameName>
@@ -390,5 +390,5 @@
       </inertial>
       <visual>
-        <origin xyz="0 -0.12 .01" rpy="0 0 0" />
+        <origin xyz="-0.06 0 -0.06" rpy="0 0 0" />
         <geometry>
             <box size = ".05 .05 .05"/>
@@ -408,5 +408,5 @@
         <bodyName>imu_link3</bodyName>
         <gaussianNoise>0.0</gaussianNoise>
-        <xyzOffset>0 -0.12 .01</xyzOffset>
+        <xyzOffset>-0.06 0 -0.06</xyzOffset>
         <rpyOffset>0 0 0</rpyOffset>
         <frameName>imu_link3</frameName>
@@ -428,7 +428,7 @@
       </inertial>
       <visual>
-        <origin xyz="0 -0.12 .01" rpy="0 0 0" />
-        <geometry>
-            <box size = ".05 .05 .05"/>
+        <origin xyz="0 0 0" rpy="0 0 0" />
+        <geometry>
+            <box size = ".25 .05 .05"/>
         </geometry>
         <material name="orange"/>
@@ -466,7 +466,7 @@
       </inertial>
       <visual>
-        <origin xyz="0 -0.12 .01" rpy="0 0 0" />
-        <geometry>
-            <box size = ".05 .05 .05"/>
+        <origin xyz="0 0 0" rpy="0 0 0" />
+        <geometry>
+            <box size = ".25 .05 .05"/>
         </geometry>
         <material name="orange"/>
@@ -504,7 +504,7 @@
       </inertial>
       <visual>
-        <origin xyz="0 -0.12 .01" rpy="0 0 0" />
-        <geometry>
-            <box size = ".05 .05 .05"/>
+        <origin xyz="0 0 0" rpy="0 0 0" />
+        <geometry>
+            <box size = ".25 .05 .05"/>
         </geometry>
         <material name="orange"/>

Commit message: Making Joint movement exactly as Caleb, not editing it

File: robots/panda_arm.xacro (robot description, xacro)
@@ -432,5 +432,5 @@
       </inertial>
       <visual>
-        <origin xyz="0 -0.12 .01" rpy="0 0 0" />
+        <origin xyz="0 0 0" rpy="0 0 0" />
         <geometry>
             <box size = ".05 .05 .05"/>

Commit message: Some good changes

File: robots/panda_arm.xacro (robot description, xacro)
@@ -280,5 +280,6 @@
             <box size = "0.05 0.05 0.05"/>
         </geometry>
-        <material name="green"/>
+       <!-- <material name="Green"/> -->
+        <material>Gazebo/Orange</material>
         </visual>
     </link>
@@ -397,5 +398,6 @@
             <box size = ".05 .05 .05"/>
         </geometry>
-        <material name="orange"/>
+<!--        <material name="orange"/>-->
+        <material>Gazebo/Green</material>
         </visual>
     </link>
@@ -471,13 +473,22 @@
       </inertial>
       <visual>
-        <origin xyz="0 -0.12 .01" rpy="0 0 0" />
+        <origin xyz="0 0 0" rpy="0 0 0" />
         <geometry>
             <box size = ".05 .05 .05"/>
         </geometry>
-        <material name="orange"/>
-        </visual>
+      </visual>
+<!--      Edited By krishna-->
+      <visual>
+        <origin xyz="0 0 0" rpy="0 0 0" />
+          <pose> -1.0 0 0 1.57 0 0</pose>
+          <geometry>
+            <cylinder length="0.2" radius="0.001"/>
+          </geometry>
+        </visual>
+<!--      edited by krishna-->
     </link>
     <gazebo reference="imu_link5">
     <gravity>true</gravity>
+      <material>Gazebo/RedBright</material>
     <sensor name="imu_sensor5" type="imu">
       <always_on>true</always_on>

Commit message: Axes Working

File: robots/panda_arm.xacro (robot description, xacro)
@@ -465,30 +465,21 @@
       <child link="imu_link5"/>
       <axis xyz="0 0 0"/>
-    </joint>
-    <link name="imu_link5">
-      <inertial>
-        <origin xyz="0 0 0" rpy="0 0 0"/>
-        <mass value="0.0"/>
-        <inertia ixx="0.0" ixy="0.0" ixz="0.0" iyy="0.0" iyz="0.0" izz="0.0"/>
-      </inertial>
-      <visual>
-        <origin xyz="0 0 0" rpy="0 0 0" />
+  </joint>
+  <link name="imu_link5">
+      <inertial>
+        <origin xyz="0 0 0" rpy="0 0 0"/>
+        <mass value="0.0"/>
+        <inertia ixx="0.0" ixy="0.0" ixz="0.0" iyy="0.0" iyz="0.0" izz="0.0"/>
+      </inertial>
+      <visual>
+        <origin xyz="-0.2 0 0" rpy="0 0 0" />
         <geometry>
             <box size = ".05 .05 .05"/>
         </geometry>
       </visual>
-<!--      Edited By krishna-->
-      <visual>
-        <origin xyz="0 0 0" rpy="0 0 0" />
-          <pose> -1.0 0 0 1.57 0 0</pose>
-          <geometry>
-            <cylinder length="0.2" radius="0.001"/>
-          </geometry>
-        </visual>
-<!--      edited by krishna-->
-    </link>
-    <gazebo reference="imu_link5">
-    <gravity>true</gravity>
-      <material>Gazebo/RedBright</material>
+  </link>
+  <gazebo reference="imu_link5">
+    <gravity>true</gravity>
+    <material name="Y">Gazebo/YellowGlow</material>
     <sensor name="imu_sensor5" type="imu">
       <always_on>true</always_on>
@@ -508,4 +499,79 @@
     </sensor>
   </gazebo>
+<!--    IMU 5 X Axis link-->
+    <joint name = "imu_link_joint5_x_axis" type ="fixed">
+      <origin rpy="0 0 0" xyz="0 0 0"/>
+      <parent link="${arm_id}_link5"/>
+      <child link="imu_link5_x_axis"/>
+      <axis xyz="0 0 0"/>
+  </joint>
+  <link name="imu_link5_x_axis">
+      <inertial>
+        <origin xyz="0 0 0" rpy="0 0 0"/>
+        <mass value="0.0"/>
+        <inertia ixx="0.0" ixy="0.0" ixz="0.0" iyy="0.0" iyz="0.0" izz="0.0"/>
+      </inertial>
+      <visual>
+        <origin xyz="-0.2 0 0" rpy="0 0 1.57" />
+          <geometry>
+            <cylinder length="0.2" radius="0.001"/>
+          </geometry>
+        </visual>
+  </link>
+  <gazebo reference="imu_link5_x_axis">
+    <gravity>true</gravity>
+    <material>Gazebo/RedBright</material>
+  </gazebo>
+<!--    End-->
+<!--    IMU 5 Y Axis link-->
+    <joint name = "imu_link_joint5_y_axis" type ="fixed">
+      <origin rpy="0 0 0" xyz="0 0 0"/>
+      <parent link="${arm_id}_link5"/>
+      <child link="imu_link5_y_axis"/>
+      <axis xyz="0 0 0"/>
+  </joint>
+  <link name="imu_link5_y_axis">
+      <inertial>
+        <origin xyz="0 0 0" rpy="0 0 0"/>
+        <mass value="0.0"/>
+        <inertia ixx="0.0" ixy="0.0" ixz="0.0" iyy="0.0" iyz="0.0" izz="0.0"/>
+      </inertial>
+      <visual>
+        <origin xyz="-0.2 0 0" rpy="0 1.57 0" />
+          <geometry>
+            <cylinder length="0.2" radius="0.001"/>
+          </geometry>
+        </visual>
+  </link>
+  <gazebo reference="imu_link5_y_axis">
+    <gravity>true</gravity>
+    <material>Gazebo/Green</material>
+  </gazebo>
+<!--    End-->
+<!--    IMU 5 Z Axis link-->
+    <joint name = "imu_link_joint5_z_axis" type ="fixed">
+      <origin rpy="0 0 0" xyz="0 0 0"/>
+      <parent link="${arm_id}_link5"/>
+      <child link="imu_link5_z_axis"/>
+      <axis xyz="0 0 0"/>
+  </joint>
+  <link name="imu_link5_z_axis">
+      <inertial>
+        <origin xyz="0 0 0" rpy="0 0 0"/>
+        <mass value="0.0"/>
+        <inertia ixx="0.0" ixy="0.0" ixz="0.0" iyy="0.0" iyz="0.0" izz="0.0"/>
+      </inertial>
+      <visual>
+        <origin xyz="-0.2 0 0" rpy="1.57 0 0" />
+          <geometry>
+            <cylinder length="0.2" radius="0.001"/>
+          </geometry>
+        </visual>
+  </link>
+  <gazebo reference="imu_link5_z_axis">
+    <gravity>true</gravity>
+    <material>Gazebo/Blue</material>
+  </gazebo>
+<!--    End-->
   <joint name = "imu_link_joint6" type ="fixed">
       <origin rpy="0 0 0" xyz="0 0 0"/>

Commit message: Added IMU 4 position

File: robots/panda_arm.xacro (robot description, xacro)
@@ -281,5 +281,5 @@
         </geometry>
         <material name="green"/>
-        </visual>
+      </visual>
     </link>
     <gazebo reference="imu_link0">
@@ -428,7 +428,7 @@
       </inertial>
       <visual>
-        <origin xyz="0 0 0" rpy="0 0 0" />
-        <geometry>
-            <box size = ".25 .05 .05"/>
+        <origin xyz="-0.14 0.09 0" rpy="0 0 0" />
+        <geometry>
+            <box size = ".05 .05 .05"/>
         </geometry>
         <material name="orange"/>
@@ -446,5 +446,5 @@
         <bodyName>imu_link4</bodyName>
         <gaussianNoise>0.0</gaussianNoise>
-        <xyzOffset>0 -0.12 .01</xyzOffset>
+        <xyzOffset>-0.14 0.09 0</xyzOffset>
         <rpyOffset>0 0 0</rpyOffset>
         <frameName>imu_link4</frameName>

Commit message: Commit all changes

File: robots/panda_arm.xacro (robot description, xacro)
@@ -434,5 +434,5 @@
       </inertial>
       <visual>
-        <origin xyz="0 0 0" rpy="0 0 0" />
+        <origin xyz="0 -0.12 .01" rpy="0 0 0" />
         <geometry>
             <box size = ".05 .05 .05"/>

Commit message: Updated IMU 5 to its correct position

File: robots/panda_arm.xacro (robot description, xacro)
@@ -466,7 +466,7 @@
       </inertial>
       <visual>
-        <origin xyz="0 0 0" rpy="0 0 0" />
-        <geometry>
-            <box size = ".25 .05 .05"/>
+        <origin xyz="0 0.10 -0.11" rpy="0 0 0" />
+        <geometry>
+            <box size = ".05 .05 .05"/>
         </geometry>
         <material name="orange"/>
@@ -484,5 +484,5 @@
         <bodyName>imu_link5</bodyName>
         <gaussianNoise>0.0</gaussianNoise>
-        <xyzOffset>0 -0.12 .01</xyzOffset>
+        <xyzOffset>0 0.10 -0.11</xyzOffset>
         <rpyOffset>0 0 0</rpyOffset>
         <frameName>imu_link5</frameName>

Commit message: Fixed IMU 6 position

File: robots/panda_arm.xacro (robot description, xacro)
@@ -504,7 +504,7 @@
       </inertial>
       <visual>
-        <origin xyz="0 0 0" rpy="0 0 0" />
-        <geometry>
-            <box size = ".25 .05 .05"/>
+        <origin xyz="0.13 0.02 0" rpy="0 0 0" />
+        <geometry>
+            <box size = ".05 .05 .05"/>
         </geometry>
         <material name="orange"/>
@@ -522,5 +522,5 @@
         <bodyName>imu_link6</bodyName>
         <gaussianNoise>0.0</gaussianNoise>
-        <xyzOffset>0 -0.12 .01</xyzOffset>
+        <xyzOffset>0.13 0.02 0</xyzOffset>
         <rpyOffset>0 0 0</rpyOffset>
         <frameName>imu_link6</frameName>

Commit message: Add material

File: robots/panda_arm.xacro (robot description, xacro)
@@ -262,5 +262,5 @@
       <axis xyz="0 0 0"/>
     </joint>
-<!-- aaaaaaaaaaaaaaaaaaaaaaaaaaaaaaaaaaaaaaaaaaaaaaaaaaaaaaaaaaaaaaaaaaaaaaaaaaaaaaaaaaaaaaaaaaaaaaaaaaaaaaaaaaaaa -->
+<!-- IMU Placement changes start from here. In kandai's words: aaaaaaaaaaa -->
     <joint name = "imu_link_joint0" type ="fixed">
       <origin rpy="0 0 0" xyz="0 0 0"/>
@@ -290,4 +290,6 @@
       <visualize>true</visualize>
       <topic>imu_data0</topic>
+<!--      Below is the line to change the material-->
+      <material>Gazebo/YellowGlow</material>
       <plugin filename="libgazebo_ros_imu_sensor.so" name="imu_plugin">
         <topicName>imu_data0</topicName>
@@ -328,4 +330,6 @@
       <visualize>true</visualize>
       <topic>imu_data1</topic>
+<!--      Below is the line to change the material-->
+      <material>Gazebo/YellowGlow</material>
       <plugin filename="libgazebo_ros_imu_sensor.so" name="imu_plugin">
         <topicName>imu_data1</topicName>
@@ -366,4 +370,6 @@
       <visualize>true</visualize>
       <topic>imu_data2</topic>
+<!--      Below is the line to change the material-->
+      <material>Gazebo/YellowGlow</material>
       <plugin filename="libgazebo_ros_imu_sensor.so" name="imu_plugin">
         <topicName>imu_data2</topicName>
@@ -404,4 +410,6 @@
       <visualize>true</visualize>
       <topic>imu_data3</topic>
+<!--      Below is the line to change the material-->
+      <material>Gazebo/YellowGlow</material>
       <plugin filename="libgazebo_ros_imu_sensor.so" name="imu_plugin">
         <topicName>imu_data3</topicName>
@@ -442,4 +450,6 @@
       <visualize>true</visualize>
       <topic>imu_data4</topic>
+<!--      Below is the line to change the material-->
+      <material>Gazebo/YellowGlow</material>
       <plugin filename="libgazebo_ros_imu_sensor.so" name="imu_plugin">
         <topicName>imu_data4</topicName>
@@ -480,4 +490,6 @@
       <visualize>true</visualize>
       <topic>imu_data5</topic>
+<!--      Below is the line to change the material-->
+      <material>Gazebo/YellowGlow</material>
       <plugin filename="libgazebo_ros_imu_sensor.so" name="imu_plugin">
         <topicName>imu_data5</topicName>
@@ -518,4 +530,6 @@
       <visualize>true</visualize>
       <topic>imu_data1</topic>
+<!--      Below is the line to change the material-->
+      <material>Gazebo/YellowGlow</material>
       <plugin filename="libgazebo_ros_imu_sensor.so" name="imu_plugin">
         <topicName>imu_data6</topicName>

Commit message: Colors Working

File: robots/panda_arm.xacro (robot description, xacro)
@@ -280,9 +280,10 @@
             <box size = "0.05 0.05 0.05"/>
         </geometry>
-        <material name="green"/>
       </visual>
     </link>
     <gazebo reference="imu_link0">
     <gravity>true</gravity>
+    <!--      Below is the line to change the material-->
+    <material>Gazebo/YellowGlow</material>
     <sensor name="imu_sensor0" type="imu">
       <always_on>true</always_on>
@@ -290,6 +291,4 @@
       <visualize>true</visualize>
       <topic>imu_data0</topic>
-<!--      Below is the line to change the material-->
-      <material>Gazebo/YellowGlow</material>
       <plugin filename="libgazebo_ros_imu_sensor.so" name="imu_plugin">
         <topicName>imu_data0</topicName>
@@ -325,4 +324,6 @@
     <gazebo reference="imu_link1">
     <gravity>true</gravity>
+    <!--      Below is the line to change the material-->
+    <material>Gazebo/YellowGlow</material>
     <sensor name="imu_sensor1" type="imu">
       <always_on>true</always_on>
@@ -330,6 +331,4 @@
       <visualize>true</visualize>
       <topic>imu_data1</topic>
-<!--      Below is the line to change the material-->
-      <material>Gazebo/YellowGlow</material>
       <plugin filename="libgazebo_ros_imu_sensor.so" name="imu_plugin">
         <topicName>imu_data1</topicName>
@@ -365,4 +364,6 @@
     <gazebo reference="imu_link2">
     <gravity>true</gravity>
+    <!--      Below is the line to change the material-->
+    <material>Gazebo/YellowGlow</material>
     <sensor name="imu_sensor2" type="imu">
       <always_on>true</always_on>
@@ -370,6 +371,4 @@
       <visualize>true</visualize>
       <topic>imu_data2</topic>
-<!--      Below is the line to change the material-->
-      <material>Gazebo/YellowGlow</material>
       <plugin filename="libgazebo_ros_imu_sensor.so" name="imu_plugin">
         <topicName>imu_data2</topicName>
@@ -405,4 +404,6 @@
     <gazebo reference="imu_link3">
     <gravity>true</gravity>
+    <!--      Below is the line to change the material-->
+    <material>Gazebo/YellowGlow</material>
     <sensor name="imu_sensor3" type="imu">
       <always_on>true</always_on>
@@ -410,6 +411,4 @@
       <visualize>true</visualize>
       <topic>imu_data3</topic>
-<!--      Below is the line to change the material-->
-      <material>Gazebo/YellowGlow</material>
       <plugin filename="libgazebo_ros_imu_sensor.so" name="imu_plugin">
         <topicName>imu_data3</topicName>
@@ -445,4 +444,6 @@
     <gazebo reference="imu_link4">
     <gravity>true</gravity>
+    <!--      Below is the line to change the material-->
+    <material>Gazebo/YellowGlow</material>
     <sensor name="imu_sensor4" type="imu">
       <always_on>true</always_on>
@@ -450,6 +451,4 @@
       <visualize>true</visualize>
       <topic>imu_data4</topic>
-<!--      Below is the line to change the material-->
-      <material>Gazebo/YellowGlow</material>
       <plugin filename="libgazebo_ros_imu_sensor.so" name="imu_plugin">
         <topicName>imu_data4</topicName>
@@ -485,4 +484,6 @@
     <gazebo reference="imu_link5">
     <gravity>true</gravity>
+    <!--      Below is the line to change the material-->
+    <material>Gazebo/YellowGlow</material>
     <sensor name="imu_sensor5" type="imu">
       <always_on>true</always_on>
@@ -490,6 +491,4 @@
       <visualize>true</visualize>
       <topic>imu_data5</topic>
-<!--      Below is the line to change the material-->
-      <material>Gazebo/YellowGlow</material>
       <plugin filename="libgazebo_ros_imu_sensor.so" name="imu_plugin">
         <topicName>imu_data5</topicName>
@@ -525,4 +524,6 @@
     <gazebo reference="imu_link6">
     <gravity>true</gravity>
+    <!--      Below is the line to change the material-->
+    <material>Gazebo/YellowGlow</material>
     <sensor name="imu_sensor6" type="imu">
       <always_on>true</always_on>
@@ -530,6 +531,4 @@
       <visualize>true</visualize>
       <topic>imu_data1</topic>
-<!--      Below is the line to change the material-->
-      <material>Gazebo/YellowGlow</material>
       <plugin filename="libgazebo_ros_imu_sensor.so" name="imu_plugin">
         <topicName>imu_data6</topicName>

Commit message: Some more cleaning up of code

File: robots/panda_arm.xacro (robot description, xacro)
@@ -319,5 +319,4 @@
             <box size = ".05 .05 .05"/>
         </geometry>
-        <material name="orange"/>
         </visual>
     </link>
@@ -359,5 +358,4 @@
             <box size = ".05 .05 .05"/>
         </geometry>
-        <material name="orange"/>
         </visual>
     </link>
@@ -399,5 +397,4 @@
             <box size = ".05 .05 .05"/>
         </geometry>
-        <material name="orange"/>
         </visual>
     </link>
@@ -439,5 +436,4 @@
             <box size = ".05 .05 .05"/>
         </geometry>
-        <material name="orange"/>
         </visual>
     </link>
@@ -479,5 +475,4 @@
             <box size = ".05 .05 .05"/>
         </geometry>
-        <material name="orange"/>
         </visual>
     </link>
@@ -519,5 +514,4 @@
             <box size = ".05 .05 .05"/>
         </geometry>
-        <material name="orange"/>
         </visual>
     </link>
