Commit message: Started writing my own xacro parser, to make everything dynamic

File: robots/panda_arm.xacro (robot description, xacro)
@@ -302,4 +302,84 @@
     </sensor>
   </gazebo>
+<!--    Joint 0 Axes Start-->
+<!--    IMU 0 X Axis link-->
+  <joint name = "imu_link_joint0_x_axis" type ="fixed">
+      <origin rpy="0 0 0" xyz="0 0 0"/>
+      <parent link="${arm_id}_link0"/>
+      <child link="imu_link0_x_axis"/>
+      <axis xyz="0 0 0"/>
+  </joint>
+  <link name="imu_link0_x_axis">
+      <inertial>
+        <origin xyz="0 0 0" rpy="0 0 0"/>
+        <mass value="0.0"/>
+        <inertia ixx="0.0" ixy="0.0" ixz="0.0" iyy="0.0" iyz="0.0" izz="0.0"/>
+      </inertial>
+      <visual>
+        <origin xyz="0.06 0 0.05" rpy="1.57 0 0" />
+          <geometry>
+            <mesh scale="0.007 0.007 0.007" filename="package://${description_pkg}/meshes/visual/arrow.dae"/>
+<!--            <cylinder length="0.07" radius="0.001"/>-->
+          </geometry>
+        </visual>
+  </link>
+  <gazebo reference="imu_link0_x_axis">
+    <gravity>true</gravity>
+    <material>Gazebo/RedBright</material>
+  </gazebo>
+<!--    End-->
+<!--    IMU 5 Y Axis link-->
+    <joint name = "imu_link_joint0_y_axis" type ="fixed">
+      <origin rpy="0 0 0" xyz="0 0 0"/>
+      <parent link="${arm_id}_link0"/>
+      <child link="imu_link0_y_axis"/>
+      <axis xyz="0 0 0"/>
+  </joint>
+  <link name="imu_link0_y_axis">
+      <inertial>
+        <origin xyz="0 0 0" rpy="0 0 0"/>
+        <mass value="0.0"/>
+        <inertia ixx="0.0" ixy="0.0" ixz="0.0" iyy="0.0" iyz="0.0" izz="0.0"/>
+      </inertial>
+      <visual>
+        <origin xyz="0.06 0 0.05" rpy="0 1.57 0" />
+          <geometry>
+            <mesh scale="0.007 0.007 0.007" filename="package://${description_pkg}/meshes/visual/arrow.dae"/>
+<!--            <cylinder length="0.07" radius="0.001"/>-->
+          </geometry>
+        </visual>
+  </link>
+  <gazebo reference="imu_link0_y_axis">
+    <gravity>true</gravity>
+    <material>Gazebo/Green</material>
+  </gazebo>
+<!--    End-->
+<!--    IMU 5 Z Axis link-->
+  <joint name = "imu_link_joint0_z_axis" type ="fixed">
+      <origin rpy="0 0 0" xyz="0 0 0"/>
+      <parent link="${arm_id}_link0"/>
+      <child link="imu_link0_z_axis"/>
+      <axis xyz="0 0 0"/>
+  </joint>
+  <link name="imu_link0_z_axis">
+      <inertial>
+        <origin xyz="0 0 0" rpy="0 0 0"/>
+        <mass value="0.0"/>
+        <inertia ixx="0.0" ixy="0.0" ixz="0.0" iyy="0.0" iyz="0.0" izz="0.0"/>
+      </inertial>
+      <visual>
+        <origin xyz="0.06 0 0.05" rpy="0 0 1.57" />
+          <geometry>
+<!--            <cylinder length="0.07" radius="0.001"/>-->
+            <mesh scale="0.007 0.007 0.007" filename="package://${description_pkg}/meshes/visual/arrow.dae"/>
+          </geometry>
+        </visual>
+  </link>
+  <gazebo reference="imu_link0_z_axis">
+    <gravity>true</gravity>
+    <material>Gazebo/Blue</material>
+  </gazebo>
+<!--    End-->
+<!--    Joint 0 Axes End-->
 <joint name = "imu_link_joint1" type ="fixed">
       <origin rpy="0 0 0" xyz="0 0 0"/>
@@ -341,4 +421,84 @@
     </sensor>
   </gazebo>
+    <!--    Joint 1 Axes Start-->
+<!--    IMU 0 X Axis link-->
+  <joint name = "imu_link_joint1_x_axis" type ="fixed">
+      <origin rpy="0 0 0" xyz="0 0 0"/>
+      <parent link="${arm_id}_link1"/>
+      <child link="imu_link1_x_axis"/>
+      <axis xyz="0 0 0"/>
+  </joint>
+  <link name="imu_link1_x_axis">
+      <inertial>
+        <origin xyz="0 0 0" rpy="0 0 0"/>
+        <mass value="0.0"/>
+        <inertia ixx="0.0" ixy="0.0" ixz="0.0" iyy="0.0" iyz="0.0" izz="0.0"/>
+      </inertial>
+      <visual>
+        <origin xyz="0.06 0 -.15" rpy="1.57 0 0" />
+          <geometry>
+            <mesh scale="0.007 0.007 0.007" filename="package://${description_pkg}/meshes/visual/arrow.dae"/>
+<!--            <cylinder length="0.07" radius="0.001"/>-->
+          </geometry>
+        </visual>
+  </link>
+  <gazebo reference="imu_link1_x_axis">
+    <gravity>true</gravity>
+    <material>Gazebo/RedBright</material>
+  </gazebo>
+<!--    End-->
+<!--    IMU 5 Y Axis link-->
+    <joint name = "imu_link_joint1_y_axis" type ="fixed">
+      <origin rpy="0 0 0" xyz="0 0 0"/>
+      <parent link="${arm_id}_link1"/>
+      <child link="imu_link1_y_axis"/>
+      <axis xyz="0 0 0"/>
+  </joint>
+  <link name="imu_link1_y_axis">
+      <inertial>
+        <origin xyz="0 0 0" rpy="0 0 0"/>
+        <mass value="0.0"/>
+        <inertia ixx="0.0" ixy="0.0" ixz="0.0" iyy="0.0" iyz="0.0" izz="0.0"/>
+      </inertial>
+      <visual>
+        <origin xyz="0.06 0 -.15" rpy="0 1.57 0" />
+          <geometry>
+            <mesh scale="0.007 0.007 0.007" filename="package://${description_pkg}/meshes/visual/arrow.dae"/>
+<!--            <cylinder length="0.07" radius="0.001"/>-->
+          </geometry>
+        </visual>
+  </link>
+  <gazebo reference="imu_link1_y_axis">
+    <gravity>true</gravity>
+    <material>Gazebo/Green</material>
+  </gazebo>
+<!--    End-->
+<!--    IMU 5 Z Axis link-->
+  <joint name = "imu_link_joint1_z_axis" type ="fixed">
+      <origin rpy="0 0 0" xyz="0 0 0"/>
+      <parent link="${arm_id}_link1"/>
+      <child link="imu_link1_z_axis"/>
+      <axis xyz="0 0 0"/>
+  </joint>
+  <link name="imu_link1_z_axis">
+      <inertial>
+        <origin xyz="0 0 0" rpy="0 0 0"/>
+        <mass value="0.0"/>
+        <inertia ixx="0.0" ixy="0.0" ixz="0.0" iyy="0.0" iyz="0.0" izz="0.0"/>
+      </inertial>
+      <visual>
+        <origin xyz="0.06 0 -.15" rpy="0 0 1.57" />
+          <geometry>
+<!--            <cylinder length="0.07" radius="0.001"/>-->
+            <mesh scale="0.007 0.007 0.007" filename="package://${description_pkg}/meshes/visual/arrow.dae"/>
+          </geometry>
+        </visual>
+  </link>
+  <gazebo reference="imu_link1_z_axis">
+    <gravity>true</gravity>
+    <material>Gazebo/Blue</material>
+  </gazebo>
+<!--    End-->
+<!--    Joint 1 Axes End-->
   <joint name = "imu_link_joint2" type ="fixed">
       <origin rpy="0 0 0" xyz="0 0 0"/>
@@ -355,4 +515,5 @@
       <visual>
         <origin xyz="0.06 -.15 0" rpy="0 0 0" />
+<!--        <origin xyz="${props['IMU2_Position_x']}" rpy="0 0 0" />-->
         <geometry>
             <box size = ".05 .05 .05"/>
@@ -380,4 +541,84 @@
     </sensor>
   </gazebo>
+    <!--    Joint 2 Axes Start-->
+<!--    IMU 2 X Axis link-->
+  <joint name = "imu_link_joint2_x_axis" type ="fixed">
+      <origin rpy="0 0 0" xyz="0 0 0"/>
+      <parent link="${arm_id}_link2"/>
+      <child link="imu_link2_x_axis"/>
+      <axis xyz="0 0 0"/>
+  </joint>
+  <link name="imu_link2_x_axis">
+      <inertial>
+        <origin xyz="0 0 0" rpy="0 0 0"/>
+        <mass value="0.0"/>
+        <inertia ixx="0.0" ixy="0.0" ixz="0.0" iyy="0.0" iyz="0.0" izz="0.0"/>
+      </inertial>
+      <visual>
+        <origin xyz="0.06 -.15 0" rpy="1.57 0 0" />
+          <geometry>
+            <mesh scale="0.007 0.007 0.007" filename="package://${description_pkg}/meshes/visual/arrow.dae"/>
+<!--            <cylinder length="0.07" radius="0.001"/>-->
+          </geometry>
+        </visual>
+  </link>
+  <gazebo reference="imu_link2_x_axis">
+    <gravity>true</gravity>
+    <material>Gazebo/RedBright</material>
+  </gazebo>
+<!--    End-->
+<!--    IMU 5 Y Axis link-->
+    <joint name = "imu_link_joint2_y_axis" type ="fixed">
+      <origin rpy="0 0 0" xyz="0 0 0"/>
+      <parent link="${arm_id}_link2"/>
+      <child link="imu_link2_y_axis"/>
+      <axis xyz="0 0 0"/>
+  </joint>
+  <link name="imu_link2_y_axis">
+      <inertial>
+        <origin xyz="0 0 0" rpy="0 0 0"/>
+        <mass value="0.0"/>
+        <inertia ixx="0.0" ixy="0.0" ixz="0.0" iyy="0.0" iyz="0.0" izz="0.0"/>
+      </inertial>
+      <visual>
+        <origin xyz="0.06 -.15 0" rpy="0 1.57 0" />
+          <geometry>
+            <mesh scale="0.007 0.007 0.007" filename="package://${description_pkg}/meshes/visual/arrow.dae"/>
+<!--            <cylinder length="0.07" radius="0.001"/>-->
+          </geometry>
+        </visual>
+  </link>
+  <gazebo reference="imu_link2_y_axis">
+    <gravity>true</gravity>
+    <material>Gazebo/Green</material>
+  </gazebo>
+<!--    End-->
+<!--    IMU 5 Z Axis link-->
+  <joint name = "imu_link_joint2_z_axis" type ="fixed">
+      <origin rpy="0 0 0" xyz="0 0 0"/>
+      <parent link="${arm_id}_link2"/>
+      <child link="imu_link2_z_axis"/>
+      <axis xyz="0 0 0"/>
+  </joint>
+  <link name="imu_link2_z_axis">
+      <inertial>
+        <origin xyz="0 0 0" rpy="0 0 0"/>
+        <mass value="0.0"/>
+        <inertia ixx="0.0" ixy="0.0" ixz="0.0" iyy="0.0" iyz="0.0" izz="0.0"/>
+      </inertial>
+      <visual>
+        <origin xyz="0.06 -.15 0" rpy="0 0 1.57" />
+          <geometry>
+<!--            <cylinder length="0.07" radius="0.001"/>-->
+            <mesh scale="0.007 0.007 0.007" filename="package://${description_pkg}/meshes/visual/arrow.dae"/>
+          </geometry>
+        </visual>
+  </link>
+  <gazebo reference="imu_link2_z_axis">
+    <gravity>true</gravity>
+    <material>Gazebo/Blue</material>
+  </gazebo>
+<!--    End-->
+<!--    Joint 2 Axes End-->
   <joint name = "imu_link_joint3" type ="fixed">
       <origin rpy="0 0 0" xyz="0 0 0"/>
