Commit message: python xacro parser

File: robots/panda_arm.xacro (robot description, xacro)
@@ -262,6 +262,5 @@
       <axis xyz="0 0 0"/>
     </joint>
-<!-- IMU Placement changes start from here. In kandai's words: aaaaaaaaaaa -->
-    <joint name = "imu_link_joint0" type ="fixed">
+<joint name = "imu_link_joint0" type ="fixed">
       <origin rpy="0 0 0" xyz="0 0 0"/>
       <parent link="${arm_id}_link0"/>
@@ -276,5 +275,5 @@
       </inertial>
       <visual>
-        <origin xyz="0.06 0 0.05" rpy="0 0 0" />
+        <origin xyz="0.06 0.0 0.05" rpy="0 0 0" />
         <geometry>
             <box size = "0.05 0.05 0.05"/>
@@ -295,5 +294,5 @@
         <bodyName>imu_link0</bodyName>
         <gaussianNoise>0.0</gaussianNoise>
-        <xyzOffset>0.06 0 0.05</xyzOffset>
+        <xyzOffset>0.06 0.0 0.05</xyzOffset>
         <rpyOffset>0 0 0</rpyOffset>
         <frameName>imu_link0</frameName>
@@ -302,84 +301,4 @@
     </sensor>
   </gazebo>
-<!--    Joint 0 Axes Start-->
-<!--    IMU 0 X Axis link-->
-  <joint name = "imu_link_joint0_x_axis" type ="fixed">
-      <origin rpy="0 0 0" xyz="0 0 0"/>
-      <parent link="${arm_id}_link0"/>
-      <child link="imu_link0_x_axis"/>
-      <axis xyz="0 0 0"/>
-  </joint>
-  <link name="imu_link0_x_axis">
-      <inertial>
-        <origin xyz="0 0 0" rpy="0 0 0"/>
-        <mass value="0.0"/>
-        <inertia ixx="0.0" ixy="0.0" ixz="0.0" iyy="0.0" iyz="0.0" izz="0.0"/>
-      </inertial>
-      <visual>
-        <origin xyz="0.06 0 0.05" rpy="1.57 0 0" />
-          <geometry>
-            <mesh scale="0.007 0.007 0.007" filename="package://${description_pkg}/meshes/visual/arrow.dae"/>
-<!--            <cylinder length="0.07" radius="0.001"/>-->
-          </geometry>
-        </visual>
-  </link>
-  <gazebo reference="imu_link0_x_axis">
-    <gravity>true</gravity>
-    <material>Gazebo/RedBright</material>
-  </gazebo>
-<!--    End-->
-<!--    IMU 5 Y Axis link-->
-    <joint name = "imu_link_joint0_y_axis" type ="fixed">
-      <origin rpy="0 0 0" xyz="0 0 0"/>
-      <parent link="${arm_id}_link0"/>
-      <child link="imu_link0_y_axis"/>
-      <axis xyz="0 0 0"/>
-  </joint>
-  <link name="imu_link0_y_axis">
-      <inertial>
-        <origin xyz="0 0 0" rpy="0 0 0"/>
-        <mass value="0.0"/>
-        <inertia ixx="0.0" ixy="0.0" ixz="0.0" iyy="0.0" iyz="0.0" izz="0.0"/>
-      </inertial>
-      <visual>
-        <origin xyz="0.06 0 0.05" rpy="0 1.57 0" />
-          <geometry>
-            <mesh scale="0.007 0.007 0.007" filename="package://${description_pkg}/meshes/visual/arrow.dae"/>
-<!--            <cylinder length="0.07" radius="0.001"/>-->
-          </geometry>
-        </visual>
-  </link>
-  <gazebo reference="imu_link0_y_axis">
-    <gravity>true</gravity>
-    <material>Gazebo/Green</material>
-  </gazebo>
-<!--    End-->
-<!--    IMU 5 Z Axis link-->
-  <joint name = "imu_link_joint0_z_axis" type ="fixed">
-      <origin rpy="0 0 0" xyz="0 0 0"/>
-      <parent link="${arm_id}_link0"/>
-      <child link="imu_link0_z_axis"/>
-      <axis xyz="0 0 0"/>
-  </joint>
-  <link name="imu_link0_z_axis">
-      <inertial>
-        <origin xyz="0 0 0" rpy="0 0 0"/>
-        <mass value="0.0"/>
-        <inertia ixx="0.0" ixy="0.0" ixz="0.0" iyy="0.0" iyz="0.0" izz="0.0"/>
-      </inertial>
-      <visual>
-        <origin xyz="0.06 0 0.05" rpy="0 0 1.57" />
-          <geometry>
-<!--            <cylinder length="0.07" radius="0.001"/>-->
-            <mesh scale="0.007 0.007 0.007" filename="package://${description_pkg}/meshes/visual/arrow.dae"/>
-          </geometry>
-        </visual>
-  </link>
-  <gazebo reference="imu_link0_z_axis">
-    <gravity>true</gravity>
-    <material>Gazebo/Blue</material>
-  </gazebo>
-<!--    End-->
-<!--    Joint 0 Axes End-->
 <joint name = "imu_link_joint1" type ="fixed">
       <origin rpy="0 0 0" xyz="0 0 0"/>
@@ -395,9 +314,9 @@
       </inertial>
       <visual>
-        <origin xyz="0.06 0 -.15" rpy="0 0 0" />
-        <geometry>
-            <box size = ".05 .05 .05"/>
-        </geometry>
-        </visual>
+        <origin xyz="0.06 0.0 -0.15" rpy="0 0 0" />
+        <geometry>
+            <box size = "0.05 0.05 0.05"/>
+        </geometry>
+      </visual>
     </link>
     <gazebo reference="imu_link1">
@@ -409,10 +328,10 @@
       <update_rate>10</update_rate>
       <visualize>true</visualize>
-      <topic>imu_data1</topic>
+      <topic>imu_data0</topic>
       <plugin filename="libgazebo_ros_imu_sensor.so" name="imu_plugin">
         <topicName>imu_data1</topicName>
         <bodyName>imu_link1</bodyName>
         <gaussianNoise>0.0</gaussianNoise>
-        <xyzOffset>0.06 0 -.15</xyzOffset>
+        <xyzOffset>0.06 0.0 -0.15</xyzOffset>
         <rpyOffset>0 0 0</rpyOffset>
         <frameName>imu_link1</frameName>
@@ -421,85 +340,5 @@
     </sensor>
   </gazebo>
-    <!--    Joint 1 Axes Start-->
-<!--    IMU 0 X Axis link-->
-  <joint name = "imu_link_joint1_x_axis" type ="fixed">
-      <origin rpy="0 0 0" xyz="0 0 0"/>
-      <parent link="${arm_id}_link1"/>
-      <child link="imu_link1_x_axis"/>
-      <axis xyz="0 0 0"/>
-  </joint>
-  <link name="imu_link1_x_axis">
-      <inertial>
-        <origin xyz="0 0 0" rpy="0 0 0"/>
-        <mass value="0.0"/>
-        <inertia ixx="0.0" ixy="0.0" ixz="0.0" iyy="0.0" iyz="0.0" izz="0.0"/>
-      </inertial>
-      <visual>
-        <origin xyz="0.06 0 -.15" rpy="1.57 0 0" />
-          <geometry>
-            <mesh scale="0.007 0.007 0.007" filename="package://${description_pkg}/meshes/visual/arrow.dae"/>
-<!--            <cylinder length="0.07" radius="0.001"/>-->
-          </geometry>
-        </visual>
-  </link>
-  <gazebo reference="imu_link1_x_axis">
-    <gravity>true</gravity>
-    <material>Gazebo/RedBright</material>
-  </gazebo>
-<!--    End-->
-<!--    IMU 5 Y Axis link-->
-    <joint name = "imu_link_joint1_y_axis" type ="fixed">
-      <origin rpy="0 0 0" xyz="0 0 0"/>
-      <parent link="${arm_id}_link1"/>
-      <child link="imu_link1_y_axis"/>
-      <axis xyz="0 0 0"/>
-  </joint>
-  <link name="imu_link1_y_axis">
-      <inertial>
-        <origin xyz="0 0 0" rpy="0 0 0"/>
-        <mass value="0.0"/>
-        <inertia ixx="0.0" ixy="0.0" ixz="0.0" iyy="0.0" iyz="0.0" izz="0.0"/>
-      </inertial>
-      <visual>
-        <origin xyz="0.06 0 -.15" rpy="0 1.57 0" />
-          <geometry>
-            <mesh scale="0.007 0.007 0.007" filename="package://${description_pkg}/meshes/visual/arrow.dae"/>
-<!--            <cylinder length="0.07" radius="0.001"/>-->
-          </geometry>
-        </visual>
-  </link>
-  <gazebo reference="imu_link1_y_axis">
-    <gravity>true</gravity>
-    <material>Gazebo/Green</material>
-  </gazebo>
-<!--    End-->
-<!--    IMU 5 Z Axis link-->
-  <joint name = "imu_link_joint1_z_axis" type ="fixed">
-      <origin rpy="0 0 0" xyz="0 0 0"/>
-      <parent link="${arm_id}_link1"/>
-      <child link="imu_link1_z_axis"/>
-      <axis xyz="0 0 0"/>
-  </joint>
-  <link name="imu_link1_z_axis">
-      <inertial>
-        <origin xyz="0 0 0" rpy="0 0 0"/>
-        <mass value="0.0"/>
-        <inertia ixx="0.0" ixy="0.0" ixz="0.0" iyy="0.0" iyz="0.0" izz="0.0"/>
-      </inertial>
-      <visual>
-        <origin xyz="0.06 0 -.15" rpy="0 0 1.57" />
-          <geometry>
-<!--            <cylinder length="0.07" radius="0.001"/>-->
-            <mesh scale="0.007 0.007 0.007" filename="package://${description_pkg}/meshes/visual/arrow.dae"/>
-          </geometry>
-        </visual>
-  </link>
-  <gazebo reference="imu_link1_z_axis">
-    <gravity>true</gravity>
-    <material>Gazebo/Blue</material>
-  </gazebo>
-<!--    End-->
-<!--    Joint 1 Axes End-->
-  <joint name = "imu_link_joint2" type ="fixed">
+<joint name = "imu_link_joint2" type ="fixed">
       <origin rpy="0 0 0" xyz="0 0 0"/>
       <parent link="${arm_id}_link2"/>
@@ -514,10 +353,9 @@
       </inertial>
       <visual>
-        <origin xyz="0.06 -.15 0" rpy="0 0 0" />
-<!--        <origin xyz="${props['IMU2_Position_x']}" rpy="0 0 0" />-->
-        <geometry>
-            <box size = ".05 .05 .05"/>
-        </geometry>
-        </visual>
+        <origin xyz="0.06 -0.15 0.0" rpy="0 0 0" />
+        <geometry>
+            <box size = "0.05 0.05 0.05"/>
+        </geometry>
+      </visual>
     </link>
     <gazebo reference="imu_link2">
@@ -529,10 +367,10 @@
       <update_rate>10</update_rate>
       <visualize>true</visualize>
-      <topic>imu_data2</topic>
+      <topic>imu_data0</topic>
       <plugin filename="libgazebo_ros_imu_sensor.so" name="imu_plugin">
         <topicName>imu_data2</topicName>
         <bodyName>imu_link2</bodyName>
         <gaussianNoise>0.0</gaussianNoise>
-        <xyzOffset>0.06 -.15 0</xyzOffset>
+        <xyzOffset>0.06 -0.15 0.0</xyzOffset>
         <rpyOffset>0 0 0</rpyOffset>
         <frameName>imu_link2</frameName>
@@ -541,85 +379,5 @@
     </sensor>
   </gazebo>
-    <!--    Joint 2 Axes Start-->
-<!--    IMU 2 X Axis link-->
-  <joint name = "imu_link_joint2_x_axis" type ="fixed">
-      <origin rpy="0 0 0" xyz="0 0 0"/>
-      <parent link="${arm_id}_link2"/>
-      <child link="imu_link2_x_axis"/>
-      <axis xyz="0 0 0"/>
-  </joint>
-  <link name="imu_link2_x_axis">
-      <inertial>
-        <origin xyz="0 0 0" rpy="0 0 0"/>
-        <mass value="0.0"/>
-        <inertia ixx="0.0" ixy="0.0" ixz="0.0" iyy="0.0" iyz="0.0" izz="0.0"/>
-      </inertial>
-      <visual>
-        <origin xyz="0.06 -.15 0" rpy="1.57 0 0" />
-          <geometry>
-            <mesh scale="0.007 0.007 0.007" filename="package://${description_pkg}/meshes/visual/arrow.dae"/>
-<!--            <cylinder length="0.07" radius="0.001"/>-->
-          </geometry>
-        </visual>
-  </link>
-  <gazebo reference="imu_link2_x_axis">
-    <gravity>true</gravity>
-    <material>Gazebo/RedBright</material>
-  </gazebo>
-<!--    End-->
-<!--    IMU 5 Y Axis link-->
-    <joint name = "imu_link_joint2_y_axis" type ="fixed">
-      <origin rpy="0 0 0" xyz="0 0 0"/>
-      <parent link="${arm_id}_link2"/>
-      <child link="imu_link2_y_axis"/>
-      <axis xyz="0 0 0"/>
-  </joint>
-  <link name="imu_link2_y_axis">
-      <inertial>
-        <origin xyz="0 0 0" rpy="0 0 0"/>
-        <mass value="0.0"/>
-        <inertia ixx="0.0" ixy="0.0" ixz="0.0" iyy="0.0" iyz="0.0" izz="0.0"/>
-      </inertial>
-      <visual>
-        <origin xyz="0.06 -.15 0" rpy="0 1.57 0" />
-          <geometry>
-            <mesh scale="0.007 0.007 0.007" filename="package://${description_pkg}/meshes/visual/arrow.dae"/>
-<!--            <cylinder length="0.07" radius="0.001"/>-->
-          </geometry>
-        </visual>
-  </link>
-  <gazebo reference="imu_link2_y_axis">
-    <gravity>true</gravity>
-    <material>Gazebo/Green</material>
-  </gazebo>
-<!--    End-->
-<!--    IMU 5 Z Axis link-->
-  <joint name = "imu_link_joint2_z_axis" type ="fixed">
-      <origin rpy="0 0 0" xyz="0 0 0"/>
-      <parent link="${arm_id}_link2"/>
-      <child link="imu_link2_z_axis"/>
-      <axis xyz="0 0 0"/>
-  </joint>
-  <link name="imu_link2_z_axis">
-      <inertial>
-        <origin xyz="0 0 0" rpy="0 0 0"/>
-        <mass value="0.0"/>
-        <inertia ixx="0.0" ixy="0.0" ixz="0.0" iyy="0.0" iyz="0.0" izz="0.0"/>
-      </inertial>
-      <visual>
-        <origin xyz="0.06 -.15 0" rpy="0 0 1.57" />
-          <geometry>
-<!--            <cylinder length="0.07" radius="0.001"/>-->
-            <mesh scale="0.007 0.007 0.007" filename="package://${description_pkg}/meshes/visual/arrow.dae"/>
-          </geometry>
-        </visual>
-  </link>
-  <gazebo reference="imu_link2_z_axis">
-    <gravity>true</gravity>
-    <material>Gazebo/Blue</material>
-  </gazebo>
-<!--    End-->
-<!--    Joint 2 Axes End-->
-  <joint name = "imu_link_joint3" type ="fixed">
+<joint name = "imu_link_joint3" type ="fixed">
       <origin rpy="0 0 0" xyz="0 0 0"/>
       <parent link="${arm_id}_link3"/>
@@ -634,9 +392,9 @@
       </inertial>
       <visual>
-        <origin xyz="-0.06 0 -0.06" rpy="0 0 0" />
-        <geometry>
-            <box size = ".05 .05 .05"/>
-        </geometry>
-        </visual>
+        <origin xyz="-0.06 0.0 -0.06" rpy="0 0 0" />
+        <geometry>
+            <box size = "0.05 0.05 0.05"/>
+        </geometry>
+      </visual>
     </link>
     <gazebo reference="imu_link3">
@@ -648,10 +406,10 @@
       <update_rate>10</update_rate>
       <visualize>true</visualize>
-      <topic>imu_data3</topic>
+      <topic>imu_data0</topic>
       <plugin filename="libgazebo_ros_imu_sensor.so" name="imu_plugin">
         <topicName>imu_data3</topicName>
         <bodyName>imu_link3</bodyName>
         <gaussianNoise>0.0</gaussianNoise>
-        <xyzOffset>-0.06 0 -0.06</xyzOffset>
+        <xyzOffset>-0.06 0.0 -0.06</xyzOffset>
         <rpyOffset>0 0 0</rpyOffset>
         <frameName>imu_link3</frameName>
@@ -660,5 +418,5 @@
     </sensor>
   </gazebo>
-  <joint name = "imu_link_joint4" type ="fixed">
+<joint name = "imu_link_joint4" type ="fixed">
       <origin rpy="0 0 0" xyz="0 0 0"/>
       <parent link="${arm_id}_link4"/>
@@ -673,9 +431,9 @@
       </inertial>
       <visual>
-        <origin xyz="-0.14 0.09 0" rpy="0 0 0" />
-        <geometry>
-            <box size = ".05 .05 .05"/>
-        </geometry>
-        </visual>
+        <origin xyz="-0.14 0.09 0.0" rpy="0 0 0" />
+        <geometry>
+            <box size = "0.05 0.05 0.05"/>
+        </geometry>
+      </visual>
     </link>
     <gazebo reference="imu_link4">
@@ -687,10 +445,10 @@
       <update_rate>10</update_rate>
       <visualize>true</visualize>
-      <topic>imu_data4</topic>
+      <topic>imu_data0</topic>
       <plugin filename="libgazebo_ros_imu_sensor.so" name="imu_plugin">
         <topicName>imu_data4</topicName>
         <bodyName>imu_link4</bodyName>
         <gaussianNoise>0.0</gaussianNoise>
-        <xyzOffset>-0.14 0.09 0</xyzOffset>
+        <xyzOffset>-0.14 0.09 0.0</xyzOffset>
         <rpyOffset>0 0 0</rpyOffset>
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