Commit message: Final PR

File: robots/panda_arm.xacro (robot description, xacro)
@@ -548,5 +548,5 @@
       </inertial>
       <visual>
-        <origin xyz="1.06 0.0 0.05" rpy="0 0 0" />
+        <origin xyz="0.56 0.0 0.05" rpy="0 0 0" />
         <geometry>
             <box size = "0.05 0.05 0.05"/>
@@ -567,5 +567,5 @@
         <bodyName>simulated_imu_link0</bodyName>
         <gaussianNoise>0.0</gaussianNoise>
-        <xyzOffset>1.06 0.0 0.05</xyzOffset>
+        <xyzOffset>0.56 0.0 0.05</xyzOffset>
         <rpyOffset>0 0 0</rpyOffset>
         <frameName>simulated_imu_link0</frameName>
@@ -587,5 +587,5 @@
       </inertial>
       <visual>
-        <origin xyz="1.06 0.0 -0.15" rpy="0 0 0" />
+        <origin xyz="0.56 0.0 -0.15" rpy="0 0 0" />
         <geometry>
             <box size = "0.05 0.05 0.05"/>
@@ -606,5 +606,5 @@
         <bodyName>simulated_imu_link1</bodyName>
         <gaussianNoise>0.0</gaussianNoise>
-        <xyzOffset>1.06 0.0 -0.15</xyzOffset>
+        <xyzOffset>0.56 0.0 -0.15</xyzOffset>
         <rpyOffset>0 0 0</rpyOffset>
         <frameName>simulated_imu_link1</frameName>
@@ -626,5 +626,5 @@
       </inertial>
       <visual>
-        <origin xyz="1.06 -0.15 0.0" rpy="0 0 0" />
+        <origin xyz="0.56 -0.15 0.0" rpy="0 0 0" />
         <geometry>
             <box size = "0.05 0.05 0.05"/>
@@ -645,5 +645,5 @@
         <bodyName>simulated_imu_link2</bodyName>
         <gaussianNoise>0.0</gaussianNoise>
-        <xyzOffset>1.06 -0.15 0.0</xyzOffset>
+        <xyzOffset>0.56 -0.15 0.0</xyzOffset>
         <rpyOffset>0 0 0</rpyOffset>
         <frameName>simulated_imu_link2</frameName>
@@ -665,5 +665,5 @@
       </inertial>
       <visual>
-        <origin xyz="0.94 0.0 -0.06" rpy="0 0 0" />
+        <origin xyz="0.44 0.0 -0.06" rpy="0 0 0" />
         <geometry>
             <box size = "0.05 0.05 0.05"/>
@@ -684,5 +684,5 @@
         <bodyName>simulated_imu_link3</bodyName>
         <gaussianNoise>0.0</gaussianNoise>
-        <xyzOffset>0.94 0.0 -0.06</xyzOffset>
+        <xyzOffset>0.44 0.0 -0.06</xyzOffset>
         <rpyOffset>0 0 0</rpyOffset>
         <frameName>simulated_imu_link3</frameName>
@@ -704,5 +704,5 @@
       </inertial>
       <visual>
-        <origin xyz="0.86 0.09 0.0" rpy="0 0 0" />
+        <origin xyz="0.36 0.09 0.0" rpy="0 0 0" />
         <geometry>
             <box size = "0.05 0.05 0.05"/>
@@ -723,5 +723,5 @@
         <bodyName>simulated_imu_link4</bodyName>
         <gaussianNoise>0.0</gaussianNoise>
-        <xyzOffset>0.86 0.09 0.0</xyzOffset>
+        <xyzOffset>0.36 0.09 0.0</xyzOffset>
         <rpyOffset>0 0 0</rpyOffset>
         <frameName>simulated_imu_link4</frameName>
@@ -743,5 +743,5 @@
       </inertial>
       <visual>
-        <origin xyz="1.0 0.1 -0.11" rpy="0 0 0" />
+        <origin xyz="0.5 0.1 -0.11" rpy="0 0 0" />
         <geometry>
             <box size = "0.05 0.05 0.05"/>
@@ -762,5 +762,5 @@
         <bodyName>simulated_imu_link5</bodyName>
         <gaussianNoise>0.0</gaussianNoise>
-        <xyzOffset>1.0 0.1 -0.11</xyzOffset>
+        <xyzOffset>0.5 0.1 -0.11</xyzOffset>
         <rpyOffset>0 0 0</rpyOffset>
         <frameName>simulated_imu_link5</frameName>
@@ -782,5 +782,5 @@
       </inertial>
       <visual>
-        <origin xyz="1.13 0.02 0.0" rpy="0 0 0" />
+        <origin xyz="0.63 0.02 0.0" rpy="0 0 0" />
         <geometry>
             <box size = "0.05 0.05 0.05"/>
@@ -801,5 +801,5 @@
         <bodyName>simulated_imu_link6</bodyName>
         <gaussianNoise>0.0</gaussianNoise>
-        <xyzOffset>1.13 0.02 0.0</xyzOffset>
+        <xyzOffset>0.63 0.02 0.0</xyzOffset>
         <rpyOffset>0 0 0</rpyOffset>
         <frameName>simulated_imu_link6</frameName>
@@ -1304,5 +1304,5 @@
       </inertial>
       <visual>
-        <origin xyz="1.06 0.0 0.05" rpy="1 0 0" />
+        <origin xyz="0.56 0.0 0.05" rpy="1 0 0" />
           <geometry>
             <mesh scale="0.007 0.007 0.007" filename="package://${description_pkg}/meshes/visual/arrow.dae"/>
@@ -1327,5 +1327,5 @@
       </inertial>
       <visual>
-        <origin xyz="1.06 0.0 0.05" rpy="0 1 0" />
+        <origin xyz="0.56 0.0 0.05" rpy="0 1 0" />
           <geometry>
             <mesh scale="0.007 0.007 0.007" filename="package://${description_pkg}/meshes/visual/arrow.dae"/>
@@ -1350,5 +1350,5 @@
       </inertial>
       <visual>
-        <origin xyz="1.06 0.0 0.05" rpy="0 0 1" />
+        <origin xyz="0.56 0.0 0.05" rpy="0 0 1" />
           <geometry>
             <mesh scale="0.007 0.007 0.007" filename="package://${description_pkg}/meshes/visual/arrow.dae"/>
@@ -1373,5 +1373,5 @@
       </inertial>
       <visual>
-        <origin xyz="1.06 0.0 -0.15" rpy="1 0 0" />
+        <origin xyz="0.56 0.0 -0.15" rpy="1 0 0" />
           <geometry>
             <mesh scale="0.007 0.007 0.007" filename="package://${description_pkg}/meshes/visual/arrow.dae"/>
@@ -1396,5 +1396,5 @@
       </inertial>
       <visual>
-        <origin xyz="1.06 0.0 -0.15" rpy="0 1 0" />
+        <origin xyz="0.56 0.0 -0.15" rpy="0 1 0" />
           <geometry>
             <mesh scale="0.007 0.007 0.007" filename="package://${description_pkg}/meshes/visual/arrow.dae"/>
@@ -1419,5 +1419,5 @@
       </inertial>
       <visual>
-        <origin xyz="1.06 0.0 -0.15" rpy="0 0 1" />
+        <origin xyz="0.56 0.0 -0.15" rpy="0 0 1" />
           <geometry>
             <mesh scale="0.007 0.007 0.007" filename="package://${description_pkg}/meshes/visual/arrow.dae"/>
@@ -1442,5 +1442,5 @@
       </inertial>
       <visual>
-        <origin xyz="1.06 -0.15 0.0" rpy="1 0 0" />
+        <origin xyz="0.56 -0.15 0.0" rpy="1 0 0" />
           <geometry>
             <mesh scale="0.007 0.007 0.007" filename="package://${description_pkg}/meshes/visual/arrow.dae"/>
@@ -1465,5 +1465,5 @@
       </inertial>
       <visual>
-        <origin xyz="1.06 -0.15 0.0" rpy="0 1 0" />
+        <origin xyz="0.56 -0.15 0.0" rpy="0 1 0" />
           <geometry>
             <mesh scale="0.007 0.007 0.007" filename="package://${description_pkg}/meshes/visual/arrow.dae"/>
@@ -1488,5 +1488,5 @@
       </inertial>
       <visual>
-        <origin xyz="1.06 -0.15 0.0" rpy="0 0 1" />
+        <origin xyz="0.56 -0.15 0.0" rpy="0 0 1" />
           <geometry>
             <mesh scale="0.007 0.007 0.007" filename="package://${description_pkg}/meshes/visual/arrow.dae"/>
@@ -1511,5 +1511,5 @@
       </inertial>
       <visual>
-        <origin xyz="0.94 0.0 -0.06" rpy="1 0 0" />
+        <origin xyz="0.44 0.0 -0.06" rpy="1 0 0" />
           <geometry>
             <mesh scale="0.007 0.007 0.007" filename="package://${description_pkg}/meshes/visual/arrow.dae"/>
@@ -1534,5 +1534,5 @@
       </inertial>
       <visual>
-        <origin xyz="0.94 0.0 -0.06" rpy="0 1 0" />
+        <origin xyz="0.44 0.0 -0.06" rpy="0 1 0" />
           <geometry>
             <mesh scale="0.007 0.007 0.007" filename="package://${description_pkg}/meshes/visual/arrow.dae"/>
@@ -1557,5 +1557,5 @@
       </inertial>
       <visual>
-        <origin xyz="0.94 0.0 -0.06" rpy="0 0 1" />
+        <origin xyz="0.44 0.0 -0.06" rpy="0 0 1" />
           <geometry>
             <mesh scale="0.007 0.007 0.007" filename="package://${description_pkg}/meshes/visual/arrow.dae"/>
@@ -1580,5 +1580,5 @@
       </inertial>
       <visual>
-        <origin xyz="0.86 0.09 0.0" rpy="1 0 0" />
+        <origin xyz="0.36 0.09 0.0" rpy="1 0 0" />
           <geometry>
             <mesh scale="0.007 0.007 0.007" filename="package://${description_pkg}/meshes/visual/arrow.dae"/>
@@ -1603,5 +1603,5 @@
       </inertial>
       <visual>
-        <origin xyz="0.86 0.09 0.0" rpy="0 1 0" />
+        <origin xyz="0.36 0.09 0.0" rpy="0 1 0" />
           <geometry>
             <mesh scale="0.007 0.007 0.007" filename="package://${description_pkg}/meshes/visual/arrow.dae"/>
@@ -1626,5 +1626,5 @@
       </inertial>
       <visual>
-        <origin xyz="0.86 0.09 0.0" rpy="0 0 1" />
+        <origin xyz="0.36 0.09 0.0" rpy="0 0 1" />
           <geometry>
             <mesh scale="0.007 0.007 0.007" filename="package://${description_pkg}/meshes/visual/arrow.dae"/>
@@ -1649,5 +1649,5 @@
       </inertial>
       <visual>
-        <origin xyz="1.0 0.1 -0.11" rpy="1 0 0" />
+        <origin xyz="0.5 0.1 -0.11" rpy="1 0 0" />
           <geometry>
             <mesh scale="0.007 0.007 0.007" filename="package://${description_pkg}/meshes/visual/arrow.dae"/>
@@ -1672,5 +1672,5 @@
       </inertial>
       <visual>
-        <origin xyz="1.0 0.1 -0.11" rpy="0 1 0" />
+        <origin xyz="0.5 0.1 -0.11" rpy="0 1 0" />
           <geometry>
             <mesh scale="0.007 0.007 0.007" filename="package://${description_pkg}/meshes/visual/arrow.dae"/>
@@ -1695,5 +1695,5 @@
       </inertial>
       <visual>
-        <origin xyz="1.0 0.1 -0.11" rpy="0 0 1" />
+        <origin xyz="0.5 0.1 -0.11" rpy="0 0 1" />
           <geometry>
             <mesh scale="0.007 0.007 0.007" filename="package://${description_pkg}/meshes/visual/arrow.dae"/>
@@ -1718,5 +1718,5 @@
       </inertial>
       <visual>
-        <origin xyz="1.13 0.02 0.0" rpy="1 0 0" />
+        <origin xyz="0.63 0.02 0.0" rpy="1 0 0" />
           <geometry>
             <mesh scale="0.007 0.007 0.007" filename="package://${description_pkg}/meshes/visual/arrow.dae"/>
@@ -1741,5 +1741,5 @@
       </inertial>
       <visual>
-        <origin xyz="1.13 0.02 0.0" rpy="0 1 0" />
+        <origin xyz="0.63 0.02 0.0" rpy="0 1 0" />
           <geometry>
             <mesh scale="0.007 0.007 0.007" filename="package://${description_pkg}/meshes/visual/arrow.dae"/>
@@ -1764,5 +1764,5 @@
       </inertial>
       <visual>
-        <origin xyz="1.13 0.02 0.0" rpy="0 0 1" />
+        <origin xyz="0.63 0.02 0.0" rpy="0 0 1" />
           <geometry>
             <mesh scale="0.007 0.007 0.007" filename="package://${description_pkg}/meshes/visual/arrow.dae"/>

Commit message: Pushing some final changes

File: robots/panda_arm.xacro (robot description, xacro)
@@ -1,5 +1,5 @@
 <?xml version='1.0' encoding='utf-8'?>
 <robot xmlns:xacro="http://www.ros.org/wiki/xacro" name="panda">
-  <xacro:macro name="panda_arm" params="arm_id:='panda' description_pkg:='franka_description' connected_to:='' xyz:='0 0 0' rpy:='0 0 0'">
+  <xacro:macro name="panda_arm" params="arm_id:='panda' description_pkg:='franka_description' axes_meshes:='ros_robotic_skin' connected_to:='' xyz:='0 0 0' rpy:='0 0 0'">
     <xacro:unless value="${not connected_to}">
       <joint name="${arm_id}_joint_${connected_to}" type="fixed">
@@ -823,5 +823,5 @@
         <origin xyz="0.06 0.0 0.05" rpy="1 0 0" />
           <geometry>
-            <mesh scale="0.007 0.007 0.007" filename="package://${description_pkg}/meshes/visual/arrow.dae"/>
+            <mesh scale="0.007 0.007 0.007" filename="package://${axes_meshes}/axes_meshes/meshes/visual/arrow.dae"/>
           </geometry>
         </visual>
@@ -892,5 +892,5 @@
         <origin xyz="0.06 0.0 -0.15" rpy="1 0 0" />
           <geometry>
-            <mesh scale="0.007 0.007 0.007" filename="package://${description_pkg}/meshes/visual/arrow.dae"/>
+            <mesh scale="0.007 0.007 0.007" filename="package://${axes_meshes}/axes_meshes/meshes/visual/arrow.dae"/>
           </geometry>
         </visual>
@@ -961,5 +961,5 @@
         <origin xyz="0.06 -0.15 0.0" rpy="1 0 0" />
           <geometry>
-            <mesh scale="0.007 0.007 0.007" filename="package://${description_pkg}/meshes/visual/arrow.dae"/>
+            <mesh scale="0.007 0.007 0.007" filename="package://${axes_meshes}/axes_meshes/meshes/visual/arrow.dae"/>
           </geometry>
         </visual>
@@ -1030,5 +1030,5 @@
         <origin xyz="-0.06 0.0 -0.06" rpy="1 0 0" />
           <geometry>
-            <mesh scale="0.007 0.007 0.007" filename="package://${description_pkg}/meshes/visual/arrow.dae"/>
+            <mesh scale="0.007 0.007 0.007" filename="package://${axes_meshes}/axes_meshes/meshes/visual/arrow.dae"/>
           </geometry>
         </visual>
@@ -1099,5 +1099,5 @@
         <origin xyz="-0.14 0.09 0.0" rpy="1 0 0" />
           <geometry>
-            <mesh scale="0.007 0.007 0.007" filename="package://${description_pkg}/meshes/visual/arrow.dae"/>
+            <mesh scale="0.007 0.007 0.007" filename="package://${axes_meshes}/axes_meshes/meshes/visual/arrow.dae"/>
           </geometry>
         </visual>
@@ -1168,5 +1168,5 @@
         <origin xyz="0.0 0.1 -0.11" rpy="1 0 0" />
           <geometry>
-            <mesh scale="0.007 0.007 0.007" filename="package://${description_pkg}/meshes/visual/arrow.dae"/>
+            <mesh scale="0.007 0.007 0.007" filename="package://${axes_meshes}/axes_meshes/meshes/visual/arrow.dae"/>
           </geometry>
         </visual>
@@ -1237,5 +1237,5 @@
         <origin xyz="0.13 0.02 0.0" rpy="1 0 0" />
           <geometry>
-            <mesh scale="0.007 0.007 0.007" filename="package://${description_pkg}/meshes/visual/arrow.dae"/>
+            <mesh scale="0.007 0.007 0.007" filename="package://${axes_meshes}/axes_meshes/meshes/visual/arrow.dae"/>
           </geometry>
         </visual>
@@ -1306,5 +1306,5 @@
         <origin xyz="0.56 0.0 0.05" rpy="1 0 0" />
           <geometry>
-            <mesh scale="0.007 0.007 0.007" filename="package://${description_pkg}/meshes/visual/arrow.dae"/>
+            <mesh scale="0.007 0.007 0.007" filename="package://${axes_meshes}/axes_meshes/meshes/visual/arrow.dae"/>
           </geometry>
         </visual>
@@ -1375,5 +1375,5 @@
         <origin xyz="0.56 0.0 -0.15" rpy="1 0 0" />
           <geometry>
-            <mesh scale="0.007 0.007 0.007" filename="package://${description_pkg}/meshes/visual/arrow.dae"/>
+            <mesh scale="0.007 0.007 0.007" filename="package://${axes_meshes}/axes_meshes/meshes/visual/arrow.dae"/>
           </geometry>
         </visual>
@@ -1444,5 +1444,5 @@
         <origin xyz="0.56 -0.15 0.0" rpy="1 0 0" />
           <geometry>
-            <mesh scale="0.007 0.007 0.007" filename="package://${description_pkg}/meshes/visual/arrow.dae"/>
+            <mesh scale="0.007 0.007 0.007" filename="package://${axes_meshes}/axes_meshes/meshes/visual/arrow.dae"/>
           </geometry>
         </visual>
@@ -1513,5 +1513,5 @@
         <origin xyz="0.44 0.0 -0.06" rpy="1 0 0" />
           <geometry>
-            <mesh scale="0.007 0.007 0.007" filename="package://${description_pkg}/meshes/visual/arrow.dae"/>
+            <mesh scale="0.007 0.007 0.007" filename="package://${axes_meshes}/axes_meshes/meshes/visual/arrow.dae"/>
           </geometry>
         </visual>
@@ -1582,5 +1582,5 @@
         <origin xyz="0.36 0.09 0.0" rpy="1 0 0" />
           <geometry>
-            <mesh scale="0.007 0.007 0.007" filename="package://${description_pkg}/meshes/visual/arrow.dae"/>
+            <mesh scale="0.007 0.007 0.007" filename="package://${axes_meshes}/axes_meshes/meshes/visual/arrow.dae"/>
           </geometry>
         </visual>
@@ -1651,5 +1651,5 @@
         <origin xyz="0.5 0.1 -0.11" rpy="1 0 0" />
           <geometry>
-            <mesh scale="0.007 0.007 0.007" filename="package://${description_pkg}/meshes/visual/arrow.dae"/>
+            <mesh scale="0.007 0.007 0.007" filename="package://${axes_meshes}/axes_meshes/meshes/visual/arrow.dae"/>
           </geometry>
         </visual>
@@ -1720,5 +1720,5 @@
         <origin xyz="0.63 0.02 0.0" rpy="1 0 0" />
           <geometry>
-            <mesh scale="0.007 0.007 0.007" filename="package://${description_pkg}/meshes/visual/arrow.dae"/>
+            <mesh scale="0.007 0.007 0.007" filename="package://${axes_meshes}/axes_meshes/meshes/visual/arrow.dae"/>
           </geometry>
         </visual>

File: robots/panda_arm_reference.xacro (robot description, xacro)
@@ -1,5 +1,5 @@
 <?xml version='1.0' encoding='utf-8'?>
 <robot xmlns:xacro="http://www.ros.org/wiki/xacro" name="panda">
-  <xacro:macro name="panda_arm" params="arm_id:='panda' description_pkg:='franka_description' connected_to:='' xyz:='0 0 0' rpy:='0 0 0'">
+  <xacro:macro name="panda_arm" params="arm_id:='panda' description_pkg:='franka_description' axes_meshes:='ros_robotic_skin' connected_to:='' xyz:='0 0 0' rpy:='0 0 0'">
     <xacro:unless value="${not connected_to}">
       <joint name="${arm_id}_joint_${connected_to}" type="fixed">
