Commit message: Make indentation perfect!

File: robots/panda_arm.xacro (robot description, xacro)
@@ -267,19 +267,19 @@
       <child link="imu_link0"/>
       <axis xyz="0 0 0"/>
-    </joint>
-    <link name="imu_link0">
-      <inertial>
+</joint>
+<link name="imu_link0">
+    <inertial>
         <origin xyz="0 0 0" rpy="0 0 0"/>
         <mass value="0.0"/>
         <inertia ixx="0.0" ixy="0.0" ixz="0.0" iyy="0.0" iyz="0.0" izz="0.0"/>
-      </inertial>
-      <visual>
+    </inertial>
+    <visual>
         <origin xyz="0.06 0.0 0.05" rpy="0 0 0" />
         <geometry>
             <box size = "0.05 0.05 0.05"/>
         </geometry>
-      </visual>
-    </link>
-    <gazebo reference="imu_link0">
+    </visual>
+</link>
+<gazebo reference="imu_link0">
     <gravity>true</gravity>
     <!--      Below is the line to change the material-->
@@ -300,5 +300,5 @@
       <pose>0 0 0 0 0 0</pose>
     </sensor>
-  </gazebo>
+</gazebo>
 <joint name = "imu_link_joint1" type ="fixed">
       <origin rpy="0 0 0" xyz="0 0 0"/>
@@ -306,19 +306,19 @@
       <child link="imu_link1"/>
       <axis xyz="0 0 0"/>
-    </joint>
-    <link name="imu_link1">
-      <inertial>
+</joint>
+<link name="imu_link1">
+    <inertial>
         <origin xyz="0 0 0" rpy="0 0 0"/>
         <mass value="0.0"/>
         <inertia ixx="0.0" ixy="0.0" ixz="0.0" iyy="0.0" iyz="0.0" izz="0.0"/>
-      </inertial>
-      <visual>
+    </inertial>
+    <visual>
         <origin xyz="0.06 0.0 -0.15" rpy="0 0 0" />
         <geometry>
             <box size = "0.05 0.05 0.05"/>
         </geometry>
-      </visual>
-    </link>
-    <gazebo reference="imu_link1">
+    </visual>
+</link>
+<gazebo reference="imu_link1">
     <gravity>true</gravity>
     <!--      Below is the line to change the material-->
@@ -339,5 +339,5 @@
       <pose>0 0 0 0 0 0</pose>
     </sensor>
-  </gazebo>
+</gazebo>
 <joint name = "imu_link_joint2" type ="fixed">
       <origin rpy="0 0 0" xyz="0 0 0"/>
@@ -345,19 +345,19 @@
       <child link="imu_link2"/>
       <axis xyz="0 0 0"/>
-    </joint>
-    <link name="imu_link2">
-      <inertial>
+</joint>
+<link name="imu_link2">
+    <inertial>
         <origin xyz="0 0 0" rpy="0 0 0"/>
         <mass value="0.0"/>
         <inertia ixx="0.0" ixy="0.0" ixz="0.0" iyy="0.0" iyz="0.0" izz="0.0"/>
-      </inertial>
-      <visual>
+    </inertial>
+    <visual>
         <origin xyz="0.06 -0.15 0.0" rpy="0 0 0" />
         <geometry>
             <box size = "0.05 0.05 0.05"/>
         </geometry>
-      </visual>
-    </link>
-    <gazebo reference="imu_link2">
+    </visual>
+</link>
+<gazebo reference="imu_link2">
     <gravity>true</gravity>
     <!--      Below is the line to change the material-->
@@ -378,5 +378,5 @@
       <pose>0 0 0 0 0 0</pose>
     </sensor>
-  </gazebo>
+</gazebo>
 <joint name = "imu_link_joint3" type ="fixed">
       <origin rpy="0 0 0" xyz="0 0 0"/>
@@ -384,19 +384,19 @@
       <child link="imu_link3"/>
       <axis xyz="0 0 0"/>
-    </joint>
-    <link name="imu_link3">
-      <inertial>
+</joint>
+<link name="imu_link3">
+    <inertial>
         <origin xyz="0 0 0" rpy="0 0 0"/>
         <mass value="0.0"/>
         <inertia ixx="0.0" ixy="0.0" ixz="0.0" iyy="0.0" iyz="0.0" izz="0.0"/>
-      </inertial>
-      <visual>
+    </inertial>
+    <visual>
         <origin xyz="-0.06 0.0 -0.06" rpy="0 0 0" />
         <geometry>
             <box size = "0.05 0.05 0.05"/>
         </geometry>
-      </visual>
-    </link>
-    <gazebo reference="imu_link3">
+    </visual>
+</link>
+<gazebo reference="imu_link3">
     <gravity>true</gravity>
     <!--      Below is the line to change the material-->
@@ -417,5 +417,5 @@
       <pose>0 0 0 0 0 0</pose>
     </sensor>
-  </gazebo>
+</gazebo>
 <joint name = "imu_link_joint4" type ="fixed">
       <origin rpy="0 0 0" xyz="0 0 0"/>
@@ -423,19 +423,19 @@
       <child link="imu_link4"/>
       <axis xyz="0 0 0"/>
-    </joint>
-    <link name="imu_link4">
-      <inertial>
+</joint>
+<link name="imu_link4">
+    <inertial>
         <origin xyz="0 0 0" rpy="0 0 0"/>
         <mass value="0.0"/>
         <inertia ixx="0.0" ixy="0.0" ixz="0.0" iyy="0.0" iyz="0.0" izz="0.0"/>
-      </inertial>
-      <visual>
+    </inertial>
+    <visual>
         <origin xyz="-0.14 0.09 0.0" rpy="0 0 0" />
         <geometry>
             <box size = "0.05 0.05 0.05"/>
         </geometry>
-      </visual>
-    </link>
-    <gazebo reference="imu_link4">
+    </visual>
+</link>
+<gazebo reference="imu_link4">
     <gravity>true</gravity>
     <!--      Below is the line to change the material-->
@@ -456,5 +456,5 @@
       <pose>0 0 0 0 0 0</pose>
     </sensor>
-  </gazebo>
+</gazebo>
 <joint name = "imu_link_joint5" type ="fixed">
       <origin rpy="0 0 0" xyz="0 0 0"/>
@@ -462,19 +462,19 @@
       <child link="imu_link5"/>
       <axis xyz="0 0 0"/>
-    </joint>
-    <link name="imu_link5">
-      <inertial>
+</joint>
+<link name="imu_link5">
+    <inertial>
         <origin xyz="0 0 0" rpy="0 0 0"/>
         <mass value="0.0"/>
         <inertia ixx="0.0" ixy="0.0" ixz="0.0" iyy="0.0" iyz="0.0" izz="0.0"/>
-      </inertial>
-      <visual>
+    </inertial>
+    <visual>
         <origin xyz="0.0 0.1 -0.11" rpy="0 0 0" />
         <geometry>
             <box size = "0.05 0.05 0.05"/>
         </geometry>
-      </visual>
-    </link>
-    <gazebo reference="imu_link5">
+    </visual>
+</link>
+<gazebo reference="imu_link5">
     <gravity>true</gravity>
     <!--      Below is the line to change the material-->
@@ -495,5 +495,5 @@
       <pose>0 0 0 0 0 0</pose>
     </sensor>
-  </gazebo>
+</gazebo>
 <joint name = "imu_link_joint6" type ="fixed">
       <origin rpy="0 0 0" xyz="0 0 0"/>
@@ -501,19 +501,19 @@
       <child link="imu_link6"/>
       <axis xyz="0 0 0"/>
-    </joint>
-    <link name="imu_link6">
-      <inertial>
+</joint>
+<link name="imu_link6">
+    <inertial>
         <origin xyz="0 0 0" rpy="0 0 0"/>
         <mass value="0.0"/>
         <inertia ixx="0.0" ixy="0.0" ixz="0.0" iyy="0.0" iyz="0.0" izz="0.0"/>
-      </inertial>
-      <visual>
+    </inertial>
+    <visual>
         <origin xyz="0.13 0.02 0.0" rpy="0 0 0" />
         <geometry>
             <box size = "0.05 0.05 0.05"/>
         </geometry>
-      </visual>
-    </link>
-    <gazebo reference="imu_link6">
+    </visual>
+</link>
+<gazebo reference="imu_link6">
     <gravity>true</gravity>
     <!--      Below is the line to change the material-->
@@ -534,5 +534,5 @@
       <pose>0 0 0 0 0 0</pose>
     </sensor>
-  </gazebo>
+</gazebo>
 <joint name = "simulated_imu_link_joint0" type ="fixed">
       <origin rpy="0 0 0" xyz="0 0 0"/>
@@ -540,19 +540,19 @@
       <child link="simulated_imu_link0"/>
       <axis xyz="0 0 0"/>
-    </joint>
-    <link name="simulated_imu_link0">
-      <inertial>
+</joint>
+<link name="simulated_imu_link0">
+    <inertial>
         <origin xyz="0 0 0" rpy="0 0 0"/>
         <mass value="0.0"/>
         <inertia ixx="0.0" ixy="0.0" ixz="0.0" iyy="0.0" iyz="0.0" izz="0.0"/>
-      </inertial>
-      <visual>
+    </inertial>
+    <visual>
         <origin xyz="0.56 0.0 0.05" rpy="0 0 0" />
         <geometry>
             <box size = "0.05 0.05 0.05"/>
         </geometry>
-      </visual>
-    </link>
-    <gazebo reference="simulated_imu_link0">
+    </visual>
+</link>
+<gazebo reference="simulated_imu_link0">
     <gravity>true</gravity>
     <!--      Below is the line to change the material-->
@@ -573,5 +573,5 @@
       <pose>0 0 0 0 0 0</pose>
     </sensor>
-  </gazebo>
+</gazebo>
 <joint name = "simulated_imu_link_joint1" type ="fixed">
       <origin rpy="0 0 0" xyz="0 0 0"/>
@@ -579,19 +579,19 @@
       <child link="simulated_imu_link1"/>
       <axis xyz="0 0 0"/>
-    </joint>
-    <link name="simulated_imu_link1">
-      <inertial>
+</joint>
+<link name="simulated_imu_link1">
+    <inertial>
         <origin xyz="0 0 0" rpy="0 0 0"/>
         <mass value="0.0"/>
         <inertia ixx="0.0" ixy="0.0" ixz="0.0" iyy="0.0" iyz="0.0" izz="0.0"/>
-      </inertial>
-      <visual>
+    </inertial>
+    <visual>
         <origin xyz="0.56 0.0 -0.15" rpy="0 0 0" />
         <geometry>
             <box size = "0.05 0.05 0.05"/>
         </geometry>
-      </visual>
-    </link>
-    <gazebo reference="simulated_imu_link1">
+    </visual>
+</link>
+<gazebo reference="simulated_imu_link1">
     <gravity>true</gravity>
     <!--      Below is the line to change the material-->
@@ -612,5 +612,5 @@
       <pose>0 0 0 0 0 0</pose>
     </sensor>
-  </gazebo>
+</gazebo>
 <joint name = "simulated_imu_link_joint2" type ="fixed">
       <origin rpy="0 0 0" xyz="0 0 0"/>
@@ -618,19 +618,19 @@
       <child link="simulated_imu_link2"/>
       <axis xyz="0 0 0"/>
-    </joint>
-    <link name="simulated_imu_link2">
-      <inertial>
+</joint>
+<link name="simulated_imu_link2">
+    <inertial>
         <origin xyz="0 0 0" rpy="0 0 0"/>
         <mass value="0.0"/>
         <inertia ixx="0.0" ixy="0.0" ixz="0.0" iyy="0.0" iyz="0.0" izz="0.0"/>
-      </inertial>
-      <visual>
+    </inertial>
+    <visual>
         <origin xyz="0.56 -0.15 0.0" rpy="0 0 0" />
         <geometry>
             <box size = "0.05 0.05 0.05"/>
         </geometry>
-      </visual>
-    </link>
-    <gazebo reference="simulated_imu_link2">
+    </visual>
+</link>
+<gazebo reference="simulated_imu_link2">
     <gravity>true</gravity>
     <!--      Below is the line to change the material-->
@@ -651,5 +651,5 @@
       <pose>0 0 0 0 0 0</pose>
     </sensor>
-  </gazebo>
+</gazebo>
 <joint name = "simulated_imu_link_joint3" type ="fixed">
       <origin rpy="0 0 0" xyz="0 0 0"/>
@@ -657,19 +657,19 @@
       <child link="simulated_imu_link3"/>
       <axis xyz="0 0 0"/>
-    </joint>
-    <link name="simulated_imu_link3">
-      <inertial>
+</joint>
+<link name="simulated_imu_link3">
+    <inertial>
         <origin xyz="0 0 0" rpy="0 0 0"/>
         <mass value="0.0"/>
         <inertia ixx="0.0" ixy="0.0" ixz="0.0" iyy="0.0" iyz="0.0" izz="0.0"/>
-      </inertial>
-      <visual>
+    </inertial>
+    <visual>
         <origin xyz="0.44 0.0 -0.06" rpy="0 0 0" />
         <geometry>
             <box size = "0.05 0.05 0.05"/>
         </geometry>
-      </visual>
-    </link>
-    <gazebo reference="simulated_imu_link3">
+    </visual>
+</link>
+<gazebo reference="simulated_imu_link3">
     <gravity>true</gravity>
     <!--      Below is the line to change the material-->
@@ -690,5 +690,5 @@
       <pose>0 0 0 0 0 0</pose>
     </sensor>
-  </gazebo>
+</gazebo>
 <joint name = "simulated_imu_link_joint4" type ="fixed">
       <origin rpy="0 0 0" xyz="0 0 0"/>
@@ -696,19 +696,19 @@
       <child link="simulated_imu_link4"/>
       <axis xyz="0 0 0"/>
-    </joint>
-    <link name="simulated_imu_link4">
-      <inertial>
+</joint>
+<link name="simulated_imu_link4">
+    <inertial>
         <origin xyz="0 0 0" rpy="0 0 0"/>
         <mass value="0.0"/>
         <inertia ixx="0.0" ixy="0.0" ixz="0.0" iyy="0.0" iyz="0.0" izz="0.0"/>
-      </inertial>
-      <visual>
+    </inertial>
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