Commit message: Some changes

File: robots/panda_arm.xacro (robot description, xacro)
@@ -548,5 +548,5 @@
         </inertial>
         <visual>
-            <origin xyz="0.56 0.0 0.05" rpy="0 0 0" />
+            <origin xyz="0.16 0.0 0.05" rpy="0 0 0" />
             <geometry>
                 <box size = "0.05 0.05 0.05"/>
@@ -567,5 +567,5 @@
             <bodyName>simulated_imu_link0</bodyName>
             <gaussianNoise>0.0</gaussianNoise>
-            <xyzOffset>0.56 0.0 0.05</xyzOffset>
+            <xyzOffset>0.16 0.0 0.05</xyzOffset>
             <rpyOffset>0 0 0</rpyOffset>
             <frameName>simulated_imu_link0</frameName>
@@ -587,5 +587,5 @@
         </inertial>
         <visual>
-            <origin xyz="0.56 0.0 -0.15" rpy="0 0 0" />
+            <origin xyz="0.16 0.0 -0.15" rpy="0 0 0" />
             <geometry>
                 <box size = "0.05 0.05 0.05"/>
@@ -606,5 +606,5 @@
             <bodyName>simulated_imu_link1</bodyName>
             <gaussianNoise>0.0</gaussianNoise>
-            <xyzOffset>0.56 0.0 -0.15</xyzOffset>
+            <xyzOffset>0.16 0.0 -0.15</xyzOffset>
             <rpyOffset>0 0 0</rpyOffset>
             <frameName>simulated_imu_link1</frameName>
@@ -626,5 +626,5 @@
         </inertial>
         <visual>
-            <origin xyz="0.56 -0.15 0.0" rpy="0 0 0" />
+            <origin xyz="0.16 -0.15 0.0" rpy="0 0 0" />
             <geometry>
                 <box size = "0.05 0.05 0.05"/>
@@ -645,5 +645,5 @@
             <bodyName>simulated_imu_link2</bodyName>
             <gaussianNoise>0.0</gaussianNoise>
-            <xyzOffset>0.56 -0.15 0.0</xyzOffset>
+            <xyzOffset>0.16 -0.15 0.0</xyzOffset>
             <rpyOffset>0 0 0</rpyOffset>
             <frameName>simulated_imu_link2</frameName>
@@ -665,5 +665,5 @@
         </inertial>
         <visual>
-            <origin xyz="0.44 0.0 -0.06" rpy="0 0 0" />
+            <origin xyz="0.04 0.0 -0.06" rpy="0 0 0" />
             <geometry>
                 <box size = "0.05 0.05 0.05"/>
@@ -684,5 +684,5 @@
             <bodyName>simulated_imu_link3</bodyName>
             <gaussianNoise>0.0</gaussianNoise>
-            <xyzOffset>0.44 0.0 -0.06</xyzOffset>
+            <xyzOffset>0.04 0.0 -0.06</xyzOffset>
             <rpyOffset>0 0 0</rpyOffset>
             <frameName>simulated_imu_link3</frameName>
@@ -704,5 +704,5 @@
         </inertial>
         <visual>
-            <origin xyz="0.36 0.09 0.0" rpy="0 0 0" />
+            <origin xyz="-0.04 0.09 0.0" rpy="0 0 0" />
             <geometry>
                 <box size = "0.05 0.05 0.05"/>
@@ -723,5 +723,5 @@
             <bodyName>simulated_imu_link4</bodyName>
             <gaussianNoise>0.0</gaussianNoise>
-            <xyzOffset>0.36 0.09 0.0</xyzOffset>
+            <xyzOffset>-0.04 0.09 0.0</xyzOffset>
             <rpyOffset>0 0 0</rpyOffset>
             <frameName>simulated_imu_link4</frameName>
@@ -743,5 +743,5 @@
         </inertial>
         <visual>
-            <origin xyz="0.5 0.1 -0.11" rpy="0 0 0" />
+            <origin xyz="0.1 0.1 -0.11" rpy="0 0 0" />
             <geometry>
                 <box size = "0.05 0.05 0.05"/>
@@ -762,5 +762,5 @@
             <bodyName>simulated_imu_link5</bodyName>
             <gaussianNoise>0.0</gaussianNoise>
-            <xyzOffset>0.5 0.1 -0.11</xyzOffset>
+            <xyzOffset>0.1 0.1 -0.11</xyzOffset>
             <rpyOffset>0 0 0</rpyOffset>
             <frameName>simulated_imu_link5</frameName>
@@ -782,5 +782,5 @@
         </inertial>
         <visual>
-            <origin xyz="0.63 0.02 0.0" rpy="0 0 0" />
+            <origin xyz="0.23 0.02 0.0" rpy="0 0 0" />
             <geometry>
                 <box size = "0.05 0.05 0.05"/>
@@ -801,5 +801,5 @@
             <bodyName>simulated_imu_link6</bodyName>
             <gaussianNoise>0.0</gaussianNoise>
-            <xyzOffset>0.63 0.02 0.0</xyzOffset>
+            <xyzOffset>0.23 0.02 0.0</xyzOffset>
             <rpyOffset>0 0 0</rpyOffset>
             <frameName>simulated_imu_link6</frameName>
@@ -821,5 +821,5 @@
       </inertial>
       <visual>
-        <origin xyz="0.06 0.0 0.05" rpy="1 0 0" />
+        <origin xyz="0.06 0.0 0.05" rpy="1.57 0 0" />
           <geometry>
             <mesh scale="0.007 0.007 0.007" filename="package://${axes_meshes}/meshes/visual/arrow.dae"/>
@@ -844,5 +844,5 @@
       </inertial>
       <visual>
-        <origin xyz="0.06 0.0 0.05" rpy="0 1 0" />
+        <origin xyz="0.06 0.0 0.05" rpy="0 1.57 0" />
           <geometry>
             <mesh scale="0.007 0.007 0.007" filename="package://${axes_meshes}/meshes/visual/arrow.dae"/>
@@ -867,5 +867,5 @@
       </inertial>
       <visual>
-        <origin xyz="0.06 0.0 0.05" rpy="0 0 1" />
+        <origin xyz="0.06 0.0 0.05" rpy="0 0 1.57" />
           <geometry>
             <mesh scale="0.007 0.007 0.007" filename="package://${axes_meshes}/meshes/visual/arrow.dae"/>
@@ -890,5 +890,5 @@
       </inertial>
       <visual>
-        <origin xyz="0.06 0.0 -0.15" rpy="1 0 0" />
+        <origin xyz="0.06 0.0 -0.15" rpy="1.57 0 0" />
           <geometry>
             <mesh scale="0.007 0.007 0.007" filename="package://${axes_meshes}/meshes/visual/arrow.dae"/>
@@ -913,5 +913,5 @@
       </inertial>
       <visual>
-        <origin xyz="0.06 0.0 -0.15" rpy="0 1 0" />
+        <origin xyz="0.06 0.0 -0.15" rpy="0 1.57 0" />
           <geometry>
             <mesh scale="0.007 0.007 0.007" filename="package://${axes_meshes}/meshes/visual/arrow.dae"/>
@@ -936,5 +936,5 @@
       </inertial>
       <visual>
-        <origin xyz="0.06 0.0 -0.15" rpy="0 0 1" />
+        <origin xyz="0.06 0.0 -0.15" rpy="0 0 1.57" />
           <geometry>
             <mesh scale="0.007 0.007 0.007" filename="package://${axes_meshes}/meshes/visual/arrow.dae"/>
@@ -959,5 +959,5 @@
       </inertial>
       <visual>
-        <origin xyz="0.06 -0.15 0.0" rpy="1 0 0" />
+        <origin xyz="0.06 -0.15 0.0" rpy="1.57 0 0" />
           <geometry>
             <mesh scale="0.007 0.007 0.007" filename="package://${axes_meshes}/meshes/visual/arrow.dae"/>
@@ -982,5 +982,5 @@
       </inertial>
       <visual>
-        <origin xyz="0.06 -0.15 0.0" rpy="0 1 0" />
+        <origin xyz="0.06 -0.15 0.0" rpy="0 1.57 0" />
           <geometry>
             <mesh scale="0.007 0.007 0.007" filename="package://${axes_meshes}/meshes/visual/arrow.dae"/>
@@ -1005,5 +1005,5 @@
       </inertial>
       <visual>
-        <origin xyz="0.06 -0.15 0.0" rpy="0 0 1" />
+        <origin xyz="0.06 -0.15 0.0" rpy="0 0 1.57" />
           <geometry>
             <mesh scale="0.007 0.007 0.007" filename="package://${axes_meshes}/meshes/visual/arrow.dae"/>
@@ -1028,5 +1028,5 @@
       </inertial>
       <visual>
-        <origin xyz="-0.06 0.0 -0.06" rpy="1 0 0" />
+        <origin xyz="-0.06 0.0 -0.06" rpy="1.57 0 0" />
           <geometry>
             <mesh scale="0.007 0.007 0.007" filename="package://${axes_meshes}/meshes/visual/arrow.dae"/>
@@ -1051,5 +1051,5 @@
       </inertial>
       <visual>
-        <origin xyz="-0.06 0.0 -0.06" rpy="0 1 0" />
+        <origin xyz="-0.06 0.0 -0.06" rpy="0 1.57 0" />
           <geometry>
             <mesh scale="0.007 0.007 0.007" filename="package://${axes_meshes}/meshes/visual/arrow.dae"/>
@@ -1074,5 +1074,5 @@
       </inertial>
       <visual>
-        <origin xyz="-0.06 0.0 -0.06" rpy="0 0 1" />
+        <origin xyz="-0.06 0.0 -0.06" rpy="0 0 1.57" />
           <geometry>
             <mesh scale="0.007 0.007 0.007" filename="package://${axes_meshes}/meshes/visual/arrow.dae"/>
@@ -1097,5 +1097,5 @@
       </inertial>
       <visual>
-        <origin xyz="-0.14 0.09 0.0" rpy="1 0 0" />
+        <origin xyz="-0.14 0.09 0.0" rpy="1.57 0 0" />
           <geometry>
             <mesh scale="0.007 0.007 0.007" filename="package://${axes_meshes}/meshes/visual/arrow.dae"/>
@@ -1120,5 +1120,5 @@
       </inertial>
       <visual>
-        <origin xyz="-0.14 0.09 0.0" rpy="0 1 0" />
+        <origin xyz="-0.14 0.09 0.0" rpy="0 1.57 0" />
           <geometry>
             <mesh scale="0.007 0.007 0.007" filename="package://${axes_meshes}/meshes/visual/arrow.dae"/>
@@ -1143,5 +1143,5 @@
       </inertial>
       <visual>
-        <origin xyz="-0.14 0.09 0.0" rpy="0 0 1" />
+        <origin xyz="-0.14 0.09 0.0" rpy="0 0 1.57" />
           <geometry>
             <mesh scale="0.007 0.007 0.007" filename="package://${axes_meshes}/meshes/visual/arrow.dae"/>
@@ -1166,5 +1166,5 @@
       </inertial>
       <visual>
-        <origin xyz="0.0 0.1 -0.11" rpy="1 0 0" />
+        <origin xyz="0.0 0.1 -0.11" rpy="1.57 0 0" />
           <geometry>
             <mesh scale="0.007 0.007 0.007" filename="package://${axes_meshes}/meshes/visual/arrow.dae"/>
@@ -1189,5 +1189,5 @@
       </inertial>
       <visual>
-        <origin xyz="0.0 0.1 -0.11" rpy="0 1 0" />
+        <origin xyz="0.0 0.1 -0.11" rpy="0 1.57 0" />
           <geometry>
             <mesh scale="0.007 0.007 0.007" filename="package://${axes_meshes}/meshes/visual/arrow.dae"/>
@@ -1212,5 +1212,5 @@
       </inertial>
       <visual>
-        <origin xyz="0.0 0.1 -0.11" rpy="0 0 1" />
+        <origin xyz="0.0 0.1 -0.11" rpy="0 0 1.57" />
           <geometry>
             <mesh scale="0.007 0.007 0.007" filename="package://${axes_meshes}/meshes/visual/arrow.dae"/>
@@ -1235,5 +1235,5 @@
       </inertial>
       <visual>
-        <origin xyz="0.13 0.02 0.0" rpy="1 0 0" />
+        <origin xyz="0.13 0.02 0.0" rpy="1.57 0 0" />
           <geometry>
             <mesh scale="0.007 0.007 0.007" filename="package://${axes_meshes}/meshes/visual/arrow.dae"/>
@@ -1258,5 +1258,5 @@
       </inertial>
       <visual>
-        <origin xyz="0.13 0.02 0.0" rpy="0 1 0" />
+        <origin xyz="0.13 0.02 0.0" rpy="0 1.57 0" />
           <geometry>
             <mesh scale="0.007 0.007 0.007" filename="package://${axes_meshes}/meshes/visual/arrow.dae"/>
@@ -1281,5 +1281,5 @@
       </inertial>
       <visual>
-        <origin xyz="0.13 0.02 0.0" rpy="0 0 1" />
+        <origin xyz="0.13 0.02 0.0" rpy="0 0 1.57" />
           <geometry>
             <mesh scale="0.007 0.007 0.007" filename="package://${axes_meshes}/meshes/visual/arrow.dae"/>
@@ -1304,5 +1304,5 @@
       </inertial>
       <visual>
-        <origin xyz="0.56 0.0 0.05" rpy="1 0 0" />
+        <origin xyz="0.16 0.0 0.05" rpy="1.57 0 0" />
           <geometry>
             <mesh scale="0.007 0.007 0.007" filename="package://${axes_meshes}/meshes/visual/arrow.dae"/>
@@ -1327,5 +1327,5 @@
       </inertial>
       <visual>
-        <origin xyz="0.56 0.0 0.05" rpy="0 1 0" />
+        <origin xyz="0.16 0.0 0.05" rpy="0 1.57 0" />
           <geometry>
             <mesh scale="0.007 0.007 0.007" filename="package://${axes_meshes}/meshes/visual/arrow.dae"/>
@@ -1350,5 +1350,5 @@
       </inertial>
       <visual>
-        <origin xyz="0.56 0.0 0.05" rpy="0 0 1" />
+        <origin xyz="0.16 0.0 0.05" rpy="0 0 1.57" />
           <geometry>
             <mesh scale="0.007 0.007 0.007" filename="package://${axes_meshes}/meshes/visual/arrow.dae"/>
@@ -1373,5 +1373,5 @@
       </inertial>
       <visual>
-        <origin xyz="0.56 0.0 -0.15" rpy="1 0 0" />
+        <origin xyz="0.16 0.0 -0.15" rpy="1.57 0 0" />
           <geometry>
             <mesh scale="0.007 0.007 0.007" filename="package://${axes_meshes}/meshes/visual/arrow.dae"/>
@@ -1396,5 +1396,5 @@
       </inertial>
       <visual>
-        <origin xyz="0.56 0.0 -0.15" rpy="0 1 0" />
+        <origin xyz="0.16 0.0 -0.15" rpy="0 1.57 0" />
           <geometry>
             <mesh scale="0.007 0.007 0.007" filename="package://${axes_meshes}/meshes/visual/arrow.dae"/>
@@ -1419,5 +1419,5 @@
       </inertial>
       <visual>
-        <origin xyz="0.56 0.0 -0.15" rpy="0 0 1" />
+        <origin xyz="0.16 0.0 -0.15" rpy="0 0 1.57" />
           <geometry>
             <mesh scale="0.007 0.007 0.007" filename="package://${axes_meshes}/meshes/visual/arrow.dae"/>
@@ -1442,5 +1442,5 @@
       </inertial>
       <visual>
-        <origin xyz="0.56 -0.15 0.0" rpy="1 0 0" />
+        <origin xyz="0.16 -0.15 0.0" rpy="1.57 0 0" />
           <geometry>
             <mesh scale="0.007 0.007 0.007" filename="package://${axes_meshes}/meshes/visual/arrow.dae"/>
@@ -1465,5 +1465,5 @@
       </inertial>
       <visual>
-        <origin xyz="0.56 -0.15 0.0" rpy="0 1 0" />
+        <origin xyz="0.16 -0.15 0.0" rpy="0 1.57 0" />
           <geometry>
             <mesh scale="0.007 0.007 0.007" filename="package://${axes_meshes}/meshes/visual/arrow.dae"/>
@@ -1488,5 +1488,5 @@
       </inertial>
       <visual>
-        <origin xyz="0.56 -0.15 0.0" rpy="0 0 1" />
+        <origin xyz="0.16 -0.15 0.0" rpy="0 0 1.57" />
           <geometry>
             <mesh scale="0.007 0.007 0.007" filename="package://${axes_meshes}/meshes/visual/arrow.dae"/>
@@ -1511,5 +1511,5 @@
       </inertial>
       <visual>
-        <origin xyz="0.44 0.0 -0.06" rpy="1 0 0" />
+        <origin xyz="0.04 0.0 -0.06" rpy="1.57 0 0" />
           <geometry>
             <mesh scale="0.007 0.007 0.007" filename="package://${axes_meshes}/meshes/visual/arrow.dae"/>
@@ -1534,5 +1534,5 @@
       </inertial>
       <visual>
-        <origin xyz="0.44 0.0 -0.06" rpy="0 1 0" />
+        <origin xyz="0.04 0.0 -0.06" rpy="0 1.57 0" />
           <geometry>
             <mesh scale="0.007 0.007 0.007" filename="package://${axes_meshes}/meshes/visual/arrow.dae"/>
@@ -1557,5 +1557,5 @@
       </inertial>
       <visual>
-        <origin xyz="0.44 0.0 -0.06" rpy="0 0 1" />
+        <origin xyz="0.04 0.0 -0.06" rpy="0 0 1.57" />
           <geometry>
             <mesh scale="0.007 0.007 0.007" filename="package://${axes_meshes}/meshes/visual/arrow.dae"/>
@@ -1580,5 +1580,5 @@
       </inertial>
       <visual>
-        <origin xyz="0.36 0.09 0.0" rpy="1 0 0" />
+        <origin xyz="-0.04 0.09 0.0" rpy="1.57 0 0" />
           <geometry>
             <mesh scale="0.007 0.007 0.007" filename="package://${axes_meshes}/meshes/visual/arrow.dae"/>
@@ -1603,5 +1603,5 @@
       </inertial>
       <visual>
-        <origin xyz="0.36 0.09 0.0" rpy="0 1 0" />
+        <origin xyz="-0.04 0.09 0.0" rpy="0 1.57 0" />
           <geometry>
             <mesh scale="0.007 0.007 0.007" filename="package://${axes_meshes}/meshes/visual/arrow.dae"/>
@@ -1626,5 +1626,5 @@
       </inertial>
       <visual>
-        <origin xyz="0.36 0.09 0.0" rpy="0 0 1" />
+        <origin xyz="-0.04 0.09 0.0" rpy="0 0 1.57" />
           <geometry>
             <mesh scale="0.007 0.007 0.007" filename="package://${axes_meshes}/meshes/visual/arrow.dae"/>
@@ -1649,5 +1649,5 @@
       </inertial>
       <visual>
-        <origin xyz="0.5 0.1 -0.11" rpy="1 0 0" />
+        <origin xyz="0.1 0.1 -0.11" rpy="1.57 0 0" />
           <geometry>
             <mesh scale="0.007 0.007 0.007" filename="package://${axes_meshes}/meshes/visual/arrow.dae"/>
@@ -1672,5 +1672,5 @@
       </inertial>
       <visual>
-        <origin xyz="0.5 0.1 -0.11" rpy="0 1 0" />
+        <origin xyz="0.1 0.1 -0.11" rpy="0 1.57 0" />
           <geometry>
             <mesh scale="0.007 0.007 0.007" filename="package://${axes_meshes}/meshes/visual/arrow.dae"/>
@@ -1695,5 +1695,5 @@
       </inertial>
       <visual>
-        <origin xyz="0.5 0.1 -0.11" rpy="0 0 1" />
+        <origin xyz="0.1 0.1 -0.11" rpy="0 0 1.57" />
           <geometry>
             <mesh scale="0.007 0.007 0.007" filename="package://${axes_meshes}/meshes/visual/arrow.dae"/>
@@ -1718,5 +1718,5 @@
       </inertial>
       <visual>
-        <origin xyz="0.63 0.02 0.0" rpy="1 0 0" />
+        <origin xyz="0.23 0.02 0.0" rpy="1.57 0 0" />
           <geometry>
             <mesh scale="0.007 0.007 0.007" filename="package://${axes_meshes}/meshes/visual/arrow.dae"/>
@@ -1741,5 +1741,5 @@
       </inertial>
       <visual>
-        <origin xyz="0.63 0.02 0.0" rpy="0 1 0" />
+        <origin xyz="0.23 0.02 0.0" rpy="0 1.57 0" />
           <geometry>
             <mesh scale="0.007 0.007 0.007" filename="package://${axes_meshes}/meshes/visual/arrow.dae"/>
@@ -1764,5 +1764,5 @@
       </inertial>
       <visual>
-        <origin xyz="0.63 0.02 0.0" rpy="0 0 1" />
+        <origin xyz="0.23 0.02 0.0" rpy="0 0 1.57" />
           <geometry>
             <mesh scale="0.007 0.007 0.007" filename="package://${axes_meshes}/meshes/visual/arrow.dae"/>
