Commit message: Add masters panda arm xacro, to remove conflicts

File: robots/panda_arm.xacro (robot description, xacro)
@@ -1,5 +1,5 @@
 <?xml version='1.0' encoding='utf-8'?>
 <robot xmlns:xacro="http://www.ros.org/wiki/xacro" name="panda">
-  <xacro:macro name="panda_arm" params="arm_id:='panda' description_pkg:='franka_description' connected_to:='' xyz:='0 0 0' rpy:='0 0 0'">
+  <xacro:macro name="panda_arm" params="arm_id:='panda' description_pkg:='franka_description' axes_meshes:='ros_robotic_skin' connected_to:='' xyz:='0 0 0' rpy:='0 0 0'">
     <xacro:unless value="${not connected_to}">
       <joint name="${arm_id}_joint_${connected_to}" type="fixed">
@@ -262,285 +262,1530 @@
       <axis xyz="0 0 0"/>
     </joint>
-<!-- IMU Placement changes start from here. In kandai's words: aaaaaaaaaaa -->
     <joint name = "imu_link_joint0" type ="fixed">
+          <origin rpy="0 0 0" xyz="0 0 0"/>
+          <parent link="${arm_id}_link0"/>
+          <child link="imu_link0"/>
+          <axis xyz="0 0 0"/>
+    </joint>
+    <link name="imu_link0">
+        <inertial>
+            <origin xyz="0 0 0" rpy="0 0 0"/>
+            <mass value="0.0"/>
+            <inertia ixx="0.0" ixy="0.0" ixz="0.0" iyy="0.0" iyz="0.0" izz="0.0"/>
+        </inertial>
+        <visual>
+            <origin xyz="0.06 0.0 0.05" rpy="0 0 0" />
+            <geometry>
+                <box size = "0.05 0.05 0.05"/>
+            </geometry>
+        </visual>
+    </link>
+    <gazebo reference="imu_link0">
+        <gravity>true</gravity>
+        <!--      Below is the line to change the material-->
+        <material>Gazebo/YellowGlow</material>
+        <sensor name="imu_sensor0" type="imu">
+          <always_on>true</always_on>
+          <update_rate>100</update_rate>
+          <visualize>true</visualize>
+          <topic>imu_data0</topic>
+          <plugin filename="libgazebo_ros_imu_sensor.so" name="imu_plugin">
+            <topicName>imu_data0</topicName>
+            <bodyName>imu_link0</bodyName>
+            <updateRateHZ>100.0</updateRateHZ>
+            <gaussianNoise>0.0</gaussianNoise>
+            <xyzOffset>0.06 0.0 0.05</xyzOffset>
+            <rpyOffset>0 0 0</rpyOffset>
+            <frameName>imu_link0</frameName>
+          </plugin>
+          <pose>0 0 0 0 0 0</pose>
+        </sensor>
+    </gazebo>
+    <joint name = "imu_link_joint1" type ="fixed">
+          <origin rpy="0 0 0" xyz="0 0 0"/>
+          <parent link="${arm_id}_link1"/>
+          <child link="imu_link1"/>
+          <axis xyz="0 0 0"/>
+    </joint>
+    <link name="imu_link1">
+        <inertial>
+            <origin xyz="0 0 0" rpy="0 0 0"/>
+            <mass value="0.0"/>
+            <inertia ixx="0.0" ixy="0.0" ixz="0.0" iyy="0.0" iyz="0.0" izz="0.0"/>
+        </inertial>
+        <visual>
+            <origin xyz="0.06 0.0 -0.15" rpy="0 0 0" />
+            <geometry>
+                <box size = "0.05 0.05 0.05"/>
+            </geometry>
+        </visual>
+    </link>
+    <gazebo reference="imu_link1">
+        <gravity>true</gravity>
+        <!--      Below is the line to change the material-->
+        <material>Gazebo/YellowGlow</material>
+        <sensor name="imu_sensor1" type="imu">
+          <always_on>true</always_on>
+          <update_rate>100</update_rate>
+          <visualize>true</visualize>
+          <topic>imu_data0</topic>
+          <plugin filename="libgazebo_ros_imu_sensor.so" name="imu_plugin">
+            <topicName>imu_data1</topicName>
+            <bodyName>imu_link1</bodyName>
+            <updateRateHZ>100.0</updateRateHZ>
+            <gaussianNoise>0.0</gaussianNoise>
+            <xyzOffset>0.06 0.0 -0.15</xyzOffset>
+            <rpyOffset>0 0 0</rpyOffset>
+            <frameName>imu_link1</frameName>
+          </plugin>
+          <pose>0 0 0 0 0 0</pose>
+        </sensor>
+    </gazebo>
+    <joint name = "imu_link_joint2" type ="fixed">
+          <origin rpy="0 0 0" xyz="0 0 0"/>
+          <parent link="${arm_id}_link2"/>
+          <child link="imu_link2"/>
+          <axis xyz="0 0 0"/>
+    </joint>
+    <link name="imu_link2">
+        <inertial>
+            <origin xyz="0 0 0" rpy="0 0 0"/>
+            <mass value="0.0"/>
+            <inertia ixx="0.0" ixy="0.0" ixz="0.0" iyy="0.0" iyz="0.0" izz="0.0"/>
+        </inertial>
+        <visual>
+            <origin xyz="0.06 -0.15 0.0" rpy="0 0 0" />
+            <geometry>
+                <box size = "0.05 0.05 0.05"/>
+            </geometry>
+        </visual>
+    </link>
+    <gazebo reference="imu_link2">
+        <gravity>true</gravity>
+        <!--      Below is the line to change the material-->
+        <material>Gazebo/YellowGlow</material>
+        <sensor name="imu_sensor2" type="imu">
+          <always_on>true</always_on>
+          <update_rate>100</update_rate>
+          <visualize>true</visualize>
+          <topic>imu_data0</topic>
+          <plugin filename="libgazebo_ros_imu_sensor.so" name="imu_plugin">
+            <topicName>imu_data2</topicName>
+            <bodyName>imu_link2</bodyName>
+            <updateRateHZ>100.0</updateRateHZ>
+            <gaussianNoise>0.0</gaussianNoise>
+            <xyzOffset>0.06 -0.15 0.0</xyzOffset>
+            <rpyOffset>0 0 0</rpyOffset>
+            <frameName>imu_link2</frameName>
+          </plugin>
+          <pose>0 0 0 0 0 0</pose>
+        </sensor>
+    </gazebo>
+    <joint name = "imu_link_joint3" type ="fixed">
+          <origin rpy="0 0 0" xyz="0 0 0"/>
+          <parent link="${arm_id}_link3"/>
+          <child link="imu_link3"/>
+          <axis xyz="0 0 0"/>
+    </joint>
+    <link name="imu_link3">
+        <inertial>
+            <origin xyz="0 0 0" rpy="0 0 0"/>
+            <mass value="0.0"/>
+            <inertia ixx="0.0" ixy="0.0" ixz="0.0" iyy="0.0" iyz="0.0" izz="0.0"/>
+        </inertial>
+        <visual>
+            <origin xyz="-0.06 0.0 -0.06" rpy="0 0 0" />
+            <geometry>
+                <box size = "0.05 0.05 0.05"/>
+            </geometry>
+        </visual>
+    </link>
+    <gazebo reference="imu_link3">
+        <gravity>true</gravity>
+        <!--      Below is the line to change the material-->
+        <material>Gazebo/YellowGlow</material>
+        <sensor name="imu_sensor3" type="imu">
+          <always_on>true</always_on>
+          <update_rate>100</update_rate>
+          <visualize>true</visualize>
+          <topic>imu_data0</topic>
+          <plugin filename="libgazebo_ros_imu_sensor.so" name="imu_plugin">
+            <topicName>imu_data3</topicName>
+            <bodyName>imu_link3</bodyName>
+            <updateRateHZ>100.0</updateRateHZ>
+            <gaussianNoise>0.0</gaussianNoise>
+            <xyzOffset>-0.06 0.0 -0.06</xyzOffset>
+            <rpyOffset>0 0 0</rpyOffset>
+            <frameName>imu_link3</frameName>
+          </plugin>
+          <pose>0 0 0 0 0 0</pose>
+        </sensor>
+    </gazebo>
+    <joint name = "imu_link_joint4" type ="fixed">
+          <origin rpy="0 0 0" xyz="0 0 0"/>
+          <parent link="${arm_id}_link4"/>
+          <child link="imu_link4"/>
+          <axis xyz="0 0 0"/>
+    </joint>
+    <link name="imu_link4">
+        <inertial>
+            <origin xyz="0 0 0" rpy="0 0 0"/>
+            <mass value="0.0"/>
+            <inertia ixx="0.0" ixy="0.0" ixz="0.0" iyy="0.0" iyz="0.0" izz="0.0"/>
+        </inertial>
+        <visual>
+            <origin xyz="-0.14 0.09 0.0" rpy="0 0 0" />
+            <geometry>
+                <box size = "0.05 0.05 0.05"/>
+            </geometry>
+        </visual>
+    </link>
+    <gazebo reference="imu_link4">
+        <gravity>true</gravity>
+        <!--      Below is the line to change the material-->
+        <material>Gazebo/YellowGlow</material>
+        <sensor name="imu_sensor4" type="imu">
+          <always_on>true</always_on>
+          <update_rate>100</update_rate>
+          <visualize>true</visualize>
+          <topic>imu_data0</topic>
+          <plugin filename="libgazebo_ros_imu_sensor.so" name="imu_plugin">
+            <topicName>imu_data4</topicName>
+            <bodyName>imu_link4</bodyName>
+            <updateRateHZ>100.0</updateRateHZ>
+            <gaussianNoise>0.0</gaussianNoise>
+            <xyzOffset>-0.14 0.09 0.0</xyzOffset>
+            <rpyOffset>0 0 0</rpyOffset>
+            <frameName>imu_link4</frameName>
+          </plugin>
+          <pose>0 0 0 0 0 0</pose>
+        </sensor>
+    </gazebo>
+    <joint name = "imu_link_joint5" type ="fixed">
+          <origin rpy="0 0 0" xyz="0 0 0"/>
+          <parent link="${arm_id}_link5"/>
+          <child link="imu_link5"/>
+          <axis xyz="0 0 0"/>
+    </joint>
+    <link name="imu_link5">
+        <inertial>
+            <origin xyz="0 0 0" rpy="0 0 0"/>
+            <mass value="0.0"/>
+            <inertia ixx="0.0" ixy="0.0" ixz="0.0" iyy="0.0" iyz="0.0" izz="0.0"/>
+        </inertial>
+        <visual>
+            <origin xyz="0.0 0.1 -0.11" rpy="0 0 0" />
+            <geometry>
+                <box size = "0.05 0.05 0.05"/>
+            </geometry>
+        </visual>
+    </link>
+    <gazebo reference="imu_link5">
+        <gravity>true</gravity>
+        <!--      Below is the line to change the material-->
+        <material>Gazebo/YellowGlow</material>
+        <sensor name="imu_sensor5" type="imu">
+          <always_on>true</always_on>
+          <update_rate>100</update_rate>
+          <visualize>true</visualize>
+          <topic>imu_data0</topic>
+          <plugin filename="libgazebo_ros_imu_sensor.so" name="imu_plugin">
+            <topicName>imu_data5</topicName>
+            <bodyName>imu_link5</bodyName>
+            <updateRateHZ>100.0</updateRateHZ>
+            <gaussianNoise>0.0</gaussianNoise>
+            <xyzOffset>0.0 0.1 -0.11</xyzOffset>
+            <rpyOffset>0 0 0</rpyOffset>
+            <frameName>imu_link5</frameName>
+          </plugin>
+          <pose>0 0 0 0 0 0</pose>
+        </sensor>
+    </gazebo>
+    <joint name = "imu_link_joint6" type ="fixed">
+          <origin rpy="0 0 0" xyz="0 0 0"/>
+          <parent link="${arm_id}_link6"/>
+          <child link="imu_link6"/>
+          <axis xyz="0 0 0"/>
+    </joint>
+    <link name="imu_link6">
+        <inertial>
+            <origin xyz="0 0 0" rpy="0 0 0"/>
+            <mass value="0.0"/>
+            <inertia ixx="0.0" ixy="0.0" ixz="0.0" iyy="0.0" iyz="0.0" izz="0.0"/>
+        </inertial>
+        <visual>
+            <origin xyz="0.13 0.02 0.0" rpy="0 0 0" />
+            <geometry>
+                <box size = "0.05 0.05 0.05"/>
+            </geometry>
+        </visual>
+    </link>
+    <gazebo reference="imu_link6">
+        <gravity>true</gravity>
+        <!--      Below is the line to change the material-->
+        <material>Gazebo/YellowGlow</material>
+        <sensor name="imu_sensor6" type="imu">
+          <always_on>true</always_on>
+          <update_rate>100</update_rate>
+          <visualize>true</visualize>
+          <topic>imu_data0</topic>
+          <plugin filename="libgazebo_ros_imu_sensor.so" name="imu_plugin">
+            <topicName>imu_data6</topicName>
+            <bodyName>imu_link6</bodyName>
+            <updateRateHZ>100.0</updateRateHZ>
+            <gaussianNoise>0.0</gaussianNoise>
+            <xyzOffset>0.13 0.02 0.0</xyzOffset>
+            <rpyOffset>0 0 0</rpyOffset>
+            <frameName>imu_link6</frameName>
+          </plugin>
+          <pose>0 0 0 0 0 0</pose>
+        </sensor>
+    </gazebo>
+    <joint name = "simulated_imu_link_joint0" type ="fixed">
+          <origin rpy="0 0 0" xyz="0 0 0"/>
+          <parent link="${arm_id}_link0"/>
+          <child link="simulated_imu_link0"/>
+          <axis xyz="0 0 0"/>
+    </joint>
+    <link name="simulated_imu_link0">
+        <inertial>
+            <origin xyz="0 0 0" rpy="0 0 0"/>
+            <mass value="0.0"/>
+            <inertia ixx="0.0" ixy="0.0" ixz="0.0" iyy="0.0" iyz="0.0" izz="0.0"/>
+        </inertial>
+        <visual>
+            <origin xyz="0.16 0.0 0.05" rpy="0 0 0" />
+            <geometry>
+                <box size = "0.05 0.05 0.05"/>
+            </geometry>
+        </visual>
+    </link>
+    <gazebo reference="simulated_imu_link0">
+        <gravity>true</gravity>
+        <!--      Below is the line to change the material-->
+        <material>Gazebo/YellowGlow</material>
+        <sensor name="simulated_imu_sensor0" type="imu">
+          <always_on>true</always_on>
+          <update_rate>100</update_rate>
+          <visualize>true</visualize>
+          <topic>imu_data0</topic>
+          <plugin filename="libgazebo_ros_imu_sensor.so" name="imu_plugin">
+            <topicName>simulated_imu_data0</topicName>
+            <bodyName>simulated_imu_link0</bodyName>
+            <updateRateHZ>100.0</updateRateHZ>
+            <gaussianNoise>0.0</gaussianNoise>
+            <xyzOffset>0.16 0.0 0.05</xyzOffset>
+            <rpyOffset>0 0 0</rpyOffset>
+            <frameName>simulated_imu_link0</frameName>
+          </plugin>
+          <pose>0 0 0 0 0 0</pose>
+        </sensor>
+    </gazebo>
+    <joint name = "simulated_imu_link_joint1" type ="fixed">
+          <origin rpy="0 0 0" xyz="0 0 0"/>
+          <parent link="${arm_id}_link1"/>
+          <child link="simulated_imu_link1"/>
+          <axis xyz="0 0 0"/>
+    </joint>
+    <link name="simulated_imu_link1">
+        <inertial>
+            <origin xyz="0 0 0" rpy="0 0 0"/>
+            <mass value="0.0"/>
+            <inertia ixx="0.0" ixy="0.0" ixz="0.0" iyy="0.0" iyz="0.0" izz="0.0"/>
+        </inertial>
+        <visual>
+            <origin xyz="0.16 0.0 -0.15" rpy="0 0 0" />
+            <geometry>
+                <box size = "0.05 0.05 0.05"/>
+            </geometry>
+        </visual>
+    </link>
+    <gazebo reference="simulated_imu_link1">
+        <gravity>true</gravity>
+        <!--      Below is the line to change the material-->
+        <material>Gazebo/YellowGlow</material>
+        <sensor name="simulated_imu_sensor1" type="imu">
+          <always_on>true</always_on>
+          <update_rate>100</update_rate>
+          <visualize>true</visualize>
+          <topic>imu_data0</topic>
+          <plugin filename="libgazebo_ros_imu_sensor.so" name="imu_plugin">
+            <topicName>simulated_imu_data1</topicName>
+            <bodyName>simulated_imu_link1</bodyName>
+            <updateRateHZ>100.0</updateRateHZ>
+            <gaussianNoise>0.0</gaussianNoise>
+            <xyzOffset>0.16 0.0 -0.15</xyzOffset>
+            <rpyOffset>0 0 0</rpyOffset>
+            <frameName>simulated_imu_link1</frameName>
+          </plugin>
+          <pose>0 0 0 0 0 0</pose>
+        </sensor>
+    </gazebo>
+    <joint name = "simulated_imu_link_joint2" type ="fixed">
+          <origin rpy="0 0 0" xyz="0 0 0"/>
+          <parent link="${arm_id}_link2"/>
+          <child link="simulated_imu_link2"/>
+          <axis xyz="0 0 0"/>
+    </joint>
+    <link name="simulated_imu_link2">
+        <inertial>
+            <origin xyz="0 0 0" rpy="0 0 0"/>
+            <mass value="0.0"/>
+            <inertia ixx="0.0" ixy="0.0" ixz="0.0" iyy="0.0" iyz="0.0" izz="0.0"/>
+        </inertial>
+        <visual>
+            <origin xyz="0.16 -0.15 0.0" rpy="0 0 0" />
+            <geometry>
+                <box size = "0.05 0.05 0.05"/>
+            </geometry>
+        </visual>
+    </link>
+    <gazebo reference="simulated_imu_link2">
+        <gravity>true</gravity>
+        <!--      Below is the line to change the material-->
+        <material>Gazebo/YellowGlow</material>
+        <sensor name="simulated_imu_sensor2" type="imu">
+          <always_on>true</always_on>
+          <update_rate>100</update_rate>
+          <visualize>true</visualize>
+          <topic>imu_data0</topic>
+          <plugin filename="libgazebo_ros_imu_sensor.so" name="imu_plugin">
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