Commit message: Fixed IMU2

File: robots/panda_arm.xacro (robot description, xacro)
@@ -343,5 +343,5 @@
     </gazebo>
     <joint name = "imu_link_joint2" type ="fixed">
-          <origin rpy="0 0 0" xyz="0 0 0"/>
+          <origin rpy="0 0 1.57" xyz="0 0 0"/>
           <parent link="${arm_id}_link2"/>
           <child link="imu_link2"/>
@@ -355,5 +355,5 @@
         </inertial>
         <visual>
-            <origin xyz="0.06 -0.15 0.0" rpy="0 0 0" />
+            <origin xyz="0.06 -0.15 0.0" rpy="0 0 1.57" />
             <geometry>
                 <box size = "0.05 0.05 0.05"/>
@@ -376,5 +376,5 @@
             <gaussianNoise>0.0</gaussianNoise>
             <xyzOffset>0.06 -0.15 0.0</xyzOffset>
-            <rpyOffset>0 0 0</rpyOffset>
+            <rpyOffset>0 0 1.57</rpyOffset>
             <frameName>imu_link2</frameName>
           </plugin>
@@ -555,5 +555,5 @@
         </inertial>
         <visual>
-            <origin xyz="0.16 0.0 0.05" rpy="0 0 0" />
+            <origin xyz="0.36 0.0 0.05" rpy="0 0 0" />
             <geometry>
                 <box size = "0.05 0.05 0.05"/>
@@ -575,5 +575,5 @@
             <updateRateHZ>100.0</updateRateHZ>
             <gaussianNoise>0.0</gaussianNoise>
-            <xyzOffset>0.16 0.0 0.05</xyzOffset>
+            <xyzOffset>0.36 0.0 0.05</xyzOffset>
             <rpyOffset>0 0 0</rpyOffset>
             <frameName>simulated_imu_link0</frameName>
@@ -595,5 +595,5 @@
         </inertial>
         <visual>
-            <origin xyz="0.16 0.0 -0.15" rpy="0 0 0" />
+            <origin xyz="0.36 0.0 -0.15" rpy="0 0 0" />
             <geometry>
                 <box size = "0.05 0.05 0.05"/>
@@ -615,5 +615,5 @@
             <updateRateHZ>100.0</updateRateHZ>
             <gaussianNoise>0.0</gaussianNoise>
-            <xyzOffset>0.16 0.0 -0.15</xyzOffset>
+            <xyzOffset>0.36 0.0 -0.15</xyzOffset>
             <rpyOffset>0 0 0</rpyOffset>
             <frameName>simulated_imu_link1</frameName>
@@ -623,5 +623,5 @@
     </gazebo>
     <joint name = "simulated_imu_link_joint2" type ="fixed">
-          <origin rpy="0 0 0" xyz="0 0 0"/>
+          <origin rpy="0 0 1.57" xyz="0 0 0"/>
           <parent link="${arm_id}_link2"/>
           <child link="simulated_imu_link2"/>
@@ -635,5 +635,5 @@
         </inertial>
         <visual>
-            <origin xyz="0.16 -0.15 0.0" rpy="0 0 0" />
+            <origin xyz="0.36 -0.15 0.0" rpy="0 0 1.57" />
             <geometry>
                 <box size = "0.05 0.05 0.05"/>
@@ -655,6 +655,6 @@
             <updateRateHZ>100.0</updateRateHZ>
             <gaussianNoise>0.0</gaussianNoise>
-            <xyzOffset>0.16 -0.15 0.0</xyzOffset>
-            <rpyOffset>0 0 0</rpyOffset>
+            <xyzOffset>0.36 -0.15 0.0</xyzOffset>
+            <rpyOffset>0 0 1.57</rpyOffset>
             <frameName>simulated_imu_link2</frameName>
           </plugin>
@@ -675,5 +675,5 @@
         </inertial>
         <visual>
-            <origin xyz="0.04 0.0 -0.06" rpy="0 0 0" />
+            <origin xyz="0.24 0.0 -0.06" rpy="0 0 0" />
             <geometry>
                 <box size = "0.05 0.05 0.05"/>
@@ -695,5 +695,5 @@
             <updateRateHZ>100.0</updateRateHZ>
             <gaussianNoise>0.0</gaussianNoise>
-            <xyzOffset>0.04 0.0 -0.06</xyzOffset>
+            <xyzOffset>0.24 0.0 -0.06</xyzOffset>
             <rpyOffset>0 0 0</rpyOffset>
             <frameName>simulated_imu_link3</frameName>
@@ -715,5 +715,5 @@
         </inertial>
         <visual>
-            <origin xyz="-0.04 0.09 0.0" rpy="0 0 0" />
+            <origin xyz="0.16 0.09 0.0" rpy="0 0 0" />
             <geometry>
                 <box size = "0.05 0.05 0.05"/>
@@ -735,5 +735,5 @@
             <updateRateHZ>100.0</updateRateHZ>
             <gaussianNoise>0.0</gaussianNoise>
-            <xyzOffset>-0.04 0.09 0.0</xyzOffset>
+            <xyzOffset>0.16 0.09 0.0</xyzOffset>
             <rpyOffset>0 0 0</rpyOffset>
             <frameName>simulated_imu_link4</frameName>
@@ -755,5 +755,5 @@
         </inertial>
         <visual>
-            <origin xyz="0.1 0.1 -0.11" rpy="0 0 0" />
+            <origin xyz="0.3 0.1 -0.11" rpy="0 0 0" />
             <geometry>
                 <box size = "0.05 0.05 0.05"/>
@@ -775,5 +775,5 @@
             <updateRateHZ>100.0</updateRateHZ>
             <gaussianNoise>0.0</gaussianNoise>
-            <xyzOffset>0.1 0.1 -0.11</xyzOffset>
+            <xyzOffset>0.3 0.1 -0.11</xyzOffset>
             <rpyOffset>0 0 0</rpyOffset>
             <frameName>simulated_imu_link5</frameName>
@@ -795,5 +795,5 @@
         </inertial>
         <visual>
-            <origin xyz="0.23 0.02 0.0" rpy="0 0 0" />
+            <origin xyz="0.43 0.02 0.0" rpy="0 0 0" />
             <geometry>
                 <box size = "0.05 0.05 0.05"/>
@@ -815,5 +815,5 @@
             <updateRateHZ>100.0</updateRateHZ>
             <gaussianNoise>0.0</gaussianNoise>
-            <xyzOffset>0.23 0.02 0.0</xyzOffset>
+            <xyzOffset>0.43 0.02 0.0</xyzOffset>
             <rpyOffset>0 0 0</rpyOffset>
             <frameName>simulated_imu_link6</frameName>
@@ -1318,5 +1318,5 @@
       </inertial>
       <visual>
-        <origin xyz="0.16 0.0 0.05" rpy="1.57 0 0" />
+        <origin xyz="0.36 0.0 0.05" rpy="1.57 0 0" />
           <geometry>
             <mesh scale="0.007 0.007 0.007" filename="package://${axes_meshes}/meshes/visual/arrow.dae"/>
@@ -1341,5 +1341,5 @@
       </inertial>
       <visual>
-        <origin xyz="0.16 0.0 0.05" rpy="0 1.57 0" />
+        <origin xyz="0.36 0.0 0.05" rpy="0 1.57 0" />
           <geometry>
             <mesh scale="0.007 0.007 0.007" filename="package://${axes_meshes}/meshes/visual/arrow.dae"/>
@@ -1364,5 +1364,5 @@
       </inertial>
       <visual>
-        <origin xyz="0.16 0.0 0.05" rpy="0 0 1.57" />
+        <origin xyz="0.36 0.0 0.05" rpy="0 0 1.57" />
           <geometry>
             <mesh scale="0.007 0.007 0.007" filename="package://${axes_meshes}/meshes/visual/arrow.dae"/>
@@ -1387,5 +1387,5 @@
       </inertial>
       <visual>
-        <origin xyz="0.16 0.0 -0.15" rpy="1.57 0 0" />
+        <origin xyz="0.36 0.0 -0.15" rpy="1.57 0 0" />
           <geometry>
             <mesh scale="0.007 0.007 0.007" filename="package://${axes_meshes}/meshes/visual/arrow.dae"/>
@@ -1410,5 +1410,5 @@
       </inertial>
       <visual>
-        <origin xyz="0.16 0.0 -0.15" rpy="0 1.57 0" />
+        <origin xyz="0.36 0.0 -0.15" rpy="0 1.57 0" />
           <geometry>
             <mesh scale="0.007 0.007 0.007" filename="package://${axes_meshes}/meshes/visual/arrow.dae"/>
@@ -1433,5 +1433,5 @@
       </inertial>
       <visual>
-        <origin xyz="0.16 0.0 -0.15" rpy="0 0 1.57" />
+        <origin xyz="0.36 0.0 -0.15" rpy="0 0 1.57" />
           <geometry>
             <mesh scale="0.007 0.007 0.007" filename="package://${axes_meshes}/meshes/visual/arrow.dae"/>
@@ -1456,5 +1456,5 @@
       </inertial>
       <visual>
-        <origin xyz="0.16 -0.15 0.0" rpy="1.57 0 0" />
+        <origin xyz="0.36 -0.15 0.0" rpy="1.57 0 0" />
           <geometry>
             <mesh scale="0.007 0.007 0.007" filename="package://${axes_meshes}/meshes/visual/arrow.dae"/>
@@ -1479,5 +1479,5 @@
       </inertial>
       <visual>
-        <origin xyz="0.16 -0.15 0.0" rpy="0 1.57 0" />
+        <origin xyz="0.36 -0.15 0.0" rpy="0 1.57 0" />
           <geometry>
             <mesh scale="0.007 0.007 0.007" filename="package://${axes_meshes}/meshes/visual/arrow.dae"/>
@@ -1502,5 +1502,5 @@
       </inertial>
       <visual>
-        <origin xyz="0.16 -0.15 0.0" rpy="0 0 1.57" />
+        <origin xyz="0.36 -0.15 0.0" rpy="0 0 1.57" />
           <geometry>
             <mesh scale="0.007 0.007 0.007" filename="package://${axes_meshes}/meshes/visual/arrow.dae"/>
@@ -1525,5 +1525,5 @@
       </inertial>
       <visual>
-        <origin xyz="0.04 0.0 -0.06" rpy="1.57 0 0" />
+        <origin xyz="0.24 0.0 -0.06" rpy="1.57 0 0" />
           <geometry>
             <mesh scale="0.007 0.007 0.007" filename="package://${axes_meshes}/meshes/visual/arrow.dae"/>
@@ -1548,5 +1548,5 @@
       </inertial>
       <visual>
-        <origin xyz="0.04 0.0 -0.06" rpy="0 1.57 0" />
+        <origin xyz="0.24 0.0 -0.06" rpy="0 1.57 0" />
           <geometry>
             <mesh scale="0.007 0.007 0.007" filename="package://${axes_meshes}/meshes/visual/arrow.dae"/>
@@ -1571,5 +1571,5 @@
       </inertial>
       <visual>
-        <origin xyz="0.04 0.0 -0.06" rpy="0 0 1.57" />
+        <origin xyz="0.24 0.0 -0.06" rpy="0 0 1.57" />
           <geometry>
             <mesh scale="0.007 0.007 0.007" filename="package://${axes_meshes}/meshes/visual/arrow.dae"/>
@@ -1594,5 +1594,5 @@
       </inertial>
       <visual>
-        <origin xyz="-0.04 0.09 0.0" rpy="1.57 0 0" />
+        <origin xyz="0.16 0.09 0.0" rpy="1.57 0 0" />
           <geometry>
             <mesh scale="0.007 0.007 0.007" filename="package://${axes_meshes}/meshes/visual/arrow.dae"/>
@@ -1617,5 +1617,5 @@
       </inertial>
       <visual>
-        <origin xyz="-0.04 0.09 0.0" rpy="0 1.57 0" />
+        <origin xyz="0.16 0.09 0.0" rpy="0 1.57 0" />
           <geometry>
             <mesh scale="0.007 0.007 0.007" filename="package://${axes_meshes}/meshes/visual/arrow.dae"/>
@@ -1640,5 +1640,5 @@
       </inertial>
       <visual>
-        <origin xyz="-0.04 0.09 0.0" rpy="0 0 1.57" />
+        <origin xyz="0.16 0.09 0.0" rpy="0 0 1.57" />
           <geometry>
             <mesh scale="0.007 0.007 0.007" filename="package://${axes_meshes}/meshes/visual/arrow.dae"/>
@@ -1663,5 +1663,5 @@
       </inertial>
       <visual>
-        <origin xyz="0.1 0.1 -0.11" rpy="1.57 0 0" />
+        <origin xyz="0.3 0.1 -0.11" rpy="1.57 0 0" />
           <geometry>
             <mesh scale="0.007 0.007 0.007" filename="package://${axes_meshes}/meshes/visual/arrow.dae"/>
@@ -1686,5 +1686,5 @@
       </inertial>
       <visual>
-        <origin xyz="0.1 0.1 -0.11" rpy="0 1.57 0" />
+        <origin xyz="0.3 0.1 -0.11" rpy="0 1.57 0" />
           <geometry>
             <mesh scale="0.007 0.007 0.007" filename="package://${axes_meshes}/meshes/visual/arrow.dae"/>
@@ -1709,5 +1709,5 @@
       </inertial>
       <visual>
-        <origin xyz="0.1 0.1 -0.11" rpy="0 0 1.57" />
+        <origin xyz="0.3 0.1 -0.11" rpy="0 0 1.57" />
           <geometry>
             <mesh scale="0.007 0.007 0.007" filename="package://${axes_meshes}/meshes/visual/arrow.dae"/>
@@ -1732,5 +1732,5 @@
       </inertial>
       <visual>
-        <origin xyz="0.23 0.02 0.0" rpy="1.57 0 0" />
+        <origin xyz="0.43 0.02 0.0" rpy="1.57 0 0" />
           <geometry>
             <mesh scale="0.007 0.007 0.007" filename="package://${axes_meshes}/meshes/visual/arrow.dae"/>
@@ -1755,5 +1755,5 @@
       </inertial>
       <visual>
-        <origin xyz="0.23 0.02 0.0" rpy="0 1.57 0" />
+        <origin xyz="0.43 0.02 0.0" rpy="0 1.57 0" />
           <geometry>
             <mesh scale="0.007 0.007 0.007" filename="package://${axes_meshes}/meshes/visual/arrow.dae"/>
@@ -1778,5 +1778,5 @@
       </inertial>
       <visual>
-        <origin xyz="0.23 0.02 0.0" rpy="0 0 1.57" />
+        <origin xyz="0.43 0.02 0.0" rpy="0 0 1.57" />
           <geometry>
             <mesh scale="0.007 0.007 0.007" filename="package://${axes_meshes}/meshes/visual/arrow.dae"/>

Commit message: Fixed IMU2 for real

File: robots/panda_arm.xacro (robot description, xacro)
@@ -343,5 +343,5 @@
     </gazebo>
     <joint name = "imu_link_joint2" type ="fixed">
-          <origin rpy="0 0 1.57" xyz="0 0 0"/>
+          <origin rpy="1.57 0 1.57" xyz="0 0 0"/>
           <parent link="${arm_id}_link2"/>
           <child link="imu_link2"/>
@@ -355,5 +355,5 @@
         </inertial>
         <visual>
-            <origin xyz="0.06 -0.15 0.0" rpy="0 0 1.57" />
+            <origin xyz="0.06 -0.15 0.0" rpy="1.57 0 1.57" />
             <geometry>
                 <box size = "0.05 0.05 0.05"/>
@@ -376,5 +376,5 @@
             <gaussianNoise>0.0</gaussianNoise>
             <xyzOffset>0.06 -0.15 0.0</xyzOffset>
-            <rpyOffset>0 0 1.57</rpyOffset>
+            <rpyOffset>1.57 0 1.57</rpyOffset>
             <frameName>imu_link2</frameName>
           </plugin>
@@ -623,5 +623,5 @@
     </gazebo>
     <joint name = "simulated_imu_link_joint2" type ="fixed">
-          <origin rpy="0 0 1.57" xyz="0 0 0"/>
+          <origin rpy="1.57 0 1.57" xyz="0 0 0"/>
           <parent link="${arm_id}_link2"/>
           <child link="simulated_imu_link2"/>
@@ -635,5 +635,5 @@
         </inertial>
         <visual>
-            <origin xyz="0.36 -0.15 0.0" rpy="0 0 1.57" />
+            <origin xyz="0.36 -0.15 0.0" rpy="1.57 0 1.57" />
             <geometry>
                 <box size = "0.05 0.05 0.05"/>
@@ -656,5 +656,5 @@
             <gaussianNoise>0.0</gaussianNoise>
             <xyzOffset>0.36 -0.15 0.0</xyzOffset>
-            <rpyOffset>0 0 1.57</rpyOffset>
+            <rpyOffset>1.57 0 1.57</rpyOffset>
             <frameName>simulated_imu_link2</frameName>
           </plugin>
