Commit message: All IMU's verified, axes verified, Stable commit

File: robots/panda_arm.xacro (robot description, xacro)
@@ -262,4 +262,124 @@
       <axis xyz="0 0 0"/>
     </joint>
+    <joint name = "imu_link_joint0" type ="fixed">
+          <origin rpy="1.57 0 1.57" xyz="0 0 0"/>
+          <parent link="${arm_id}_link0"/>
+          <child link="imu_link0"/>
+          <axis xyz="0 0 0"/>
+    </joint>
+    <link name="imu_link0">
+        <inertial>
+            <origin xyz="0 0 0" rpy="0 0 0"/>
+            <mass value="0.0"/>
+            <inertia ixx="0.0" ixy="0.0" ixz="0.0" iyy="0.0" iyz="0.0" izz="0.0"/>
+        </inertial>
+        <visual>
+            <origin xyz="0.0 0.05 0.06" rpy="1.57 0 1.57" />
+            <geometry>
+                <box size = "0.05 0.05 0.05"/>
+            </geometry>
+        </visual>
+    </link>
+    <gazebo reference="imu_link0">
+        <gravity>true</gravity>
+        <!--      Below is the line to change the material-->
+        <material>Gazebo/YellowGlow</material>
+        <sensor name="imu_sensor0" type="imu">
+          <always_on>true</always_on>
+          <update_rate>100</update_rate>
+          <visualize>true</visualize>
+          <topic>imu_data0</topic>
+          <plugin filename="libgazebo_ros_imu_sensor.so" name="imu_plugin">
+            <topicName>imu_data0</topicName>
+            <bodyName>imu_link0</bodyName>
+            <updateRateHZ>100.0</updateRateHZ>
+            <gaussianNoise>0.0</gaussianNoise>
+            <xyzOffset>0.0 0.05 0.06</xyzOffset>
+            <rpyOffset>1.57 0 1.57</rpyOffset>
+            <frameName>imu_link0</frameName>
+          </plugin>
+          <pose>0 0 0 0 0 0</pose>
+        </sensor>
+    </gazebo>
+    <joint name = "imu_link_joint1" type ="fixed">
+          <origin rpy="1.57 0 1.57" xyz="0 0 0"/>
+          <parent link="${arm_id}_link1"/>
+          <child link="imu_link1"/>
+          <axis xyz="0 0 0"/>
+    </joint>
+    <link name="imu_link1">
+        <inertial>
+            <origin xyz="0 0 0" rpy="0 0 0"/>
+            <mass value="0.0"/>
+            <inertia ixx="0.0" ixy="0.0" ixz="0.0" iyy="0.0" iyz="0.0" izz="0.0"/>
+        </inertial>
+        <visual>
+            <origin xyz="0.0 -0.15 0.06" rpy="1.57 0 1.57" />
+            <geometry>
+                <box size = "0.05 0.05 0.05"/>
+            </geometry>
+        </visual>
+    </link>
+    <gazebo reference="imu_link1">
+        <gravity>true</gravity>
+        <!--      Below is the line to change the material-->
+        <material>Gazebo/YellowGlow</material>
+        <sensor name="imu_sensor1" type="imu">
+          <always_on>true</always_on>
+          <update_rate>100</update_rate>
+          <visualize>true</visualize>
+          <topic>imu_data0</topic>
+          <plugin filename="libgazebo_ros_imu_sensor.so" name="imu_plugin">
+            <topicName>imu_data1</topicName>
+            <bodyName>imu_link1</bodyName>
+            <updateRateHZ>100.0</updateRateHZ>
+            <gaussianNoise>0.0</gaussianNoise>
+            <xyzOffset>0.0 -0.15 0.06</xyzOffset>
+            <rpyOffset>1.57 0 1.57</rpyOffset>
+            <frameName>imu_link1</frameName>
+          </plugin>
+          <pose>0 0 0 0 0 0</pose>
+        </sensor>
+    </gazebo>
+    <joint name = "imu_link_joint2" type ="fixed">
+          <origin rpy="3.14 -1.57 0" xyz="0 0 0"/>
+          <parent link="${arm_id}_link2"/>
+          <child link="imu_link2"/>
+          <axis xyz="0 0 0"/>
+    </joint>
+    <link name="imu_link2">
+        <inertial>
+            <origin xyz="0 0 0" rpy="0 0 0"/>
+            <mass value="0.0"/>
+            <inertia ixx="0.0" ixy="0.0" ixz="0.0" iyy="0.0" iyz="0.0" izz="0.0"/>
+        </inertial>
+        <visual>
+            <origin xyz="0.0 0.15 0.06" rpy="3.14 -1.57 0" />
+            <geometry>
+                <box size = "0.05 0.05 0.05"/>
+            </geometry>
+        </visual>
+    </link>
+    <gazebo reference="imu_link2">
+        <gravity>true</gravity>
+        <!--      Below is the line to change the material-->
+        <material>Gazebo/YellowGlow</material>
+        <sensor name="imu_sensor2" type="imu">
+          <always_on>true</always_on>
+          <update_rate>100</update_rate>
+          <visualize>true</visualize>
+          <topic>imu_data0</topic>
+          <plugin filename="libgazebo_ros_imu_sensor.so" name="imu_plugin">
+            <topicName>imu_data2</topicName>
+            <bodyName>imu_link2</bodyName>
+            <updateRateHZ>100.0</updateRateHZ>
+            <gaussianNoise>0.0</gaussianNoise>
+            <xyzOffset>0.0 0.15 0.06</xyzOffset>
+            <rpyOffset>3.14 -1.57 0</rpyOffset>
+            <frameName>imu_link2</frameName>
+          </plugin>
+          <pose>0 0 0 0 0 0</pose>
+        </sensor>
+    </gazebo>
     <joint name = "imu_link_joint3" type ="fixed">
           <origin rpy="0 -1.57 0" xyz="0 0 0"/>
@@ -275,5 +395,5 @@
         </inertial>
         <visual>
-            <origin xyz="0.06 0.0 0.06" rpy="0 -1.57 0" />
+            <origin xyz="-0.06 0.0 0.06" rpy="0 -1.57 0" />
             <geometry>
                 <box size = "0.05 0.05 0.05"/>
@@ -295,5 +415,5 @@
             <updateRateHZ>100.0</updateRateHZ>
             <gaussianNoise>0.0</gaussianNoise>
-            <xyzOffset>0.06 0.0 0.06</xyzOffset>
+            <xyzOffset>-0.06 0.0 0.06</xyzOffset>
             <rpyOffset>0 -1.57 0</rpyOffset>
             <frameName>imu_link3</frameName>
@@ -302,4 +422,331 @@
         </sensor>
     </gazebo>
+    <joint name = "imu_link_joint4" type ="fixed">
+          <origin rpy="0 -1.57 0" xyz="0 0 0"/>
+          <parent link="${arm_id}_link4"/>
+          <child link="imu_link4"/>
+          <axis xyz="0 0 0"/>
+    </joint>
+    <link name="imu_link4">
+        <inertial>
+            <origin xyz="0 0 0" rpy="0 0 0"/>
+            <mass value="0.0"/>
+            <inertia ixx="0.0" ixy="0.0" ixz="0.0" iyy="0.0" iyz="0.0" izz="0.0"/>
+        </inertial>
+        <visual>
+            <origin xyz="0.0 0.09 0.14" rpy="0 -1.57 0" />
+            <geometry>
+                <box size = "0.05 0.05 0.05"/>
+            </geometry>
+        </visual>
+    </link>
+    <gazebo reference="imu_link4">
+        <gravity>true</gravity>
+        <!--      Below is the line to change the material-->
+        <material>Gazebo/YellowGlow</material>
+        <sensor name="imu_sensor4" type="imu">
+          <always_on>true</always_on>
+          <update_rate>100</update_rate>
+          <visualize>true</visualize>
+          <topic>imu_data0</topic>
+          <plugin filename="libgazebo_ros_imu_sensor.so" name="imu_plugin">
+            <topicName>imu_data4</topicName>
+            <bodyName>imu_link4</bodyName>
+            <updateRateHZ>100.0</updateRateHZ>
+            <gaussianNoise>0.0</gaussianNoise>
+            <xyzOffset>0.0 0.09 0.14</xyzOffset>
+            <rpyOffset>0 -1.57 0</rpyOffset>
+            <frameName>imu_link4</frameName>
+          </plugin>
+          <pose>0 0 0 0 0 0</pose>
+        </sensor>
+    </gazebo>
+    <joint name = "imu_link_joint5" type ="fixed">
+          <origin rpy="-1.57 3.14 0" xyz="0 0 0"/>
+          <parent link="${arm_id}_link5"/>
+          <child link="imu_link5"/>
+          <axis xyz="0 0 0"/>
+    </joint>
+    <link name="imu_link5">
+        <inertial>
+            <origin xyz="0 0 0" rpy="0 0 0"/>
+            <mass value="0.0"/>
+            <inertia ixx="0.0" ixy="0.0" ixz="0.0" iyy="0.0" iyz="0.0" izz="0.0"/>
+        </inertial>
+        <visual>
+            <origin xyz="0.0 -0.11 0.1" rpy="-1.57 3.14 0" />
+            <geometry>
+                <box size = "0.05 0.05 0.05"/>
+            </geometry>
+        </visual>
+    </link>
+    <gazebo reference="imu_link5">
+        <gravity>true</gravity>
+        <!--      Below is the line to change the material-->
+        <material>Gazebo/YellowGlow</material>
+        <sensor name="imu_sensor5" type="imu">
+          <always_on>true</always_on>
+          <update_rate>100</update_rate>
+          <visualize>true</visualize>
+          <topic>imu_data0</topic>
+          <plugin filename="libgazebo_ros_imu_sensor.so" name="imu_plugin">
+            <topicName>imu_data5</topicName>
+            <bodyName>imu_link5</bodyName>
+            <updateRateHZ>100.0</updateRateHZ>
+            <gaussianNoise>0.0</gaussianNoise>
+            <xyzOffset>0.0 -0.11 0.1</xyzOffset>
+            <rpyOffset>-1.57 3.14 0</rpyOffset>
+            <frameName>imu_link5</frameName>
+          </plugin>
+          <pose>0 0 0 0 0 0</pose>
+        </sensor>
+    </gazebo>
+    <joint name = "imu_link_joint6" type ="fixed">
+          <origin rpy="1.57 0 1.57" xyz="0 0 0"/>
+          <parent link="${arm_id}_link6"/>
+          <child link="imu_link6"/>
+          <axis xyz="0 0 0"/>
+    </joint>
+    <link name="imu_link6">
+        <inertial>
+            <origin xyz="0 0 0" rpy="0 0 0"/>
+            <mass value="0.0"/>
+            <inertia ixx="0.0" ixy="0.0" ixz="0.0" iyy="0.0" iyz="0.0" izz="0.0"/>
+        </inertial>
+        <visual>
+            <origin xyz="0.02 0.0 0.13" rpy="1.57 0 1.57" />
+            <geometry>
+                <box size = "0.05 0.05 0.05"/>
+            </geometry>
+        </visual>
+    </link>
+    <gazebo reference="imu_link6">
+        <gravity>true</gravity>
+        <!--      Below is the line to change the material-->
+        <material>Gazebo/YellowGlow</material>
+        <sensor name="imu_sensor6" type="imu">
+          <always_on>true</always_on>
+          <update_rate>100</update_rate>
+          <visualize>true</visualize>
+          <topic>imu_data0</topic>
+          <plugin filename="libgazebo_ros_imu_sensor.so" name="imu_plugin">
+            <topicName>imu_data6</topicName>
+            <bodyName>imu_link6</bodyName>
+            <updateRateHZ>100.0</updateRateHZ>
+            <gaussianNoise>0.0</gaussianNoise>
+            <xyzOffset>0.02 0.0 0.13</xyzOffset>
+            <rpyOffset>1.57 0 1.57</rpyOffset>
+            <frameName>imu_link6</frameName>
+          </plugin>
+          <pose>0 0 0 0 0 0</pose>
+        </sensor>
+    </gazebo>
+    <joint name = "imu_link_joint0_x_axis" type ="fixed">
+      <origin rpy="1.57 0 1.57" xyz="0 0 0"/>
+      <parent link="${arm_id}_link0"/>
+      <child link="imu_link_axes0_x_axis"/>
+      <axis xyz="0 0 0"/>
+    </joint>
+    <link name="imu_link_axes0_x_axis">
+      <inertial>
+        <origin xyz="0 0 0" rpy="0 0 0"/>
+        <mass value="0.0"/>
+        <inertia ixx="0.0" ixy="0.0" ixz="0.0" iyy="0.0" iyz="0.0" izz="0.0"/>
+      </inertial>
+      <visual>
+        <origin xyz="0.0 0.05 0.06" rpy="0 1.57 0" />
+          <geometry>
+            <mesh scale="0.007 0.007 0.007" filename="package://${axes_meshes}/meshes/visual/arrow.dae"/>
+          </geometry>
+        </visual>
+    </link>
+    <gazebo reference="imu_link_axes0_x_axis">
+    <gravity>true</gravity>
+    <material>Gazebo/RedBright</material>
+    </gazebo>
+    <joint name = "imu_link_joint0_y_axis" type ="fixed">
+      <origin rpy="1.57 0 1.57" xyz="0 0 0"/>
+      <parent link="${arm_id}_link0"/>
+      <child link="imu_link_axes0_y_axis"/>
+      <axis xyz="0 0 0"/>
+    </joint>
+    <link name="imu_link_axes0_y_axis">
+      <inertial>
+        <origin xyz="0 0 0" rpy="0 0 0"/>
+        <mass value="0.0"/>
+        <inertia ixx="0.0" ixy="0.0" ixz="0.0" iyy="0.0" iyz="0.0" izz="0.0"/>
+      </inertial>
+      <visual>
+        <origin xyz="0.0 0.05 0.06" rpy="-1.57 0 0" />
+          <geometry>
+            <mesh scale="0.007 0.007 0.007" filename="package://${axes_meshes}/meshes/visual/arrow.dae"/>
+          </geometry>
+        </visual>
+    </link>
+    <gazebo reference="imu_link_axes0_y_axis">
+    <gravity>true</gravity>
+    <material>Gazebo/Green</material>
+    </gazebo>
+    <joint name = "imu_link_joint0_z_axis" type ="fixed">
+      <origin rpy="1.57 0 1.57" xyz="0 0 0"/>
+      <parent link="${arm_id}_link0"/>
+      <child link="imu_link_axes0_z_axis"/>
+      <axis xyz="0 0 0"/>
+    </joint>
+    <link name="imu_link_axes0_z_axis">
+      <inertial>
+        <origin xyz="0 0 0" rpy="0 0 0"/>
+        <mass value="0.0"/>
+        <inertia ixx="0.0" ixy="0.0" ixz="0.0" iyy="0.0" iyz="0.0" izz="0.0"/>
+      </inertial>
+      <visual>
+        <origin xyz="0.0 0.05 0.06" rpy="0 0 1.57" />
+          <geometry>
+            <mesh scale="0.007 0.007 0.007" filename="package://${axes_meshes}/meshes/visual/arrow.dae"/>
+          </geometry>
+        </visual>
+    </link>
+    <gazebo reference="imu_link_axes0_z_axis">
+    <gravity>true</gravity>
+    <material>Gazebo/Blue</material>
+    </gazebo>
+    <joint name = "imu_link_joint1_x_axis" type ="fixed">
+      <origin rpy="1.57 0 1.57" xyz="0 0 0"/>
+      <parent link="${arm_id}_link1"/>
+      <child link="imu_link_axes1_x_axis"/>
+      <axis xyz="0 0 0"/>
+    </joint>
+    <link name="imu_link_axes1_x_axis">
+      <inertial>
+        <origin xyz="0 0 0" rpy="0 0 0"/>
+        <mass value="0.0"/>
+        <inertia ixx="0.0" ixy="0.0" ixz="0.0" iyy="0.0" iyz="0.0" izz="0.0"/>
+      </inertial>
+      <visual>
+        <origin xyz="0.0 -0.15 0.06" rpy="0 1.57 0" />
+          <geometry>
+            <mesh scale="0.007 0.007 0.007" filename="package://${axes_meshes}/meshes/visual/arrow.dae"/>
+          </geometry>
+        </visual>
+    </link>
+    <gazebo reference="imu_link_axes1_x_axis">
+    <gravity>true</gravity>
+    <material>Gazebo/RedBright</material>
+    </gazebo>
+    <joint name = "imu_link_joint1_y_axis" type ="fixed">
+      <origin rpy="1.57 0 1.57" xyz="0 0 0"/>
+      <parent link="${arm_id}_link1"/>
+      <child link="imu_link_axes1_y_axis"/>
+      <axis xyz="0 0 0"/>
+    </joint>
+    <link name="imu_link_axes1_y_axis">
+      <inertial>
+        <origin xyz="0 0 0" rpy="0 0 0"/>
+        <mass value="0.0"/>
+        <inertia ixx="0.0" ixy="0.0" ixz="0.0" iyy="0.0" iyz="0.0" izz="0.0"/>
+      </inertial>
+      <visual>
+        <origin xyz="0.0 -0.15 0.06" rpy="-1.57 0 0" />
+          <geometry>
+            <mesh scale="0.007 0.007 0.007" filename="package://${axes_meshes}/meshes/visual/arrow.dae"/>
+          </geometry>
+        </visual>
+    </link>
+    <gazebo reference="imu_link_axes1_y_axis">
+    <gravity>true</gravity>
+    <material>Gazebo/Green</material>
+    </gazebo>
+    <joint name = "imu_link_joint1_z_axis" type ="fixed">
+      <origin rpy="1.57 0 1.57" xyz="0 0 0"/>
+      <parent link="${arm_id}_link1"/>
+      <child link="imu_link_axes1_z_axis"/>
+      <axis xyz="0 0 0"/>
+    </joint>
+    <link name="imu_link_axes1_z_axis">
+      <inertial>
+        <origin xyz="0 0 0" rpy="0 0 0"/>
+        <mass value="0.0"/>
+        <inertia ixx="0.0" ixy="0.0" ixz="0.0" iyy="0.0" iyz="0.0" izz="0.0"/>
+      </inertial>
+      <visual>
+        <origin xyz="0.0 -0.15 0.06" rpy="0 0 1.57" />
+          <geometry>
+            <mesh scale="0.007 0.007 0.007" filename="package://${axes_meshes}/meshes/visual/arrow.dae"/>
+          </geometry>
+        </visual>
+    </link>
+    <gazebo reference="imu_link_axes1_z_axis">
+    <gravity>true</gravity>
+    <material>Gazebo/Blue</material>
+    </gazebo>
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
Commit message: fix to xacro with collision

File: robots/panda_arm.xacro (robot description, xacro)
@@ -25,4 +25,5 @@
       </visual>
       <collision>
+        <origin rpy="0 0 0" xyz="0 0 0.035"/>
         <geometry>
           <mesh filename="package://${description_pkg}/meshes/collision/link0.stl"/>
@@ -44,4 +45,5 @@
       </visual>
       <collision>
+        <origin rpy="0 0 0" xyz="0 0 0.035"/>
         <geometry>
           <mesh filename="package://${description_pkg}/meshes/collision/link1.stl"/>
@@ -74,4 +76,5 @@
       </visual>
       <collision>
+        <origin rpy="0 0 0" xyz="0 0 0.035"/>
         <geometry>
           <mesh filename="package://${description_pkg}/meshes/collision/link2.stl"/>
@@ -104,4 +107,5 @@
       </visual>
       <collision>
+        <origin rpy="0 0 0" xyz="0 0 0.035"/>
         <geometry>
           <mesh filename="package://${description_pkg}/meshes/collision/link3.stl"/>
@@ -134,4 +138,5 @@
       </visual>
       <collision>
+        <origin rpy="0 0 0" xyz="0 0 0.035"/>
         <geometry>
           <mesh filename="package://${description_pkg}/meshes/collision/link4.stl"/>
@@ -164,4 +169,5 @@
       </visual>
       <collision>
+        <origin rpy="0 0 0" xyz="0 0 0.035"/>
         <geometry>
           <mesh filename="package://${description_pkg}/meshes/collision/link5.stl"/>
@@ -194,4 +200,5 @@
       </visual>
       <collision>
+        <origin rpy="0 0 0" xyz="0 0 0.035"/>
         <geometry>
           <mesh filename="package://${description_pkg}/meshes/collision/link6.stl"/>
@@ -224,4 +231,5 @@
       </visual>
       <collision>
+        <origin rpy="0 0 0" xyz="0 0 0.035"/>
         <geometry>
           <mesh filename="package://${description_pkg}/meshes/collision/link7.stl"/>
