Commit message: Cover body with proximity sensors

File: robots/panda_arm_hand_flacco.urdf.xacro (robot description, xacro)
@@ -23,8 +23,139 @@
   <xacro:end_effector/>
   <!-- Proximity sensors -->
-  <xacro:proximity proximity_id="0" radius="0.06" theta="${2*pi/4 * 0}" z0="-0.16" connected_to="panda_link3"/>
-  <xacro:proximity proximity_id="1" radius="0.06" theta="${2*pi/4 * 1}" z0="-0.16" connected_to="panda_link3"/>
-  <xacro:proximity proximity_id="2" radius="0.06" theta="${2*pi/4 * 2}" z0="-0.16" connected_to="panda_link3"/>
-  <xacro:proximity proximity_id="3" radius="0.06" theta="${2*pi/4 * 3}" z0="-0.16" connected_to="panda_link3"/>
+  <!-- panda_link1 -->
+  <xacro:property name="ring_id" value="30"/>
+  <xacro:property name="radius" value="0.06"/>
+  <xacro:property name="z0" value="-0.185"/>
+  <xacro:property name="connected_to" value="panda_link1"/>
+  <xacro:proximity proximity_id="${8*ring_id+0}" radius="${radius}" theta="${2*pi/8 * 0}" z0="${z0}" connected_to="${connected_to}"/>
+  <xacro:proximity proximity_id="${8*ring_id+1}" radius="${radius}" theta="${2*pi/8 * 1}" z0="${z0}" connected_to="${connected_to}"/>
+  <xacro:proximity proximity_id="${8*ring_id+2}" radius="${radius}" theta="${2*pi/8 * 2}" z0="${z0}" connected_to="${connected_to}"/>
+  <xacro:proximity proximity_id="${8*ring_id+3}" radius="${radius}" theta="${2*pi/8 * 3}" z0="${z0}" connected_to="${connected_to}"/>
+  <xacro:proximity proximity_id="${8*ring_id+4}" radius="${radius}" theta="${2*pi/8 * 4}" z0="${z0}" connected_to="${connected_to}"/>
+  <xacro:proximity proximity_id="${8*ring_id+5}" radius="${radius}" theta="${2*pi/8 * 5}" z0="${z0}" connected_to="${connected_to}"/>
+  <xacro:proximity proximity_id="${8*ring_id+6}" radius="${radius}" theta="${2*pi/8 * 6}" z0="${z0}" connected_to="${connected_to}"/>
+  <xacro:proximity proximity_id="${8*ring_id+7}" radius="${radius}" theta="${2*pi/8 * 7}" z0="${z0}" connected_to="${connected_to}"/>
+  <xacro:property name="ring_id" value="31"/>
+  <xacro:property name="z0" value="-0.14"/>
+  <xacro:proximity proximity_id="${8*ring_id+0}" radius="${radius}" theta="${2*pi/8 * 0}" z0="${z0}" connected_to="${connected_to}"/>
+  <xacro:proximity proximity_id="${8*ring_id+1}" radius="${radius}" theta="${2*pi/8 * 1}" z0="${z0}" connected_to="${connected_to}"/>
+  <xacro:proximity proximity_id="${8*ring_id+2}" radius="${radius}" theta="${2*pi/8 * 2}" z0="${z0}" connected_to="${connected_to}"/>
+  <xacro:proximity proximity_id="${8*ring_id+3}" radius="${radius}" theta="${2*pi/8 * 3}" z0="${z0}" connected_to="${connected_to}"/>
+  <xacro:proximity proximity_id="${8*ring_id+4}" radius="${radius}" theta="${2*pi/8 * 4}" z0="${z0}" connected_to="${connected_to}"/>
+  <xacro:proximity proximity_id="${8*ring_id+5}" radius="${radius}" theta="${2*pi/8 * 5}" z0="${z0}" connected_to="${connected_to}"/>
+  <xacro:proximity proximity_id="${8*ring_id+6}" radius="${radius}" theta="${2*pi/8 * 6}" z0="${z0}" connected_to="${connected_to}"/>
+  <xacro:proximity proximity_id="${8*ring_id+7}" radius="${radius}" theta="${2*pi/8 * 7}" z0="${z0}" connected_to="${connected_to}"/>
+  <!-- panda_link3 -->
+  <xacro:property name="ring_id" value="0"/>
+  <xacro:property name="radius" value="0.06"/>
+  <xacro:property name="z0" value="-0.13"/>
+  <xacro:property name="connected_to" value="panda_link3"/>
+  <xacro:proximity proximity_id="${8*ring_id+0}" radius="${radius}" theta="${2*pi/8 * 0}" z0="${z0}" connected_to="${connected_to}"/>
+  <xacro:proximity proximity_id="${8*ring_id+1}" radius="${radius}" theta="${2*pi/8 * 1}" z0="${z0}" connected_to="${connected_to}"/>
+  <xacro:proximity proximity_id="${8*ring_id+2}" radius="${radius}" theta="${2*pi/8 * 2}" z0="${z0}" connected_to="${connected_to}"/>
+  <xacro:proximity proximity_id="${8*ring_id+3}" radius="${radius}" theta="${2*pi/8 * 3}" z0="${z0}" connected_to="${connected_to}"/>
+  <xacro:proximity proximity_id="${8*ring_id+4}" radius="${radius}" theta="${2*pi/8 * 4}" z0="${z0}" connected_to="${connected_to}"/>
+  <xacro:proximity proximity_id="${8*ring_id+5}" radius="${radius}" theta="${2*pi/8 * 5}" z0="${z0}" connected_to="${connected_to}"/>
+  <xacro:proximity proximity_id="${8*ring_id+6}" radius="${radius}" theta="${2*pi/8 * 6}" z0="${z0}" connected_to="${connected_to}"/>
+  <xacro:proximity proximity_id="${8*ring_id+7}" radius="${radius}" theta="${2*pi/8 * 7}" z0="${z0}" connected_to="${connected_to}"/>
+  <xacro:property name="ring_id" value="10"/>
+  <xacro:property name="z0" value="-0.20"/>
+  <xacro:proximity proximity_id="${8*ring_id+0}" radius="${radius}" theta="${2*pi/8 * 0}" z0="${z0}" connected_to="${connected_to}"/>
+  <xacro:proximity proximity_id="${8*ring_id+1}" radius="${radius}" theta="${2*pi/8 * 1}" z0="${z0}" connected_to="${connected_to}"/>
+  <xacro:proximity proximity_id="${8*ring_id+2}" radius="${radius}" theta="${2*pi/8 * 2}" z0="${z0}" connected_to="${connected_to}"/>
+  <xacro:proximity proximity_id="${8*ring_id+3}" radius="${radius}" theta="${2*pi/8 * 3}" z0="${z0}" connected_to="${connected_to}"/>
+  <xacro:proximity proximity_id="${8*ring_id+4}" radius="${radius}" theta="${2*pi/8 * 4}" z0="${z0}" connected_to="${connected_to}"/>
+  <xacro:proximity proximity_id="${8*ring_id+5}" radius="${radius}" theta="${2*pi/8 * 5}" z0="${z0}" connected_to="${connected_to}"/>
+  <xacro:proximity proximity_id="${8*ring_id+6}" radius="${radius}" theta="${2*pi/8 * 6}" z0="${z0}" connected_to="${connected_to}"/>
+  <xacro:proximity proximity_id="${8*ring_id+7}" radius="${radius}" theta="${2*pi/8 * 7}" z0="${z0}" connected_to="${connected_to}"/>
+  <!-- panda_link4 -->
+  <xacro:property name="ring_id" value="100000"/>
+  <xacro:property name="radius" value="0.05"/>
+  <xacro:property name="z0" value="0.07"/>
+  <xacro:property name="connected_to" value="panda_link4"/>
+  <xacro:proximity proximity_id="${8*ring_id+0}" radius="${radius}" theta="${2*pi/8 * 0}" z0="${z0}" connected_to="${connected_to}"/>
+  <xacro:proximity proximity_id="${8*ring_id+1}" radius="${radius}" theta="${2*pi/8 * 1}" z0="${z0}" connected_to="${connected_to}"/>
+  <xacro:proximity proximity_id="${8*ring_id+2}" radius="${radius}" theta="${2*pi/8 * 2}" z0="${z0}" connected_to="${connected_to}"/>
+  <xacro:proximity proximity_id="${8*ring_id+3}" radius="${radius}" theta="${2*pi/8 * 3}" z0="${z0}" connected_to="${connected_to}"/>
+  <xacro:proximity proximity_id="${8*ring_id+4}" radius="${radius}" theta="${2*pi/8 * 4}" z0="${z0}" connected_to="${connected_to}"/>
+  <xacro:proximity proximity_id="${8*ring_id+5}" radius="${radius}" theta="${2*pi/8 * 5}" z0="${z0}" connected_to="${connected_to}"/>
+  <xacro:proximity proximity_id="${8*ring_id+6}" radius="${radius}" theta="${2*pi/8 * 6}" z0="${z0}" connected_to="${connected_to}"/>
+  <xacro:proximity proximity_id="${8*ring_id+7}" radius="${radius}" theta="${2*pi/8 * 7}" z0="${z0}" connected_to="${connected_to}"/>
+  <xacro:property name="ring_id" value="100100"/>
+  <xacro:property name="radius" value="0.055"/>
+  <xacro:property name="z0" value="-0.085"/>
+  <xacro:property name="connected_to" value="panda_link4"/>
+  <xacro:proximity proximity_id="${8*ring_id+0}" radius="${radius}" theta="${2*pi/8 * 0}" z0="${z0}" connected_to="${connected_to}"/>
+  <xacro:proximity proximity_id="${8*ring_id+1}" radius="${radius}" theta="${2*pi/8 * 1}" z0="${z0}" connected_to="${connected_to}"/>
+  <xacro:proximity proximity_id="${8*ring_id+2}" radius="${radius}" theta="${2*pi/8 * 2}" z0="${z0}" connected_to="${connected_to}"/>
+  <xacro:proximity proximity_id="${8*ring_id+3}" radius="${radius}" theta="${2*pi/8 * 3}" z0="${z0}" connected_to="${connected_to}"/>
+  <xacro:proximity proximity_id="${8*ring_id+4}" radius="${radius}" theta="${2*pi/8 * 4}" z0="${z0}" connected_to="${connected_to}"/>
+  <xacro:proximity proximity_id="${8*ring_id+5}" radius="${radius}" theta="${2*pi/8 * 5}" z0="${z0}" connected_to="${connected_to}"/>
+  <xacro:proximity proximity_id="${8*ring_id+6}" radius="${radius}" theta="${2*pi/8 * 6}" z0="${z0}" connected_to="${connected_to}"/>
+  <xacro:proximity proximity_id="${8*ring_id+7}" radius="${radius}" theta="${2*pi/8 * 7}" z0="${z0}" connected_to="${connected_to}"/>
+  <!-- panda_link5 -->
+  <xacro:property name="ring_id" value="1"/>
+  <xacro:property name="radius" value="0.06"/>
+  <xacro:property name="z0" value="-0.24"/>
+  <xacro:property name="connected_to" value="panda_link5"/>
+  <xacro:proximity proximity_id="${8*ring_id+0}" radius="${radius}" theta="${2*pi/8 * 0}" z0="${z0}" connected_to="${connected_to}"/>
+  <xacro:proximity proximity_id="${8*ring_id+1}" radius="${radius}" theta="${2*pi/8 * 1}" z0="${z0}" connected_to="${connected_to}"/>
+  <xacro:proximity proximity_id="${8*ring_id+2}" radius="${radius}" theta="${2*pi/8 * 2}" z0="${z0}" connected_to="${connected_to}"/>
+  <xacro:proximity proximity_id="${8*ring_id+3}" radius="${radius}" theta="${2*pi/8 * 3}" z0="${z0}" connected_to="${connected_to}"/>
+  <xacro:proximity proximity_id="${8*ring_id+4}" radius="${radius}" theta="${2*pi/8 * 4}" z0="${z0}" connected_to="${connected_to}"/>
+  <xacro:proximity proximity_id="${8*ring_id+5}" radius="${radius}" theta="${2*pi/8 * 5}" z0="${z0}" connected_to="${connected_to}"/>
+  <xacro:proximity proximity_id="${8*ring_id+6}" radius="${radius}" theta="${2*pi/8 * 6}" z0="${z0}" connected_to="${connected_to}"/>
+  <xacro:proximity proximity_id="${8*ring_id+7}" radius="${radius}" theta="${2*pi/8 * 7}" z0="${z0}" connected_to="${connected_to}"/>
+  <xacro:property name="ring_id" value="2"/>
+  <xacro:property name="z0" value="-0.30"/>
+  <xacro:proximity proximity_id="${8*ring_id+0}" radius="${radius}" theta="${2*pi/8 * 0}" z0="${z0}" connected_to="${connected_to}"/>
+  <xacro:proximity proximity_id="${8*ring_id+1}" radius="${radius}" theta="${2*pi/8 * 1}" z0="${z0}" connected_to="${connected_to}"/>
+  <xacro:proximity proximity_id="${8*ring_id+2}" radius="${radius}" theta="${2*pi/8 * 2}" z0="${z0}" connected_to="${connected_to}"/>
+  <xacro:proximity proximity_id="${8*ring_id+3}" radius="${radius}" theta="${2*pi/8 * 3}" z0="${z0}" connected_to="${connected_to}"/>
+  <xacro:proximity proximity_id="${8*ring_id+4}" radius="${radius}" theta="${2*pi/8 * 4}" z0="${z0}" connected_to="${connected_to}"/>
+  <xacro:proximity proximity_id="${8*ring_id+5}" radius="${radius}" theta="${2*pi/8 * 5}" z0="${z0}" connected_to="${connected_to}"/>
+  <xacro:proximity proximity_id="${8*ring_id+6}" radius="${radius}" theta="${2*pi/8 * 6}" z0="${z0}" connected_to="${connected_to}"/>
+  <xacro:proximity proximity_id="${8*ring_id+7}" radius="${radius}" theta="${2*pi/8 * 7}" z0="${z0}" connected_to="${connected_to}"/>
+  <!-- panda_link7 -->
+  <xacro:property name="ring_id" value="100"/>
+  <xacro:property name="radius" value="0.0425"/>
+  <xacro:property name="z0" value="0"/>
+  <xacro:property name="connected_to" value="panda_link7"/>
+  <xacro:proximity proximity_id="${8*ring_id+0}" radius="${radius}" theta="${2*pi/8 * 0}" z0="${z0}" connected_to="${connected_to}"/>
+  <xacro:proximity proximity_id="${8*ring_id+1}" radius="${radius}" theta="${2*pi/8 * 1}" z0="${z0}" connected_to="${connected_to}"/>
+  <xacro:proximity proximity_id="${8*ring_id+2}" radius="${radius}" theta="${2*pi/8 * 2}" z0="${z0}" connected_to="${connected_to}"/>
+  <xacro:proximity proximity_id="${8*ring_id+3}" radius="${radius}" theta="${2*pi/8 * 3}" z0="${z0}" connected_to="${connected_to}"/>
+  <xacro:proximity proximity_id="${8*ring_id+4}" radius="${radius}" theta="${2*pi/8 * 4}" z0="${z0}" connected_to="${connected_to}"/>
+  <xacro:property name="ring_id" value="101"/>
+  <xacro:property name="radius" value="0.0425"/>
+  <xacro:property name="z0" value="-0.05"/>
+  <xacro:property name="connected_to" value="panda_link7"/>
+  <xacro:proximity proximity_id="${8*ring_id+0}" radius="${radius}" theta="${2*pi/8 * 0}" z0="${z0}" connected_to="${connected_to}"/>
+  <xacro:proximity proximity_id="${8*ring_id+1}" radius="${radius}" theta="${2*pi/8 * 1}" z0="${z0}" connected_to="${connected_to}"/>
+  <xacro:proximity proximity_id="${8*ring_id+2}" radius="${radius}" theta="${2*pi/8 * 2}" z0="${z0}" connected_to="${connected_to}"/>
+  <xacro:proximity proximity_id="${8*ring_id+3}" radius="${radius}" theta="${2*pi/8 * 3}" z0="${z0}" connected_to="${connected_to}"/>
+  <xacro:proximity proximity_id="${8*ring_id+4}" radius="${radius}" theta="${2*pi/8 * 4}" z0="${z0}" connected_to="${connected_to}"/>
+  <!-- panda_hand -->
+  <xacro:property name="ring_id" value="102"/>
+  <xacro:property name="radius" value="0.10"/>
+  <xacro:property name="z0" value="0.03"/>
+  <xacro:property name="connected_to" value="panda_hand"/>
+  <xacro:proximity proximity_id="${8*ring_id+0}" radius="${radius}" theta="${2*pi/8 * 0}" z0="${z0}" connected_to="${connected_to}"/>
+  <xacro:proximity proximity_id="${8*ring_id+8}" radius="${radius}" theta="${2*pi/8 * 4}" z0="${z0}" connected_to="${connected_to}"/>
+  <xacro:property name="radius" value="0.025"/>
+  <xacro:proximity proximity_id="${8*ring_id+1}" radius="${radius}" theta="${2*pi/8 * 2}" z0="${z0}" y0="-0.09" connected_to="${connected_to}"/>
+  <xacro:proximity proximity_id="${8*ring_id+2}" radius="${radius}" theta="${2*pi/8 * 2}" z0="${z0}" y0="-0.06" connected_to="${connected_to}"/>
+  <xacro:proximity proximity_id="${8*ring_id+3}" radius="${radius}" theta="${2*pi/8 * 2}" z0="${z0}" y0="-0.03" connected_to="${connected_to}"/>
+  <xacro:proximity proximity_id="${8*ring_id+4}" radius="${radius}" theta="${2*pi/8 * 2}" z0="${z0}" y0="0" connected_to="${connected_to}"/>
+  <xacro:proximity proximity_id="${8*ring_id+5}" radius="${radius}" theta="${2*pi/8 * 2}" z0="${z0}" y0="0.03" connected_to="${connected_to}"/>
+  <xacro:proximity proximity_id="${8*ring_id+6}" radius="${radius}" theta="${2*pi/8 * 2}" z0="${z0}" y0="0.06" connected_to="${connected_to}"/>
+  <xacro:proximity proximity_id="${8*ring_id+7}" radius="${radius}" theta="${2*pi/8 * 2}" z0="${z0}" y0="0.09" connected_to="${connected_to}"/>
+  <xacro:proximity proximity_id="${8*ring_id+8+1}" radius="${radius}" theta="${2*pi/8 * 6}" z0="${z0}" y0="-0.09" connected_to="${connected_to}"/>
+  <xacro:proximity proximity_id="${8*ring_id+8+2}" radius="${radius}" theta="${2*pi/8 * 6}" z0="${z0}" y0="-0.06" connected_to="${connected_to}"/>
+  <xacro:proximity proximity_id="${8*ring_id+8+3}" radius="${radius}" theta="${2*pi/8 * 6}" z0="${z0}" y0="-0.03" connected_to="${connected_to}"/>
+  <xacro:proximity proximity_id="${8*ring_id+8+4}" radius="${radius}" theta="${2*pi/8 * 6}" z0="${z0}" y0="0" connected_to="${connected_to}"/>
+  <xacro:proximity proximity_id="${8*ring_id+8+5}" radius="${radius}" theta="${2*pi/8 * 6}" z0="${z0}" y0="0.03" connected_to="${connected_to}"/>
+  <xacro:proximity proximity_id="${8*ring_id+8+6}" radius="${radius}" theta="${2*pi/8 * 6}" z0="${z0}" y0="0.06" connected_to="${connected_to}"/>
+  <xacro:proximity proximity_id="${8*ring_id+8+7}" radius="${radius}" theta="${2*pi/8 * 6}" z0="${z0}" y0="0.09" connected_to="${connected_to}"/>
   <!-- for simulation -->
   <xacro:arg name="robot_name" default="panda"/>

File: robots/proximity.xacro (robot description, xacro)
@@ -1,10 +1,10 @@
 <?xml version='1.0' encoding='utf-8'?>
 <robot xmlns:xacro="http://www.ros.org/wiki/xacro" name="proximity">
-    <xacro:macro name="proximity" params="proximity_id:='0' radius:='0.2' theta:='0.0' z0:='0' type:='fixed' freq:='100' connected_to:=''">
+    <xacro:macro name="proximity" params="proximity_id:='0' radius:=0.2 theta:=0.0 z0:=0 type:='fixed' freq:='100' connected_to:='' x0:=0.0 y0:=0.0">
         <!-- Connect proximity sensor to ${connected_to} -->
         <joint name="proximity${proximity_id}_to_${connected_to}" type="${type}">
             <parent link="${connected_to}"/>
             <child link="proximity_link${proximity_id}"/>
-            <origin xyz="${radius*sin(theta)} ${radius*cos(theta)} ${z0}" rpy=" 0 0 ${pi/2 -theta}" />
+            <origin xyz="${x0+radius*sin(theta)} ${y0+radius*cos(theta)} ${z0}" rpy=" 0 0 ${pi/2 -theta}" />
         </joint>
         <!-- Box that represents sensor -->
@@ -38,6 +38,6 @@
                     </scan>
                     <range>
-                        <min>0.05</min>
-                        <max>1.2</max>
+                        <min>0.02</min>
+                        <max>2.0</max>
                         <resolution>0.01</resolution>
                     </range>
