Commit message: sensor name bug fix and x axis pointing outwards

File: robots/proximity.xacro (robot description, xacro)
@@ -6,9 +6,7 @@
             <parent link="${connected_to}"/>
             <child link="proximity_link${proximity_id}"/>
-            <origin xyz="${radius*sin(theta)} ${radius*cos(theta)} ${z0}" rpy="${-pi/2} 0 ${-theta}" />
+            <origin xyz="${radius*sin(theta)} ${radius*cos(theta)} ${z0}" rpy=" 0 0 ${pi/2 -theta}" />
         </joint>
         <!-- Box that represents sensor -->
-        <xacro:property name="boxxy" value="0.02"/>
-        <xacro:property name="boxz" value="0.001"/>
         <link name="proximity_link${proximity_id}">
             <inertial>
@@ -18,7 +16,7 @@
             </inertial>
             <visual>
-                <origin xyz="0 0 0" rpy="0 0 0"/>
+                <origin xyz="0 0 0.01" rpy="0 0 0"/>
                 <geometry>
-                    <box size="${boxxy} ${boxxy} ${boxz}"/>
+                    <box size="0.01 0.03 0.03"/>
                 </geometry>
             </visual>
@@ -26,8 +24,8 @@
         <gazebo reference="proximity_link${proximity_id}">
             <material>Gazebo/YellowGlow</material>
-            <sensor type="ray" name="proximity_sensor">
-                <pose>0 0 0 0 ${-pi/2} 0</pose>
+            <sensor type="ray" name="proximity_sensor${proximity_id}">
+                <pose>0 0 0 0 0 0</pose>
                 <visualize>true</visualize>
-                <update_rate>30</update_rate>
+                <update_rate>${freq}</update_rate>
                 <ray>
                     <scan>
@@ -44,15 +42,6 @@
                         <resolution>0.01</resolution>
                     </range>
-                    <noise>
-                        <type>gaussian</type>
-                        <!-- Noise parameters based on published spec for Hokuyo laser
-                            achieving "+-30mm" accuracy at range < 10m.  A mean of 0.0m and
-                            stddev of 0.01m will put 99.7% of samples within 0.03m of the true
-                            reading. -->
-                        <mean>0.0</mean>
-                        <stddev>0.01</stddev>
-                    </noise>
                 </ray>
-                <plugin filename="libgazebo_ros_laser.so" name="proximity_plugin">
+                <plugin filename="libgazebo_ros_laser.so" name="proximity_plugin${proximity_id}">
                     <topicName>proximity_data${proximity_id}</topicName>
                     <bodyName>proximity_link${proximity_id}</bodyName>

Commit message: Testing the listener efficiency

File: robots/proximity.xacro (robot description, xacro)
@@ -1,5 +1,6 @@
 <?xml version='1.0' encoding='utf-8'?>
 <robot xmlns:xacro="http://www.ros.org/wiki/xacro" name="proximity">
-    <xacro:macro name="proximity" params="proximity_id:='0' radius:=0.2 theta:=0.0 z0:=0 type:='fixed' freq:='100' connected_to:='' x0:=0.0 y0:=0.0">
+    <xacro:macro name="proximity" params="proximity_id:='0' radius:=0.2 theta:=0.0 z0:=0 type:='fixed' connected_to:='' x0:=0.0 y0:=0.0">
+        <xacro:property name="freq" value="100.0"/>
         <!-- Connect proximity sensor to ${connected_to} -->
         <joint name="proximity${proximity_id}_to_${connected_to}" type="${type}">
