Commit message: simplified imu.xacro

File: robots/imu.xacro (robot description, xacro)
@@ -1,12 +1,24 @@
 <?xml version='1.0' encoding='utf-8'?>
 <robot xmlns:xacro="http://www.ros.org/wiki/xacro" name="imu">
-    <xacro:macro name="imu" params="imu_id:='0' xyz:='0 0 0' rpy:='0 0 0' boxxy:='0.02 0.02' boxz:='0.01'">
-        <joint name="imu_to_world${imu_id}" type="floating">
-            <parent link="world" />
-            <child link="imu_link${imu_id}" />
-            <!-- XYZ, RPY from parent Visual Origin (Center o Gravity) -->
-            <!-- in this case it's 0 0 0-->
-            <origin xyz="${xyz}" rpy="${rpy}"/>
-        </joint>
+    <xacro:macro name="imu" params="imu_id:='0' xyz:='0 0 0' rpy:='0 0 0' boxxy:='0.05 0.05' boxz:='0.03' gravity:='false' type:='floating' freq:='50' connected_to:=''">
+        <!-- Connect IMU to the world if not specified -->
+        <xacro:if value="${connected_to == ''}">
+            <joint name="imu${imu_id}_to_world" type="${type}">
+                <!-- XYZ, RPY from parent Visual Origin (Center o Gravity) -->
+                <!-- in this case it's 0 0 0-->
+                <parent link="world" />
+                <child link="imu_link${imu_id}" />
+                <origin rpy="${rpy}" xyz="${xyz}"/>
+            </joint>
+        </xacro:if>
+        <!-- Connect IMU to ${connected_to} if specified -->
+        <xacro:if value="${connected_to != ''}">
+            <joint name="imu${imu_id}_to_${connected_to}" type="${type}">
+                <parent link="${connected_to}"/>
+                <child link="imu_link${imu_id}"/>
+                <origin rpy="${rpy}" xyz="${xyz}"/>
+                <!-- <dynamics damping="100" friction="100"/> -->
+            </joint>
+        </xacro:if>
         <!-- XYZ, RPY from the joint-->
         <!-- in this case it's imu_to_world${imu_id}-->
@@ -17,5 +29,5 @@
             <inertial>
                 <origin xyz="0 0 ${displacement/2}" rpy="0 0 0"/>
-                <mass value="0.01"/>
+                <mass value="0.1"/>
                 <inertia ixx="0.0" ixy="0.0" ixz="0.0" iyy="0.0" iyz="0.0" izz="0.0"/>
             </inertial>
@@ -28,15 +40,18 @@
         </link>
         <gazebo reference="imu_link${imu_id}">
-            <material>Gazebo/White</material>
-            <gravity>false</gravity>
+            <material>Gazebo/YellowGlow</material>
+            <gravity>${gravity}</gravity>
             <sensor name="imu_sensor${imu_id}" type="imu">
             <always_on>true</always_on>
-            <update_rate>100</update_rate>
+            <update_rate>${freq}</update_rate>
             <visualize>true</visualize>
             <topic>imu_data${imu_id}</topic>
+            <!-- <cfmDamping>true</cfmDamping> -->
+            <!-- <kp>10000</kp> -->
+            <!-- <kd>100</kd> -->
             <plugin filename="libgazebo_ros_imu_sensor.so" name="imu_plugin">
                 <topicName>imu_data${imu_id}</topicName>
                 <bodyName>imu_link${imu_id}</bodyName>
-                <updateRateHZ>100.0</updateRateHZ>
+                <updateRateHZ>${freq}</updateRateHZ>
                 <gaussianNoise>0.0</gaussianNoise>
                 <xyzOffset>0.0 0.0 0.0</xyzOffset>

File: robots/panda_arm.xacro (robot description, xacro)
@@ -262,767 +262,4 @@
       <axis xyz="0 0 0"/>
     </joint>
-    <joint name = "imu_link_joint0" type ="fixed">
-          <origin rpy="1.57 0 1.57" xyz="0 0 0"/>
-          <parent link="${arm_id}_link0"/>
-          <child link="imu_link0"/>
-          <axis xyz="0 0 0"/>
-    </joint>
-    <link name="imu_link0">
-        <inertial>
-            <origin xyz="0 0 0" rpy="0 0 0"/>
-            <mass value="0.0"/>
-            <inertia ixx="0.0" ixy="0.0" ixz="0.0" iyy="0.0" iyz="0.0" izz="0.0"/>
-        </inertial>
-        <visual>
-            <origin xyz="0.0 0.05 0.06" rpy="1.57 0 1.57" />
-            <geometry>
-                <box size = "0.05 0.05 0.05"/>
-            </geometry>
-        </visual>
-    </link>
-    <gazebo reference="imu_link0">
-        <gravity>true</gravity>
-        <!--      Below is the line to change the material-->
-        <material>Gazebo/YellowGlow</material>
-        <sensor name="imu_sensor0" type="imu">
-          <always_on>true</always_on>
-          <update_rate>100</update_rate>
-          <visualize>true</visualize>
-          <topic>imu_data0</topic>
-          <plugin filename="libgazebo_ros_imu_sensor.so" name="imu_plugin">
-            <topicName>imu_data0</topicName>
-            <bodyName>imu_link0</bodyName>
-            <updateRateHZ>100.0</updateRateHZ>
-            <gaussianNoise>0.0</gaussianNoise>
-            <xyzOffset>0.0 0.05 0.06</xyzOffset>
-            <rpyOffset>1.57 0 1.57</rpyOffset>
-            <frameName>imu_link0</frameName>
-          </plugin>
-          <pose>0 0 0 0 0 0</pose>
-        </sensor>
-    </gazebo>
-    <joint name = "imu_link_joint1" type ="fixed">
-          <origin rpy="1.57 0 1.57" xyz="0 0 0"/>
-          <parent link="${arm_id}_link1"/>
-          <child link="imu_link1"/>
-          <axis xyz="0 0 0"/>
-    </joint>
-    <link name="imu_link1">
-        <inertial>
-            <origin xyz="0 0 0" rpy="0 0 0"/>
-            <mass value="0.0"/>
-            <inertia ixx="0.0" ixy="0.0" ixz="0.0" iyy="0.0" iyz="0.0" izz="0.0"/>
-        </inertial>
-        <visual>
-            <origin xyz="0.0 -0.15 0.06" rpy="1.57 0 1.57" />
-            <geometry>
-                <box size = "0.05 0.05 0.05"/>
-            </geometry>
-        </visual>
-    </link>
-    <gazebo reference="imu_link1">
-        <gravity>true</gravity>
-        <!--      Below is the line to change the material-->
-        <material>Gazebo/YellowGlow</material>
-        <sensor name="imu_sensor1" type="imu">
-          <always_on>true</always_on>
-          <update_rate>100</update_rate>
-          <visualize>true</visualize>
-          <topic>imu_data0</topic>
-          <plugin filename="libgazebo_ros_imu_sensor.so" name="imu_plugin">
-            <topicName>imu_data1</topicName>
-            <bodyName>imu_link1</bodyName>
-            <updateRateHZ>100.0</updateRateHZ>
-            <gaussianNoise>0.0</gaussianNoise>
-            <xyzOffset>0.0 -0.15 0.06</xyzOffset>
-            <rpyOffset>1.57 0 1.57</rpyOffset>
-            <frameName>imu_link1</frameName>
-          </plugin>
-          <pose>0 0 0 0 0 0</pose>
-        </sensor>
-    </gazebo>
-    <joint name = "imu_link_joint2" type ="fixed">
-          <origin rpy="3.14 -1.57 0" xyz="0 0 0"/>
-          <parent link="${arm_id}_link2"/>
-          <child link="imu_link2"/>
-          <axis xyz="0 0 0"/>
-    </joint>
-    <link name="imu_link2">
-        <inertial>
-            <origin xyz="0 0 0" rpy="0 0 0"/>
-            <mass value="0.0"/>
-            <inertia ixx="0.0" ixy="0.0" ixz="0.0" iyy="0.0" iyz="0.0" izz="0.0"/>
-        </inertial>
-        <visual>
-            <origin xyz="0.0 0.15 0.06" rpy="3.14 -1.57 0" />
-            <geometry>
-                <box size = "0.05 0.05 0.05"/>
-            </geometry>
-        </visual>
-    </link>
-    <gazebo reference="imu_link2">
-        <gravity>true</gravity>
-        <!--      Below is the line to change the material-->
-        <material>Gazebo/YellowGlow</material>
-        <sensor name="imu_sensor2" type="imu">
-          <always_on>true</always_on>
-          <update_rate>100</update_rate>
-          <visualize>true</visualize>
-          <topic>imu_data0</topic>
-          <plugin filename="libgazebo_ros_imu_sensor.so" name="imu_plugin">
-            <topicName>imu_data2</topicName>
-            <bodyName>imu_link2</bodyName>
-            <updateRateHZ>100.0</updateRateHZ>
-            <gaussianNoise>0.0</gaussianNoise>
-            <xyzOffset>0.0 0.15 0.06</xyzOffset>
-            <rpyOffset>3.14 -1.57 0</rpyOffset>
-            <frameName>imu_link2</frameName>
-          </plugin>
-          <pose>0 0 0 0 0 0</pose>
-        </sensor>
-    </gazebo>
-    <joint name = "imu_link_joint3" type ="fixed">
-          <origin rpy="0 -1.57 0" xyz="0 0 0"/>
-          <parent link="${arm_id}_link3"/>
-          <child link="imu_link3"/>
-          <axis xyz="0 0 0"/>
-    </joint>
-    <link name="imu_link3">
-        <inertial>
-            <origin xyz="0 0 0" rpy="0 0 0"/>
-            <mass value="0.0"/>
-            <inertia ixx="0.0" ixy="0.0" ixz="0.0" iyy="0.0" iyz="0.0" izz="0.0"/>
-        </inertial>
-        <visual>
-            <origin xyz="-0.06 0.0 0.06" rpy="0 -1.57 0" />
-            <geometry>
-                <box size = "0.05 0.05 0.05"/>
-            </geometry>
-        </visual>
-    </link>
-    <gazebo reference="imu_link3">
-        <gravity>true</gravity>
-        <!--      Below is the line to change the material-->
-        <material>Gazebo/YellowGlow</material>
-        <sensor name="imu_sensor3" type="imu">
-          <always_on>true</always_on>
-          <update_rate>100</update_rate>
-          <visualize>true</visualize>
-          <topic>imu_data0</topic>
-          <plugin filename="libgazebo_ros_imu_sensor.so" name="imu_plugin">
-            <topicName>imu_data3</topicName>
-            <bodyName>imu_link3</bodyName>
-            <updateRateHZ>100.0</updateRateHZ>
-            <gaussianNoise>0.0</gaussianNoise>
-            <xyzOffset>-0.06 0.0 0.06</xyzOffset>
-            <rpyOffset>0 -1.57 0</rpyOffset>
-            <frameName>imu_link3</frameName>
-          </plugin>
-          <pose>0 0 0 0 0 0</pose>
-        </sensor>
-    </gazebo>
-    <joint name = "imu_link_joint4" type ="fixed">
-          <origin rpy="0 -1.57 0" xyz="0 0 0"/>
-          <parent link="${arm_id}_link4"/>
-          <child link="imu_link4"/>
-          <axis xyz="0 0 0"/>
-    </joint>
-    <link name="imu_link4">
-        <inertial>
-            <origin xyz="0 0 0" rpy="0 0 0"/>
-            <mass value="0.0"/>
-            <inertia ixx="0.0" ixy="0.0" ixz="0.0" iyy="0.0" iyz="0.0" izz="0.0"/>
-        </inertial>
-        <visual>
-            <origin xyz="0.0 0.09 0.14" rpy="0 -1.57 0" />
-            <geometry>
-                <box size = "0.05 0.05 0.05"/>
-            </geometry>
-        </visual>
-    </link>
-    <gazebo reference="imu_link4">
-        <gravity>true</gravity>
-        <!--      Below is the line to change the material-->
-        <material>Gazebo/YellowGlow</material>
-        <sensor name="imu_sensor4" type="imu">
-          <always_on>true</always_on>
-          <update_rate>100</update_rate>
-          <visualize>true</visualize>
-          <topic>imu_data0</topic>
-          <plugin filename="libgazebo_ros_imu_sensor.so" name="imu_plugin">
-            <topicName>imu_data4</topicName>
-            <bodyName>imu_link4</bodyName>
-            <updateRateHZ>100.0</updateRateHZ>
-            <gaussianNoise>0.0</gaussianNoise>
-            <xyzOffset>0.0 0.09 0.14</xyzOffset>
-            <rpyOffset>0 -1.57 0</rpyOffset>
-            <frameName>imu_link4</frameName>
-          </plugin>
-          <pose>0 0 0 0 0 0</pose>
-        </sensor>
-    </gazebo>
-    <joint name = "imu_link_joint5" type ="fixed">
-          <origin rpy="-1.57 3.14 0" xyz="0 0 0"/>
-          <parent link="${arm_id}_link5"/>
-          <child link="imu_link5"/>
-          <axis xyz="0 0 0"/>
-    </joint>
-    <link name="imu_link5">
-        <inertial>
-            <origin xyz="0 0 0" rpy="0 0 0"/>
-            <mass value="0.0"/>
-            <inertia ixx="0.0" ixy="0.0" ixz="0.0" iyy="0.0" iyz="0.0" izz="0.0"/>
-        </inertial>
-        <visual>
-            <origin xyz="0.0 -0.11 0.1" rpy="-1.57 3.14 0" />
-            <geometry>
-                <box size = "0.05 0.05 0.05"/>
-            </geometry>
-        </visual>
-    </link>
-    <gazebo reference="imu_link5">
-        <gravity>true</gravity>
-        <!--      Below is the line to change the material-->
-        <material>Gazebo/YellowGlow</material>
-        <sensor name="imu_sensor5" type="imu">
-          <always_on>true</always_on>
-          <update_rate>100</update_rate>
-          <visualize>true</visualize>
-          <topic>imu_data0</topic>
-          <plugin filename="libgazebo_ros_imu_sensor.so" name="imu_plugin">
-            <topicName>imu_data5</topicName>
-            <bodyName>imu_link5</bodyName>
-            <updateRateHZ>100.0</updateRateHZ>
-            <gaussianNoise>0.0</gaussianNoise>
-            <xyzOffset>0.0 -0.11 0.1</xyzOffset>
-            <rpyOffset>-1.57 3.14 0</rpyOffset>
-            <frameName>imu_link5</frameName>
-          </plugin>
-          <pose>0 0 0 0 0 0</pose>
-        </sensor>
-    </gazebo>
-    <joint name = "imu_link_joint6" type ="fixed">
-          <origin rpy="1.57 0 1.57" xyz="0 0 0"/>
-          <parent link="${arm_id}_link6"/>
-          <child link="imu_link6"/>
-          <axis xyz="0 0 0"/>
-    </joint>
-    <link name="imu_link6">
-        <inertial>
-            <origin xyz="0 0 0" rpy="0 0 0"/>
-            <mass value="0.0"/>
-            <inertia ixx="0.0" ixy="0.0" ixz="0.0" iyy="0.0" iyz="0.0" izz="0.0"/>
-        </inertial>
-        <visual>
-            <origin xyz="0.02 0.0 0.13" rpy="1.57 0 1.57" />
-            <geometry>
-                <box size = "0.05 0.05 0.05"/>
-            </geometry>
-        </visual>
-    </link>
-    <gazebo reference="imu_link6">
-        <gravity>true</gravity>
-        <!--      Below is the line to change the material-->
-        <material>Gazebo/YellowGlow</material>
-        <sensor name="imu_sensor6" type="imu">
-          <always_on>true</always_on>
-          <update_rate>100</update_rate>
-          <visualize>true</visualize>
-          <topic>imu_data0</topic>
-          <plugin filename="libgazebo_ros_imu_sensor.so" name="imu_plugin">
-            <topicName>imu_data6</topicName>
-            <bodyName>imu_link6</bodyName>
-            <updateRateHZ>100.0</updateRateHZ>
-            <gaussianNoise>0.0</gaussianNoise>
-            <xyzOffset>0.02 0.0 0.13</xyzOffset>
-            <rpyOffset>1.57 0 1.57</rpyOffset>
-            <frameName>imu_link6</frameName>
-          </plugin>
-          <pose>0 0 0 0 0 0</pose>
-        </sensor>
-    </gazebo>
-    <joint name = "imu_link_joint0_x_axis" type ="fixed">
-      <origin rpy="1.57 0 1.57" xyz="0 0 0"/>
-      <parent link="${arm_id}_link0"/>
-      <child link="imu_link_axes0_x_axis"/>
-      <axis xyz="0 0 0"/>
-    </joint>
-    <link name="imu_link_axes0_x_axis">
-      <inertial>
-        <origin xyz="0 0 0" rpy="0 0 0"/>
-        <mass value="0.0"/>
-        <inertia ixx="0.0" ixy="0.0" ixz="0.0" iyy="0.0" iyz="0.0" izz="0.0"/>
-      </inertial>
-      <visual>
-        <origin xyz="0.0 0.05 0.06" rpy="0 1.57 0" />
-          <geometry>
-            <mesh scale="0.007 0.007 0.007" filename="package://${axes_meshes}/meshes/visual/arrow.dae"/>
-          </geometry>
-        </visual>
-    </link>
-    <gazebo reference="imu_link_axes0_x_axis">
-    <gravity>true</gravity>
-    <material>Gazebo/RedBright</material>
-    </gazebo>
-    <joint name = "imu_link_joint0_y_axis" type ="fixed">
-      <origin rpy="1.57 0 1.57" xyz="0 0 0"/>
-      <parent link="${arm_id}_link0"/>
-      <child link="imu_link_axes0_y_axis"/>
-      <axis xyz="0 0 0"/>
-    </joint>
-    <link name="imu_link_axes0_y_axis">
-      <inertial>
-        <origin xyz="0 0 0" rpy="0 0 0"/>
-        <mass value="0.0"/>
-        <inertia ixx="0.0" ixy="0.0" ixz="0.0" iyy="0.0" iyz="0.0" izz="0.0"/>
-      </inertial>
-      <visual>
-        <origin xyz="0.0 0.05 0.06" rpy="-1.57 0 0" />
-          <geometry>
-            <mesh scale="0.007 0.007 0.007" filename="package://${axes_meshes}/meshes/visual/arrow.dae"/>
-          </geometry>
-        </visual>
-    </link>
-    <gazebo reference="imu_link_axes0_y_axis">
-    <gravity>true</gravity>
-    <material>Gazebo/Green</material>
-    </gazebo>
-    <joint name = "imu_link_joint0_z_axis" type ="fixed">
-      <origin rpy="1.57 0 1.57" xyz="0 0 0"/>
-      <parent link="${arm_id}_link0"/>
-      <child link="imu_link_axes0_z_axis"/>
-      <axis xyz="0 0 0"/>
-    </joint>
-    <link name="imu_link_axes0_z_axis">
-      <inertial>
-        <origin xyz="0 0 0" rpy="0 0 0"/>
-        <mass value="0.0"/>
-        <inertia ixx="0.0" ixy="0.0" ixz="0.0" iyy="0.0" iyz="0.0" izz="0.0"/>
-      </inertial>
-      <visual>
-        <origin xyz="0.0 0.05 0.06" rpy="0 0 1.57" />
-          <geometry>
-            <mesh scale="0.007 0.007 0.007" filename="package://${axes_meshes}/meshes/visual/arrow.dae"/>
-          </geometry>
-        </visual>
-    </link>
-    <gazebo reference="imu_link_axes0_z_axis">
-    <gravity>true</gravity>
-    <material>Gazebo/Blue</material>
-    </gazebo>
-    <joint name = "imu_link_joint1_x_axis" type ="fixed">
-      <origin rpy="1.57 0 1.57" xyz="0 0 0"/>
-      <parent link="${arm_id}_link1"/>
-      <child link="imu_link_axes1_x_axis"/>
-      <axis xyz="0 0 0"/>
-    </joint>
-    <link name="imu_link_axes1_x_axis">
-      <inertial>
-        <origin xyz="0 0 0" rpy="0 0 0"/>
-        <mass value="0.0"/>
-        <inertia ixx="0.0" ixy="0.0" ixz="0.0" iyy="0.0" iyz="0.0" izz="0.0"/>
-      </inertial>
-      <visual>
-        <origin xyz="0.0 -0.15 0.06" rpy="0 1.57 0" />
-          <geometry>
-            <mesh scale="0.007 0.007 0.007" filename="package://${axes_meshes}/meshes/visual/arrow.dae"/>
-          </geometry>
-        </visual>
-    </link>
-    <gazebo reference="imu_link_axes1_x_axis">
-    <gravity>true</gravity>
-    <material>Gazebo/RedBright</material>
-    </gazebo>
-    <joint name = "imu_link_joint1_y_axis" type ="fixed">
-      <origin rpy="1.57 0 1.57" xyz="0 0 0"/>
-      <parent link="${arm_id}_link1"/>
-      <child link="imu_link_axes1_y_axis"/>
-      <axis xyz="0 0 0"/>
-    </joint>
-    <link name="imu_link_axes1_y_axis">
-      <inertial>
-        <origin xyz="0 0 0" rpy="0 0 0"/>
-        <mass value="0.0"/>
-        <inertia ixx="0.0" ixy="0.0" ixz="0.0" iyy="0.0" iyz="0.0" izz="0.0"/>
-      </inertial>
-      <visual>
-        <origin xyz="0.0 -0.15 0.06" rpy="-1.57 0 0" />
-          <geometry>
-            <mesh scale="0.007 0.007 0.007" filename="package://${axes_meshes}/meshes/visual/arrow.dae"/>
-          </geometry>
-        </visual>
-    </link>
-    <gazebo reference="imu_link_axes1_y_axis">
-    <gravity>true</gravity>
-    <material>Gazebo/Green</material>
-    </gazebo>
-    <joint name = "imu_link_joint1_z_axis" type ="fixed">
-      <origin rpy="1.57 0 1.57" xyz="0 0 0"/>
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
File: robots/panda_arm_hand.urdf.xacro (robot description, xacro)
@@ -3,4 +3,5 @@
   <xacro:include filename="$(find ros_robotic_skin)/robots/panda_arm.xacro"/>
   <xacro:include filename="$(find franka_description)/robots/hand.xacro"/>
+  <xacro:include filename="$(find ros_robotic_skin)/robots/imu.xacro"/>
   <!-- for simulation -->
   <xacro:include filename="$(find franka_description)/robots/panda.gazebo.xacro"/>
@@ -9,4 +10,11 @@
   <xacro:panda_arm />
   <xacro:hand ns="panda" rpy="0 0 ${-pi/4}" connected_to="panda_link8"/>
+  <xacro:imu imu_id="0" xyz="0.06 0 0.1" rpy="0 1.57 0" gravity="true" type="fixed" connected_to="panda_link0"/>
+  <xacro:imu imu_id="1" xyz="0.05 0 -0.15" rpy="0 1.57 0" gravity="true" type="fixed" connected_to="panda_link1"/>
+  <xacro:imu imu_id="2" xyz="0 -0.12 0.05" rpy="0 0 0" gravity="true" type="fixed" connected_to="panda_link2"/>
+  <xacro:imu imu_id="3" xyz="0 -0.05 -0.08" rpy="1.57 0 0" gravity="true" type="fixed" connected_to="panda_link3"/>
+  <xacro:imu imu_id="4" xyz="-0.13 0.08 0" rpy="0 -1.57 0" gravity="true" type="fixed" connected_to="panda_link4"/>
+  <xacro:imu imu_id="5" xyz="0 0.1 -0.1" rpy="-1.57 0 0" gravity="true" type="fixed" connected_to="panda_link5"/>
+  <xacro:imu imu_id="6" xyz="0.13 0 0" rpy="0 1.57 0" gravity="true" type="fixed" connected_to="panda_link6"/>
   <!-- for simulation -->
   <xacro:arg name="robot_name" default="panda"/>
