Commit message: completed imu setting and deleted unnecessary files

File: robots/imu.xacro (robot description, xacro)
@@ -1,5 +1,5 @@
 <?xml version='1.0' encoding='utf-8'?>
 <robot xmlns:xacro="http://www.ros.org/wiki/xacro" name="imu">
-    <xacro:macro name="imu" params="imu_id:='0' xyz:='0 0 0' rpy:='0 0 0' boxxy:='0.05 0.05' boxz:='0.03' gravity:='false' type:='floating' freq:='50' connected_to:=''">
+    <xacro:macro name="imu" params="imu_id:='0' xyz:='0 0 0' rpy:='0 0 0' boxxy:='0.05 0.05' boxz:='0.03' gravity:='false' type:='fixed' freq:='100' connected_to:=''">
         <!-- Connect IMU to the world if not specified -->
         <xacro:if value="${connected_to == ''}">
@@ -18,5 +18,4 @@
                 <child link="imu_link${imu_id}"/>
                 <origin rpy="${rpy}" xyz="${xyz}"/>
-                <!-- <dynamics damping="100" friction="100"/> -->
             </joint>
         </xacro:if>
@@ -30,5 +29,5 @@
                 <origin xyz="0 0 ${displacement/2}" rpy="0 0 0"/>
                 <mass value="0.1"/>
-                <inertia ixx="0.0" ixy="0.0" ixz="0.0" iyy="0.0" iyz="0.0" izz="0.0"/>
+                <inertia ixx="0.1" ixy="0.0" ixz="0.0" iyy="0.1" iyz="0.0" izz="0.1"/>
             </inertial>
             <visual>
@@ -42,22 +41,21 @@
             <material>Gazebo/YellowGlow</material>
             <gravity>${gravity}</gravity>
+            <mu1>20</mu1>
+            <mu2>20</mu2>
             <sensor name="imu_sensor${imu_id}" type="imu">
-            <always_on>true</always_on>
-            <update_rate>${freq}</update_rate>
-            <visualize>true</visualize>
-            <topic>imu_data${imu_id}</topic>
-            <!-- <cfmDamping>true</cfmDamping> -->
-            <!-- <kp>10000</kp> -->
-            <!-- <kd>100</kd> -->
-            <plugin filename="libgazebo_ros_imu_sensor.so" name="imu_plugin">
-                <topicName>imu_data${imu_id}</topicName>
-                <bodyName>imu_link${imu_id}</bodyName>
-                <updateRateHZ>${freq}</updateRateHZ>
-                <gaussianNoise>0.0</gaussianNoise>
-                <xyzOffset>0.0 0.0 0.0</xyzOffset>
-                <rpyOffset>0 0 0</rpyOffset>
-                <frameName>imu_link${imu_id}</frameName>
-            </plugin>
-            <pose>0 0 0 0 0 0</pose>
+                <always_on>true</always_on>
+                <update_rate>${freq}</update_rate>
+                <visualize>true</visualize>
+                <topic>__default_topic__</topic>
+                <plugin filename="libgazebo_ros_imu_sensor.so" name="imu_plugin">
+                    <topicName>imu_data${imu_id}</topicName>
+                    <bodyName>imu_link${imu_id}</bodyName>
+                    <updateRateHZ>${freq}</updateRateHZ>
+                    <gaussianNoise>0.0</gaussianNoise>
+                    <xyzOffset>0.0 0.0 0.0</xyzOffset>
+                    <rpyOffset>0 0 0</rpyOffset>
+                    <frameName>imu_frame${imu_id}</frameName>
+                </plugin>
+                <pose>0 0 0 0 0 0</pose>
             </sensor>
         </gazebo>

File: robots/panda_arm_hand.urdf.xacro (robot description, xacro)
@@ -10,11 +10,11 @@
   <xacro:panda_arm />
   <xacro:hand ns="panda" rpy="0 0 ${-pi/4}" connected_to="panda_link8"/>
-  <xacro:imu imu_id="0" xyz="0.06 0 0.1" rpy="0 1.57 0" gravity="true" type="fixed" connected_to="panda_link0"/>
-  <xacro:imu imu_id="1" xyz="0.05 0 -0.15" rpy="0 1.57 0" gravity="true" type="fixed" connected_to="panda_link1"/>
-  <xacro:imu imu_id="2" xyz="0 -0.12 0.05" rpy="0 0 0" gravity="true" type="fixed" connected_to="panda_link2"/>
-  <xacro:imu imu_id="3" xyz="0 -0.05 -0.08" rpy="1.57 0 0" gravity="true" type="fixed" connected_to="panda_link3"/>
-  <xacro:imu imu_id="4" xyz="-0.13 0.08 0" rpy="0 -1.57 0" gravity="true" type="fixed" connected_to="panda_link4"/>
-  <xacro:imu imu_id="5" xyz="0 0.1 -0.1" rpy="-1.57 0 0" gravity="true" type="fixed" connected_to="panda_link5"/>
-  <xacro:imu imu_id="6" xyz="0.13 0 0" rpy="0 1.57 0" gravity="true" type="fixed" connected_to="panda_link6"/>
+  <xacro:imu imu_id="0" xyz="0.06 0 0.1" rpy="0 1.57 0" gravity="true" connected_to="panda_link0"/>
+  <xacro:imu imu_id="1" xyz="0.05 0 -0.15" rpy="0 1.57 0" gravity="true" connected_to="panda_link1"/>
+  <xacro:imu imu_id="2" xyz="0 -0.12 0.05" rpy="0 0 0" gravity="true" connected_to="panda_link2"/>
+  <xacro:imu imu_id="3" xyz="0 -0.05 -0.08" rpy="1.57 0 0" gravity="true" connected_to="panda_link3"/>
+  <xacro:imu imu_id="4" xyz="-0.13 0.08 0" rpy="0 -1.57 0" gravity="true" connected_to="panda_link4"/>
+  <xacro:imu imu_id="5" xyz="0 0.1 -0.1" rpy="-1.57 0 0" gravity="true" connected_to="panda_link5"/>
+  <xacro:imu imu_id="6" xyz="0.13 0 0" rpy="0 1.57 0" gravity="true" connected_to="panda_link6"/>
   <!-- for simulation -->
   <xacro:arg name="robot_name" default="panda"/>

Commit message: added xyz axes for imus

File: robots/imu.xacro (robot description, xacro)
@@ -1,5 +1,5 @@
 <?xml version='1.0' encoding='utf-8'?>
 <robot xmlns:xacro="http://www.ros.org/wiki/xacro" name="imu">
-    <xacro:macro name="imu" params="imu_id:='0' xyz:='0 0 0' rpy:='0 0 0' boxxy:='0.05 0.05' boxz:='0.03' gravity:='false' type:='fixed' freq:='100' connected_to:=''">
+    <xacro:macro name="imu" params="imu_id:='0' xyz:='0 0 0' rpy:='0 0 0' gravity:='false' type:='fixed' freq:='100' connected_to:=''">
         <!-- Connect IMU to the world if not specified -->
         <xacro:if value="${connected_to == ''}">
@@ -24,15 +24,17 @@
         <!-- To set the CoG to the joint, do not add any displacement -->
         <!-- To set the box base to the joint, add displacement-->
+        <xacro:property name="boxxy" value="0.05"/>
+        <xacro:property name="boxz" value="0.03"/>
         <xacro:property name="displacement" value="${boxz}"/>
         <link name="imu_link${imu_id}">
             <inertial>
-                <origin xyz="0 0 ${displacement/2}" rpy="0 0 0"/>
-                <mass value="0.1"/>
-                <inertia ixx="0.1" ixy="0.0" ixz="0.0" iyy="0.1" iyz="0.0" izz="0.1"/>
+                <origin xyz="0 0 0" rpy="0 0 0"/>
+                <mass value="0.01"/>
+                <inertia ixx="0.01" ixy="0.0" ixz="0.0" iyy="0.01" iyz="0.0" izz="0.01"/>
             </inertial>
             <visual>
-                <origin xyz="0 0 ${displacement/2}" rpy="0 0 0"/>
+                <origin xyz="0 0 0" rpy="0 0 0"/>
                 <geometry>
-                    <box size="${boxxy} ${boxz}"/>
+                    <box size="${boxxy} ${boxxy} ${boxz}"/>
                 </geometry>
             </visual>
@@ -60,4 +62,70 @@
             </sensor>
         </gazebo>
+        <!-- ////////////////////////////////////////// -->
+        <!--                    AXIS                    -->
+        <!-- ////////////////////////////////////////// -->
+        <joint name="imu${imu_id}_to_xaxis" type="fixed">
+            <parent link="imu_link${imu_id}"/>
+            <child link="imu_link${imu_id}_xaxis"/>
+            <origin rpy="0 1.57 0" xyz="0 0 0"/>
+        </joint>
+        <joint name="imu${imu_id}_to_yaxis" type="fixed">
+            <parent link="imu_link${imu_id}"/>
+            <child link="imu_link${imu_id}_yaxis"/>
+            <origin rpy="-1.57 0 0" xyz="0 0 0"/>
+        </joint>
+        <joint name="imu${imu_id}_to_zaxis" type="fixed">
+            <parent link="imu_link${imu_id}"/>
+            <child link="imu_link${imu_id}_zaxis"/>
+            <origin rpy="0 0 0" xyz="0 0 0"/>
+        </joint>
+        <link name="imu_link${imu_id}_xaxis">
+            <inertial>
+                <origin xyz="0 0 ${boxz}" rpy="0 0 0"/>
+                <mass value="0.001"/>
+                <inertia ixx="0.001" ixy="0.0" ixz="0.0" iyy="0.001" iyz="0.0" izz="0.001"/>
+            </inertial>
+            <visual>
+                <origin xyz="0 0 ${boxz}" rpy="0 0 0"/>
+                <geometry>
+                    <cylinder radius="${boxxy/20}" length="${2*boxz}"/>
+                </geometry>
+            </visual>
+        </link>
+        <link name="imu_link${imu_id}_yaxis">
+            <inertial>
+                <origin xyz="0 0 ${boxz}" rpy="0 0 0"/>
+                <mass value="0.001"/>
+                <inertia ixx="0.001" ixy="0.0" ixz="0.0" iyy="0.001" iyz="0.0" izz="0.001"/>
+            </inertial>
+            <visual>
+                <origin xyz="0 0 ${boxz}" rpy="0 0 0"/>
+                <geometry>
+                    <cylinder radius="${boxxy/20}" length="${2*boxz}"/>
+                </geometry>
+            </visual>
+        </link>
+        <link name="imu_link${imu_id}_zaxis">
+            <inertial>
+                <origin xyz="0 0 ${boxz}" rpy="0 0 0"/>
+                <mass value="0.001"/>
+                <inertia ixx="0.001" ixy="0.0" ixz="0.0" iyy="0.001" iyz="0.0" izz="0.001"/>
+            </inertial>
+            <visual>
+                <origin xyz="0 0 ${boxz}" rpy="0 0 0"/>
+                <geometry>
+                    <cylinder radius="${boxxy/20}" length="${2*boxz}"/>
+                </geometry>
+            </visual>
+        </link>
+        <gazebo reference="imu_link${imu_id}_xaxis">
+            <material>Gazebo/Red</material>
+        </gazebo>
+        <gazebo reference="imu_link${imu_id}_yaxis">
+            <material>Gazebo/Green</material>
+        </gazebo>
+        <gazebo reference="imu_link${imu_id}_zaxis">
+            <material>Gazebo/Blue</material>
+        </gazebo>
     </xacro:macro>
 </robot>

File: robots/sawyer.urdf.xacro (robot description, xacro)
@@ -23,9 +23,9 @@
   </xacro:if>
   <xacro:include filename="$(find ros_robotic_skin)/robots/imu.xacro"/>
-  <xacro:imu imu_id="0" xyz="0.06 0 0.08" rpy="0 1.57 0" gravity="true" connected_to="right_l0"/>
-  <xacro:imu imu_id="1" xyz="-0.06 0 0.05" rpy="0 -1.57 0" gravity="true" connected_to="right_l1"/>
+  <xacro:imu imu_id="0" xyz="0.07 0 0.08" rpy="0 1.57 0" gravity="true" connected_to="right_l0"/>
+  <xacro:imu imu_id="1" xyz="-0.07 0 0.05" rpy="0 -1.57 0" gravity="true" connected_to="right_l1"/>
   <xacro:imu imu_id="2" xyz="-0.05 0.0 0.1" rpy="0 -1.57 0" gravity="true" connected_to="right_l2"/>
   <xacro:imu imu_id="3" xyz="-0.05 0 -0.10" rpy="0 -1.57 0" gravity="true" connected_to="right_l3"/>
-  <xacro:imu imu_id="4" xyz="-0.04 0 0.10" rpy="0 -1.57 0" gravity="true" connected_to="right_l4"/>
+  <xacro:imu imu_id="4" xyz="-0.05 0 0.10" rpy="0 -1.57 0" gravity="true" connected_to="right_l4"/>
   <xacro:imu imu_id="5" xyz="-0.04 0 0.1" rpy="0 -1.57 0" gravity="true" connected_to="right_l5"/>
 <xacro:imu imu_id="6" xyz="0.0 0.03 0.1" rpy="-1.57 0 0" gravity="true" connected_to="right_l6"/>

Commit message: refactored DynamicPoseData Saver

File: robots/imu.xacro (robot description, xacro)
@@ -1,5 +1,5 @@
 <?xml version='1.0' encoding='utf-8'?>
 <robot xmlns:xacro="http://www.ros.org/wiki/xacro" name="imu">
-    <xacro:macro name="imu" params="imu_id:='0' xyz:='0 0 0' rpy:='0 0 0' gravity:='false' type:='fixed' freq:='100' connected_to:=''">
+    <xacro:macro name="imu" params="imu_id:='0' xyz:='0 0 0' rpy:='0 0 0' gravity:='true' type:='fixed' freq:='100' connected_to:=''">
         <!-- Connect IMU to the world if not specified -->
         <xacro:if value="${connected_to == ''}">

File: robots/panda_arm_hand.urdf.xacro (robot description, xacro)
@@ -10,20 +10,11 @@
   <xacro:panda_arm />
   <xacro:hand ns="panda" rpy="0 0 ${-pi/4}" connected_to="panda_link8"/>
-  <xacro:imu imu_id="0" xyz="0.05 0.0 -0.15" rpy="0.0 1.57 0.0" gravity="true" connected_to="panda_link1"/>
-  <xacro:imu imu_id="1" xyz="0.06 0.0 0.06" rpy="0.0 1.57 0.0" gravity="true" connected_to="panda_link2"/>
-  <xacro:imu imu_id="2" xyz="0.0 -0.05 -0.08" rpy="1.57 0.0 0.0" gravity="true" connected_to="panda_link3"/>
-  <xacro:imu imu_id="3" xyz="-0.06 0.0 0.08" rpy="0.0 -1.57 0.0" gravity="true" connected_to="panda_link4"/>
-  <xacro:imu imu_id="4" xyz="0.0 0.1 -0.1" rpy="-1.57 0.0 0.0" gravity="true" connected_to="panda_link5"/>
-  <xacro:imu imu_id="5" xyz="-0.05 0.0 0.03" rpy="0.0 -1.57 0.0" gravity="true" connected_to="panda_link6"/>
-  <xacro:imu imu_id="6" xyz="0.05 0.0 0.0" rpy="0.0 1.57 0.0" gravity="true" connected_to="panda_link7"/>
-  <!--
-  <xacro:imu imu_id="0" xyz="0.06 0 0.1" rpy="0 1.57 0" gravity="true" connected_to="panda_link0"/>
-  <xacro:imu imu_id="1" xyz="0.05 0 -0.15" rpy="0 1.57 0" gravity="true" connected_to="panda_link1"/>
-  <xacro:imu imu_id="2" xyz="0 -0.12 0.05" rpy="0 0 0" gravity="true" connected_to="panda_link2"/>
-  <xacro:imu imu_id="3" xyz="0 -0.05 -0.08" rpy="1.57 0 0" gravity="true" connected_to="panda_link3"/>
-  <xacro:imu imu_id="4" xyz="-0.13 0.08 0" rpy="0 -1.57 0" gravity="true" connected_to="panda_link4"/>
-  <xacro:imu imu_id="5" xyz="0 0.1 -0.1" rpy="-1.57 0 0" gravity="true" connected_to="panda_link5"/>
-  <xacro:imu imu_id="6" xyz="0.13 0 0" rpy="0 1.57 0" gravity="true" connected_to="panda_link6"/>
-  -->
+  <xacro:imu imu_id="0" xyz="0.05 0.0 -0.15" rpy="0.0 1.57 0.0" connected_to="panda_link1"/>
+  <xacro:imu imu_id="1" xyz="0.06 0.0 0.06" rpy="0.0 1.57 0.0" connected_to="panda_link2"/>
+  <xacro:imu imu_id="2" xyz="0.0 -0.05 -0.08" rpy="1.57 0.0 0.0" connected_to="panda_link3"/>
+  <xacro:imu imu_id="3" xyz="-0.06 0.0 0.08" rpy="0.0 -1.57 0.0" connected_to="panda_link4"/>
+  <xacro:imu imu_id="4" xyz="0.0 0.1 -0.1" rpy="-1.57 0.0 0.0" connected_to="panda_link5"/>
+  <xacro:imu imu_id="5" xyz="-0.05 0.0 0.03" rpy="0.0 -1.57 0.0" connected_to="panda_link6"/>
+  <xacro:imu imu_id="6" xyz="0.05 0.0 0.0" rpy="0.0 1.57 0.0" connected_to="panda_link7"/>
   <!-- for simulation -->
   <xacro:arg name="robot_name" default="panda"/>
