Commit message: Most recent commit to add-imu, will be working on this whenever I have free time, but not first priority

File: robots/panda_arm_hand.urdf.xacro (robot description, xacro)
@@ -4,4 +4,5 @@
   <xacro:include filename="$(find franka_description)/robots/hand.xacro"/>
   <xacro:include filename="$(find ros_robotic_skin)/robots/imu.xacro"/>
+  <xacro:include filename="$(find ros_robotic_skin)/robots/su.xacro"/>
   <!-- comment to open up pr-->
   <!-- for simulation -->
@@ -11,6 +12,6 @@
   <xacro:panda_arm />
   <xacro:hand ns="panda" rpy="0 0 ${-pi/4}" connected_to="panda_link8"/>
-  <xacro:imu imu_id="0" xyz="0.05 0.0 -0.15" rpy="0.0 1.57 0.0" gravity="true" connected_to="panda_link1"/>
-  <xacro:imu imu_id="7" xyz="0.05 0.0 -0.17" rpy="0.0 1.57 0.0" gravity="true" connected_to="panda_link1"/>
+  <!-- <xacro:imu imu_id="0" xyz="0.05 0.0 -0.15" rpy="0.0 1.57 0.0" gravity="true" connected_to="panda_link1"/>
+  <xacro:imu imu_id="7" xyz="0.05 0.0 -0.17" rpy="0.0 1.57 0.0" gravity="true" connected_to="panda_link1"/> -->
   <xacro:imu imu_id="1" xyz="0.06 0.0 0.06" rpy="0.0 1.57 0.0" gravity="true" connected_to="panda_link2"/>
   <xacro:imu imu_id="8" xyz="0.06 -0.02 0.06" rpy="0.0 1.57 0.0" gravity="true" connected_to="panda_link2"/>
@@ -25,4 +26,5 @@
   <xacro:imu imu_id="6" xyz="0.05 0.0 0.0" rpy="0.0 1.57 0.0" gravity="true" connected_to="panda_link7"/>
   <xacro:imu imu_id="13" xyz="0.05 0.0 0.02" rpy="0.0 1.57 0.0" gravity="true" connected_to="panda_link7"/>
+  <xacro:su su_id="0" xyz="0.05 0.0 -0.15" rpy="0.0 1.57 0.0" gravity="true" connected_to="panda_link1"/>
   <!--
   <xacro:imu imu_id="0" xyz="0.06 0 0.1" rpy="0 1.57 0" gravity="true" connected_to="panda_link0"/>

File: robots/su.xacro (robot description, xacro)
@@ -1,23 +1,37 @@
 <?xml version='1.0' encoding='utf-8'?>
-<robot xmlns:xacro="http://www.ros.org/wiki/xacro" name="imu">
-    <xacro:macro name="imu" params="imu_id:='0' xyz:='0 0 0' rpy:='0 0 0' gravity:='false' type:='fixed' freq:='100' connected_to:=''">
-        <!-- Connect IMU to the world if not specified -->
+<robot xmlns:xacro="http://www.ros.org/wiki/xacro" name="su">
+  <!-- <xacro:include filename="$(find ros_robotic_skin)/robots/imu.xacro"/> -->
+    <xacro:macro name="su" params="su_id:='0' xyz:='0 0 0' rpy:='0 0 0' gravity:='false' type:='fixed' freq:='100' connected_to:=''">
+        <!-- Connect SU to the world if not specified -->
         <xacro:if value="${connected_to == ''}">
-            <joint name="imu${imu_id}_to_world" type="${type}">
+            <joint name="su${su_id}_to_world" type="${type}">
                 <!-- XYZ, RPY from parent Visual Origin (Center o Gravity) -->
                 <!-- in this case it's 0 0 0-->
                 <parent link="world" />
-                <child link="imu_link${imu_id}" />
+                <child link="su_link${su_id}" />
                 <origin rpy="${rpy}" xyz="${xyz}"/>
             </joint>
         </xacro:if>
-        <!-- Connect IMU to ${connected_to} if specified -->
+        <!-- Connect SU to ${connected_to} if specified -->
         <xacro:if value="${connected_to != ''}">
-            <joint name="imu${imu_id}_to_${connected_to}" type="${type}">
+            <joint name="su${su_id}_to_${connected_to}" type="${type}">
                 <parent link="${connected_to}"/>
-                <child link="imu_link${imu_id}"/>
+                <child link="su_link${su_id}"/>
                 <origin rpy="${rpy}" xyz="${xyz}"/>
             </joint>
         </xacro:if>
+        <!-- Connecting 2 IMUs to the SU -->
+        <!-- <xacro:if value="${rpy[0] != '0'}">
+            <xacro:imu imu_id="{su_id + 0}" xyz="{xyz}" rpy="{rpy}" gravity="true" connected_to="panda_link{su_id + 1}"/>
+            <xacro:imu imu_id="{su_id + 1}" xyz="{xyz[0] + 0.02} {xyz[1]} {xyz[2]}" rpy="{rpy}" gravity="true" connected_to="panda_link{su_id + 1}"/>
+        </xacro:if>
+        <xacro:if value="${rpy[1] != '0'}">
+            <xacro:imu imu_id="{su_id + 0}" xyz="{xyz}" rpy="{rpy}" gravity="true" connected_to="panda_link{su_id + 1}"/>
+            <xacro:imu imu_id="{su_id + 1}" xyz="{xyz[0]} {xyz[1] + 0.02} {xyz[2]}" rpy="{rpy}" gravity="true" connected_to="panda_link{su_id + 1}"/>
+        </xacro:if>
+        <xacro:if value="${rpy[2] != '0'}">
+            <xacro:imu imu_id="{su_id + 0}" xyz="{xyz}" rpy="{rpy}" gravity="true" connected_to="panda_link{su_id + 1}"/>
+            <xacro:imu imu_id="{su_id + 1}" xyz="{xyz[0]} {xyz[1]} {xyz[2] + 0.02}" rpy="{rpy}" gravity="true" connected_to="panda_link{su_id + 1}"/>
+        </xacro:if> -->
         <!-- XYZ, RPY from the joint-->
         <!-- in this case it's imu_to_world${imu_id}-->
@@ -27,5 +41,5 @@
         <xacro:property name="boxz" value="0.03"/>
         <xacro:property name="displacement" value="${boxz}"/>
-        <link name="imu_link${imu_id}">
+        <link name="su_link${su_id}">
             <inertial>
                 <origin xyz="0 0 0" rpy="0 0 0"/>
@@ -40,10 +54,10 @@
             </visual>
         </link>
-        <gazebo reference="imu_link${imu_id}">
+        <!-- <gazebo reference="su_link${su_id}">
             <material>Gazebo/YellowGlow</material>
             <gravity>${gravity}</gravity>
             <mu1>20</mu1>
             <mu2>20</mu2>
-            <sensor name="imu_sensor${imu_id}" type="imu">
+            <sensor name="su_sensor${su_id}" type="su">
                 <always_on>true</always_on>
                 <update_rate>${freq}</update_rate>
@@ -61,9 +75,9 @@
                 <pose>0 0 0 0 0 0</pose>
             </sensor>
-        </gazebo>
+        </gazebo> -->
         <!-- ////////////////////////////////////////// -->
         <!--                    AXIS                    -->
         <!-- ////////////////////////////////////////// -->
-        <joint name="imu${imu_id}_to_xaxis" type="fixed">
+        <!-- <joint name="imu${imu_id}_to_xaxis" type="fixed">
             <parent link="imu_link${imu_id}"/>
             <child link="imu_link${imu_id}_xaxis"/>
@@ -127,5 +141,5 @@
         <gazebo reference="imu_link${imu_id}_zaxis">
             <material>Gazebo/Blue</material>
-        </gazebo>
+        </gazebo> -->
     </xacro:macro>
 </robot>
