Commit message: Ready to start collaboration with Garrett

File: robots/control_point.xacro (robot description, xacro)
@@ -1,4 +1,4 @@
 <?xml version='1.0' encoding='utf-8'?>
-<robot xmlns:xacro="http://www.ros.org/wiki/xacro" name="imu">
+<robot xmlns:xacro="http://www.ros.org/wiki/xacro" name="control_point">
     <xacro:macro name="control_point" params=" point_id:='0' parent_id:='8' rpy:='0 0 0' xyz:='0 0 0' ">
     <link name="control_point${point_id}"></link>
@@ -9,3 +9,11 @@
     </joint>
   </xacro:macro>
+  <xacro:macro name="end_effector">
+    <link name="end_effector"></link>
+    <joint name="end_effector_to_panda_link8" type="fixed">
+      <parent link="panda_link8"/>
+      <child link="end_effector"/>
+      <origin rpy="0 0 0" xyz="0 0 0.10"/>
+    </joint>
+  </xacro:macro>
 </robot>

File: robots/panda_arm_hand_flacco.urdf.xacro (robot description, xacro)
@@ -16,5 +16,5 @@
   <xacro:control_point point_id='3' parent_id='5' rpy='0 0 0' xyz='0 0 -${0.333/2}'/>
   <!-- end effector control point -->
-  <xacro:control_point point_id='4' parent_id='8' rpy='0 0 0' xyz='0 0 0.0584'/>
+  <xacro:end_effector/>
   <!-- for simulation -->
   <xacro:arg name="robot_name" default="panda"/>

Commit message: Proximity sensors with pose bug

File: robots/control_point.xacro (robot description, xacro)
@@ -1,5 +1,5 @@
 <?xml version='1.0' encoding='utf-8'?>
 <robot xmlns:xacro="http://www.ros.org/wiki/xacro" name="control_point">
-    <xacro:macro name="control_point" params=" point_id:='0' parent_id:='8' rpy:='0 0 0' xyz:='0 0 0' ">
+  <xacro:macro name="control_point" params=" point_id:='0' parent_id:='8' rpy:='0 0 0' xyz:='0 0 0' ">
     <link name="control_point${point_id}"></link>
     <joint name="control_point${point_id}_to_panda_link${parent_id}" type="fixed">

File: robots/panda_arm_hand_flacco.urdf.xacro (robot description, xacro)
@@ -11,5 +11,5 @@
   <xacro:hand ns="panda" rpy="0 0 ${-pi/4}" connected_to="panda_link8"/>
   <!-- As many control points as needed to cover the robot body -->
-  <xacro:control_point point_id='0  ' parent_id='3' rpy='0 0 0' xyz='0 0 -${0.333/2}'/>
+  <xacro:control_point point_id='0' parent_id='3' rpy='0 0 0' xyz='0 0 -${0.333/2}'/>
   <!-- <xacro:control_point point_id='0' parent_id='8' rpy='0 0 0' xyz='0 0 0'/>
   <xacro:control_point point_id='1' parent_id='7' rpy='0 0 0' xyz='0 -${0.333/2} 0'/>

Commit message: Tune spheres

File: robots/control_point.xacro (robot description, xacro)
@@ -1,10 +1,10 @@
 <?xml version='1.0' encoding='utf-8'?>
 <robot xmlns:xacro="http://www.ros.org/wiki/xacro" name="control_point">
-  <xacro:macro name="control_point" params=" point_id:='0' parent_id:='8' rpy:='0 0 0' xyz:='0 0 0' ">
+  <xacro:macro name="control_point" params=" point_id:='0' parent_id:='8' rpy:='0 0 0' x0y0:='0 0' z0:='0' ">
     <link name="control_point${point_id}"></link>
     <joint name="control_point${point_id}_to_panda_link${parent_id}" type="fixed">
       <parent link="panda_link${parent_id}"/>
       <child link="control_point${point_id}"/>
-      <origin rpy="${rpy}" xyz="${xyz}"/>
+      <origin rpy="${rpy}" xyz="${x0y0} ${z0}"/>
     </joint>
   </xacro:macro>

File: robots/panda_arm_hand_flacco.urdf.xacro (robot description, xacro)
@@ -13,12 +13,11 @@
   <!-- As many control points as needed to cover the robot body -->
   <!-- <xacro:control_point point_id='0' parent_id='3' rpy='0 0 0' xyz='0 0 -${0.333/2}'/> -->
-  <!-- <xacro:control_point point_id='0' parent_id='8' rpy='0 0 0' xyz='0 0 0'/>
-  <xacro:control_point point_id='1' parent_id='7' rpy='0 0 0' xyz='0 -${0.333/2} 0'/>
-  <xacro:control_point point_id='2' parent_id='5' rpy='0 0 0' xyz='0 0 0'/>
-  <xacro:control_point point_id='3' parent_id='5' rpy='0 0 0' xyz='0 0 -${0.333/2}'/>
-  <xacro:control_point point_id='4' parent_id='4' rpy='0 0 0' xyz='0 0 -${0.333/2}'/>
-  <xacro:control_point point_id='5' parent_id='3' rpy='0 0 0' xyz='0 0 0'/>
-  <xacro:control_point point_id='6' parent_id='3' rpy='0 0 0' xyz='0 0 -${0.333/2}'/>
-  <xacro:control_point point_id='7' parent_id='2' rpy='0 0 0' xyz='0 0 0'/> -->
+  <xacro:control_point point_id='0' parent_id='8' z0='0.01'/>
+  <xacro:control_point point_id='1' parent_id='7' x0y0='-0.05 -0.03' z0='-0.03'/>
+  <xacro:control_point point_id='2' parent_id='5' x0y0='0 0.07' z0='-0.09'/>
+  <xacro:control_point point_id='3' parent_id='5' x0y0='0 0' z0='-0.25'/>
+  <xacro:control_point point_id='4' parent_id='4'/>
+  <xacro:control_point point_id='5' parent_id='3' x0y0='0 0' z0='-0.1'/>
+  <xacro:control_point point_id='6' parent_id='3' x0y0='0 0' z0='-0.3'/>
   <!-- end effector control point -->
   <xacro:end_effector/>

Commit message: CartesianPositionController working in real robot. Need to check panda_EE

File: robots/control_point.xacro (robot description, xacro)
@@ -9,9 +9,9 @@
     </joint>
   </xacro:macro>
-  <xacro:macro name="end_effector">
-    <link name="end_effector"></link>
-    <joint name="end_effector_to_panda_link8" type="fixed">
+  <xacro:macro name="panda_EE">
+    <link name="panda_EE"></link>
+    <joint name="panda_EE_to_panda_link8" type="fixed">
       <parent link="panda_link8"/>
-      <child link="end_effector"/>
+      <child link="panda_EE"/>
       <origin rpy="0 0 0" xyz="0 0 0.10"/>
     </joint>

File: robots/panda_arm_hand_flacco.urdf.xacro (robot description, xacro)
@@ -22,5 +22,5 @@
   <xacro:control_point point_id='7' parent_id='0' x0y0='-0.05 0' z0='0.1'/>
   <!-- end effector control point -->
-  <xacro:end_effector/>
+  <xacro:panda_EE/>
   <!-- Proximity sensors -->
   <xacro:property name="sensors_per_ring" value="16"/>
